File: Steuerwerk.kicad_pcb (KiCad board)
At the start: 2 copper layers, 100 x 160 mm, 117 parts, among them J1 2PinTerminalBlocktg, J10 2PinTerminalBlocktg, J11 2PinTerminalBlocktg, J12 2PinTerminalBlocktg, J2 2PinTerminalBlocktg, J3 3PinTerminalBlocktg, J4 3PinTerminalBlocktg, J5 2PinTerminalBlocktg, J6 2PinTerminalBlocktg, J7 2PinTerminalBlocktg, J8 2PinTerminalBlocktg, J9 2PinTerminalBlocktg, Q1 Q_PNP_BCE, U2 74541, U3 74LS161, U4 74LS138, U5 74LS138, U6 74541, U7 74LS374, U8 74LS374, U9 74ls240

Commit message: redesign Steuerwerk angefangen
Parts:
- removed G***: LOGO, allBonsaiFootprintsLibs:agi5
- removed the REF** at (141.6, 193.6)
- added REF**: EuroBoard160mmX100mm_holes, allBonsaiFootprintsLibs:EuroBoard160mmX100mm_holes, F.Cu at (140.9, 193.3)
- D17, D18, D19, D20, D21, D23, D24, D25, D26, D27, D28, D30, D31, D33, D35, D37, D38, D39, D40: footprint tg_foodprint:LED_D1.8mm_W3.3mm_H2.4mmBonsai -> LED_THT:LED_D3.0mm
- D42, D43, D44, D45, D46, D47, D48, D49, D50, D51, D52, D53, D54, D55, D56, D57, D58, D59, D60, D61: footprint tg_foodprint:LED_D1.8mm_W3.3mm_H2.4mmBonsai -> LED_THT:LED_D1.8mm_W3.3mm_H2.4mm
- moved D50 154.1 mm to (-38.4, 83.5)
- moved D63 153.1 mm to (-34.9, 93.7)
- moved D51 146.7 mm to (-30.8, 89.6)
- moved D42 146.4 mm to (-38.4, 97.2)
- moved D53 145.9 mm to (-30.3, 93.7)
- moved D57 145.3 mm to (-29.8, 101.8)
- moved D56 143.9 mm to (-28.3, 98.3)
- moved D39 141.2 mm to (-49.6, 83.0)
- moved D30 140.7 mm to (-59.3, 84.0)
- moved D26 139.6 mm to (-60.8, 89.6)
- moved D38 139.6 mm to (-50.6, 89.1)
- moved D40 139.1 mm to (-47.6, 96.2)
- moved D27 139.1 mm to (-60.3, 100.8)
- moved D43 138.4 mm to (-27.9, 64.7)
- moved D37 138.3 mm to (-49.2, 79.2)
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Connections:
- U2 pad 8: (no net) -> Net-(U2-Pad8)
- U3 pad 15: (no net) -> Net-(U3-Pad15)
- U5 pad 7: (no net) -> Net-(U5-Pad7)
- U7 pad 2: (no net) -> Net-(U2-Pad8)
Routing:
- net VCC: track 1013.5 -> 879.0 mm, vias 9 -> 3
- net GND: track 542.3 -> 418.5 mm, vias 9 -> 7
- net /Takt: track 184.2 -> 83.5 mm, vias 2 -> 0
- net (no net): track 97.1 -> 0.00 mm
- net /clrMPC: track 182.9 -> 102.6 mm, vias 1 -> 0
- net Net-(D21-Pad2): track 71.9 -> 1.21 mm
- net Net-(D23-Pad2): track 67.8 -> 0.00 mm
- net /b3: track 54.6 -> 111.3 mm
- net /b7: track 54.6 -> 0.00 mm
- net /b2: track 63.3 -> 117.6 mm
- net /b8: track 64.4 -> 10.9 mm
- net Net-(J9-Pad2): track 72.3 -> 22.1 mm
- net Net-(J10-Pad2): track 74.3 -> 27.5 mm
- net /5: track 81.4 -> 36.5 mm
- net /16: track 79.2 -> 34.7 mm
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
Commit message: vor Umbau 74541 im Schaltplan
Parts:
- U9: value 74ls240 -> 74240
Connections:
- U2 pad 4: Net-(J7-Pad2) -> Net-(U2-Pad4)
- U2 pad 6: Net-(J6-Pad2) -> Net-(U2-Pad6)
- U6 pad 4: Net-(J11-Pad2) -> Net-(U6-Pad4)
- U6 pad 6: Net-(J10-Pad2) -> Net-(U6-Pad6)
- U6 pad 8: Net-(J9-Pad2) -> Net-(U6-Pad8)
- U7 pad 5: Net-(J6-Pad2) -> Net-(U2-Pad6)
- U7 pad 6: Net-(J7-Pad2) -> Net-(U2-Pad4)
- U8 pad 2: Net-(J9-Pad2) -> Net-(U6-Pad8)
- U8 pad 5: Net-(J10-Pad2) -> Net-(U6-Pad6)
- U8 pad 6: Net-(J11-Pad2) -> Net-(U6-Pad4)
Routing:
- net Net-(U2-Pad4): track 0.00 -> 9.42 mm
- net Net-(J7-Pad2): track 36.1 -> 26.7 mm
- net Net-(U6-Pad4): track 0.00 -> 5.96 mm
- net Net-(J11-Pad2): track 47.8 -> 41.8 mm
- net Net-(J6-Pad2): track 31.1 -> 26.4 mm
- net Net-(U2-Pad6): track 0.00 -> 4.74 mm
- net Net-(J10-Pad2): track 27.5 -> 25.3 mm
- net Net-(U6-Pad6): track 0.00 -> 2.20 mm
- net Net-(J9-Pad2): track 22.1 -> 20.3 mm
- net Net-(U6-Pad8): track 0.00 -> 1.80 mm

Commit message: Steuerwerk: beide 74541 umgebaut
Parts:
- U2, U6: footprint Housings_DIP:DIP-20_W7.62mm_Socket_LongPads -> Package_DIP:DIP-20_W7.62mm_Socket_LongPads

Commit message: Steuerwerk vor Entfernen der Busse
Connections:
- D17 pad 1: /a1 -> Net-(D17-Pad1)
- D18 pad 1: /a1 -> Net-(D17-Pad1)
- D19 pad 1: /a1 -> Net-(D17-Pad1)
- D20 pad 1: /a1 -> Net-(D17-Pad1)
- D21 pad 1: /a2 -> Net-(D21-Pad1)
- D21 pad 2: Net-(D21-Pad2) -> Net-(D17-Pad2)
- D23 pad 1: /a3 -> Net-(D23-Pad1)
- D24 pad 1: /a3 -> Net-(D23-Pad1)
- D24 pad 2: Net-(D21-Pad2) -> Net-(D17-Pad2)
- D25 pad 1: /a3 -> Net-(D23-Pad1)
- D25 pad 2: Net-(D25-Pad2) -> Net-(D17-Pad2)
- D26 pad 1: /a3 -> Net-(D23-Pad1)
- D27 pad 1: /a3 -> Net-(D23-Pad1)
- D28 pad 1: /a3 -> Net-(D23-Pad1)
- D30 pad 1: /a4 -> Net-(D30-Pad1)
- D31 pad 1: /a4 -> Net-(D30-Pad1)
- D33 pad 1: /a5 -> Net-(D17-Pad2)
- D33 pad 2: Net-(D33-Pad2) -> Net-(D17-Pad2)
- D35 pad 1: /a6 -> Net-(D35-Pad1)
- D37 pad 1: /a7 -> Net-(D37-Pad1)
- D37 pad 2: Net-(D25-Pad2) -> Net-(D17-Pad2)
- D38 pad 1: /a7 -> Net-(D37-Pad1)
- D39 pad 1: /a8 -> Net-(D39-Pad1)
- D40 pad 1: /a8 -> Net-(D39-Pad1)
- D42 pad 1: /b1 -> Net-(D42-Pad1)
- D43 pad 1: /b2 -> Net-(D43-Pad1)
- D44 pad 1: /b2 -> Net-(D43-Pad1)
- D45 pad 1: /b2 -> Net-(D43-Pad1)
- D45 pad 2: Net-(D21-Pad2) -> Net-(D17-Pad2)
- D46 pad 1: /b3 -> Net-(D46-Pad1)
- D47 pad 1: /b4 -> Net-(D17-Pad2)
- D47 pad 2: Net-(D47-Pad2) -> Net-(D17-Pad2)
- D48 pad 1: /b4 -> Net-(D17-Pad2)
- D48 pad 2: Net-(D25-Pad2) -> Net-(D17-Pad2)
- D49 pad 1: /b4 -> Net-(D17-Pad2)
- D49 pad 2: Net-(D33-Pad2) -> Net-(D17-Pad2)
- D50 pad 1: /b4 -> Net-(D17-Pad2)
- D51 pad 1: /b4 -> Net-(D17-Pad2)
- D52 pad 1: /b4 -> Net-(D17-Pad2)
- D53 pad 1: /b4 -> Net-(D17-Pad2)
- D54 pad 1: /b4 -> Net-(D17-Pad2)
- D55 pad 1: /b4 -> Net-(D17-Pad2)
- D56 pad 1: /b4 -> Net-(D17-Pad2)
- D57 pad 1: /b4 -> Net-(D17-Pad2)
- D58 pad 1: /b4 -> Net-(D17-Pad2)
- D59 pad 1: /b5 -> Net-(D59-Pad1)
- D59 pad 2: Net-(D33-Pad2) -> Net-(D17-Pad2)
- D60 pad 1: /b5 -> Net-(D59-Pad1)
- D61 pad 1: /b6 -> Net-(D61-Pad1)
- D63 pad 1: /b5 -> Net-(D59-Pad1)
- R16 pad 1: /a2 -> Net-(D21-Pad1)
- RP1 pad 4: /b3 -> VCC
- RP1 pad 6: /b5 -> /b4
- U3 pad 9: /a2 -> Net-(D21-Pad1)
- U4 pad 10: Net-(D33-Pad2) -> Net-(D17-Pad2)
- U4 pad 11: Net-(D25-Pad2) -> Net-(D17-Pad2)
- U4 pad 12: Net-(D47-Pad2) -> Net-(D17-Pad2)
- U4 pad 13: Net-(D21-Pad2) -> Net-(D17-Pad2)
- U7 pad 13: /a7 -> Net-(D37-Pad1)
- U7 pad 14: /a5 -> Net-(D17-Pad2)
- U7 pad 17: /a3 -> Net-(D23-Pad1)
- U7 pad 18: /a1 -> Net-(D17-Pad1)
- U7 pad 3: /a2 -> Net-(D21-Pad1)
- U7 pad 4: /a4 -> Net-(D30-Pad1)
- U7 pad 7: /a6 -> Net-(D35-Pad1)
- U7 pad 8: /a8 -> Net-(D39-Pad1)
- U8 pad 13: /b7 -> Net-(U8-Pad13)
- U8 pad 14: /b5 -> Net-(D59-Pad1)
- U8 pad 17: /b3 -> Net-(D46-Pad1)
- U8 pad 18: /b1 -> Net-(D42-Pad1)
- U8 pad 3: /b2 -> Net-(D43-Pad1)
- U8 pad 4: /b4 -> Net-(D17-Pad2)
- U8 pad 7: /b6 -> Net-(D61-Pad1)
- U8 pad 8: /b8 -> Net-(U8-Pad8)
Routing:
- net /b5: track 63.3 -> 0.00 mm
- net /b3: track 111.3 -> 50.2 mm
- net VCC: track 879.0 -> 940.1 mm
- net /b4: track 72.5 -> 125.3 mm
- net Net-(D21-Pad1): track 0.00 -> 49.4 mm
- net /a2: track 110.7 -> 61.4 mm
- net Net-(D17-Pad2): track 50.2 -> 64.0 mm
- net Net-(U8-Pad8): track 0.00 -> 10.9 mm
- net /b8: track 10.9 -> 0.00 mm
- net /a6: track 71.4 -> 61.4 mm
- net Net-(D61-Pad1): track 0.00 -> 10.1 mm
- net Net-(D35-Pad1): track 0.00 -> 10.1 mm
- net Net-(D30-Pad1): track 0.00 -> 10.1 mm
- net /b6: track 74.6 -> 64.6 mm
- net /a8: track 74.0 -> 63.9 mm
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
Commit message: weitergemacht
Parts:
- removed J10, J11, J12: 2PinTerminalBlocktg, 2PinTerminalBlocktg
- J6, J8: value 2PinTerminalBlocktg -> Conn_01x02; footprint 2PinTerminalBlocktg -> Connector_Molex:Molex_KK-254_AE-6410-02A_1x02_P2.54mm_Vertical
- J7, J9: value 2PinTerminalBlocktg -> Conn_01x04; footprint 2PinTerminalBlocktg -> Connector_Molex:Molex_KK-254_AE-6410-04A_1x04_P2.54mm_Vertical
- R11, R13, R14, R15, R17, R19, R2, R21, R24, R26, R28, R3, R30, R5, R7, R9: value R -> 330
- moved J9 12.5 mm to (106.7, 188.6)
- moved J8 11.9 mm to (95.9, 187.9)
- moved J6 10.1 mm to (73.7, 187.9)
- moved J7 8.19 mm to (82.0, 187.9)
- moved C5 0.40 mm to (100.4, 153.6)
- moved U2 0.36 mm to (97.2, 147.3)
- moved U6 0.36 mm to (126.4, 147.3)
- moved C4 0.08 mm to (103.9, 127.0)
Connections:
- net /15 renamed Net-(U6-Pad3)
- net /16 renamed Net-(U6-Pad2)
- net /3 renamed Net-(J6-Pad1)
- net /5 renamed Net-(J7-Pad1)
- D21 pad 2: Net-(D17-Pad2) -> Net-(D21-Pad2)
- D24 pad 2: Net-(D17-Pad2) -> Net-(D21-Pad2)
- D25 pad 2: Net-(D17-Pad2) -> Net-(D25-Pad2)
- D30 pad 2: Net-(D17-Pad2) -> Net-(D30-Pad2)
- D33 pad 1: Net-(D17-Pad2) -> Net-(D33-Pad1)
- D33 pad 2: Net-(D17-Pad2) -> Net-(D33-Pad2)
- D37 pad 2: Net-(D17-Pad2) -> Net-(D25-Pad2)
- D39 pad 2: Net-(D17-Pad2) -> Net-(D30-Pad2)
- D45 pad 2: Net-(D17-Pad2) -> Net-(D21-Pad2)
- D47 pad 1: Net-(D17-Pad2) -> Net-(D47-Pad1)
- D48 pad 1: Net-(D17-Pad2) -> Net-(D47-Pad1)
- D48 pad 2: Net-(D17-Pad2) -> Net-(D25-Pad2)
- D49 pad 1: Net-(D17-Pad2) -> Net-(D47-Pad1)
- D49 pad 2: Net-(D17-Pad2) -> Net-(D33-Pad2)
- D50 pad 1: Net-(D17-Pad2) -> Net-(D47-Pad1)
- D50 pad 2: Net-(D17-Pad2) -> Net-(D30-Pad2)
- D51 pad 1: Net-(D17-Pad2) -> Net-(D47-Pad1)
- D52 pad 1: Net-(D17-Pad2) -> Net-(D47-Pad1)
- D53 pad 1: Net-(D17-Pad2) -> Net-(D47-Pad1)
- D54 pad 1: Net-(D17-Pad2) -> Net-(D47-Pad1)
- D55 pad 1: Net-(D17-Pad2) -> Net-(D47-Pad1)
- D56 pad 1: Net-(D17-Pad2) -> Net-(D47-Pad1)
- D57 pad 1: Net-(D17-Pad2) -> Net-(D47-Pad1)
- D58 pad 1: Net-(D17-Pad2) -> Net-(D47-Pad1)
- D59 pad 2: Net-(D17-Pad2) -> Net-(D33-Pad2)
- J4 pad 1: /11 -> /loadIR
- J8 pad 1: /7 -> Net-(J8-Pad1)
- J8 pad 2: /enAkku -> Net-(J8-Pad2)
- J9 pad 1: /9 -> /loadIR
- RP1 pad 2: /b1 -> Net-(D42-Pad1)
- RP1 pad 3: /b2 -> Net-(D43-Pad1)
- RP1 pad 4: VCC -> Net-(D46-Pad1)
- RP1 pad 5: /b4 -> Net-(D47-Pad1)
- RP1 pad 6: /b4 -> Net-(D59-Pad1)
- RP1 pad 7: /b6 -> Net-(D61-Pad1)
- RP1 pad 8: /b7 -> Net-(RP1-Pad8)
- RP1 pad 9: /b8 -> Net-(RP1-Pad9)
- RP2 pad 2: /a1 -> Net-(D17-Pad1)
- RP2 pad 3: /a2 -> Net-(D21-Pad1)
- RP2 pad 4: /a3 -> Net-(D23-Pad1)
- RP2 pad 5: /a4 -> Net-(D30-Pad1)
- RP2 pad 6: /a5 -> Net-(D33-Pad1)
- RP2 pad 7: /a6 -> Net-(D35-Pad1)
- RP2 pad 8: /a7 -> Net-(D37-Pad1)
- RP2 pad 9: /a8 -> Net-(D39-Pad1)
- U2 pad 3: /7 -> Net-(J7-Pad3)
- U2 pad 4: Net-(U2-Pad4) -> Net-(J7-Pad2)
- U2 pad 6: Net-(U2-Pad6) -> Net-(J6-Pad2)
- U4 pad 10: Net-(D17-Pad2) -> Net-(D33-Pad2)
- U4 pad 11: Net-(D17-Pad2) -> Net-(D25-Pad2)
- U4 pad 13: Net-(D17-Pad2) -> Net-(D21-Pad2)
- U4 pad 9: Net-(D17-Pad2) -> Net-(D30-Pad2)
- U6 pad 4: Net-(U6-Pad4) -> Net-(J9-Pad4)
- U6 pad 5: /13 -> Net-(J9-Pad3)
- U6 pad 6: Net-(U6-Pad6) -> Net-(J9-Pad2)
- U6 pad 7: /11 -> /loadIR
- U6 pad 8: Net-(U6-Pad8) -> Net-(J8-Pad2)
- U6 pad 9: /9 -> Net-(J8-Pad1)
- U7 pad 12: /7 -> Net-(J7-Pad3)
- U7 pad 14: Net-(D17-Pad2) -> Net-(D33-Pad1)
- U7 pad 5: Net-(U2-Pad6) -> Net-(J6-Pad2)
- U7 pad 6: Net-(U2-Pad4) -> Net-(J7-Pad2)
- U8 pad 13: Net-(U8-Pad13) -> Net-(RP1-Pad8)
- U8 pad 15: /13 -> Net-(J9-Pad3)
- U8 pad 16: /11 -> /loadIR
- U8 pad 19: /9 -> Net-(J8-Pad1)
- U8 pad 2: Net-(U6-Pad8) -> Net-(J8-Pad2)
- U8 pad 4: Net-(D17-Pad2) -> Net-(D47-Pad1)
- U8 pad 5: Net-(U6-Pad6) -> Net-(J9-Pad2)
- U8 pad 6: Net-(U6-Pad4) -> Net-(J9-Pad4)
- U8 pad 8: Net-(U8-Pad8) -> Net-(RP1-Pad9)
Routing:
- net VCC: track 940.1 -> 639.1 mm
- net /b4: track 125.3 -> 0.00 mm
- net /11: track 107.9 -> 0.00 mm, vias 2 -> 0
- net GND: track 418.5 -> 336.4 mm, vias 7 -> 4
- net /enSTW: track 136.9 -> 67.8 mm, vias 6 -> 3
- net /b6: track 64.6 -> 0.00 mm
- net /a8: track 63.9 -> 0.00 mm
- net Net-(D59-Pad1): track 0.00 -> 63.3 mm
- net /a1: track 63.0 -> 0.00 mm
- net Net-(D37-Pad1): track 0.00 -> 62.6 mm
- net /a7: track 62.6 -> 0.00 mm
- net Net-(D17-Pad1): track 0.40 -> 63.0 mm
- net Net-(D47-Pad1): track 0.00 -> 62.0 mm
- net /a6: track 61.4 -> 0.00 mm
- net /a2: track 61.4 -> 0.00 mm
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
Commit message: Steuerwerk weitergemacht
Parts:
- removed J5: 2PinTerminalBlocktg, 2PinTerminalBlocktg
- added C7: 100n, Capacitor_THT:C_Disc_D10.0mm_W2.5mm_P5.00mm, F.Cu at (79.4, 130.8)
- added C8: 100n, Capacitor_THT:C_Disc_D10.0mm_W2.5mm_P5.00mm, F.Cu at (111.2, 154.9)
- C1, C2, C3, C4, C5, C6: footprint Capacitors_ThroughHole:C_Disc_D10.0mm_W2.5mm_P5.00mm -> Capacitor_THT:C_Disc_D10.0mm_W2.5mm_P5.00mm
- J1: value 2PinTerminalBlocktg -> Conn_01x04; footprint 2PinTerminalBlocktg -> Connector_Molex:Molex_KK-254_AE-6410-04A_1x04_P2.54mm_Vertical
- J2: value 2PinTerminalBlocktg -> Conn_01x03; footprint 2PinTerminalBlocktg -> Connector_Molex:Molex_KK-254_AE-6410-03A_1x03_P2.54mm_Vertical
- J3: value 3PinTerminalBlocktg -> Conn_01x03; footprint 3PinTerminalBlocktg -> Connector_Molex:Molex_KK-254_AE-6410-03A_1x03_P2.54mm_Vertical
- J4: value 3PinTerminalBlocktg -> Conn_01x02; footprint 3PinTerminalBlocktg -> Connector_Molex:Molex_KK-254_AE-6410-02A_1x02_P2.54mm_Vertical
- moved J4 122.0 mm to (51.5, 40.0), turned to 0 degrees
- moved J2 94.7 mm to (51.5, 97.8), turned to 90 degrees
- moved C6 70.3 mm to (75.6, 60.9), turned to 180 degrees
- moved J3 69.1 mm to (48.9, 164.4)
- moved C3 22.9 mm to (48.9, 116.8), turned to 270 degrees
- moved J7 21.6 mm to (103.5, 188.6), turned to 180 degrees
- moved C5 21.0 mm to (79.4, 154.9)
- moved J9 19.7 mm to (126.4, 187.9), turned to 180 degrees
- moved C2 19.4 mm to (47.7, 55.8)
- moved J8 15.2 mm to (111.2, 187.9), turned to 180 degrees
- moved C1 14.1 mm to (75.6, 87.6)
- moved U5 11.9 mm to (69.3, 91.4)
- moved U6 11.5 mm to (137.8, 148.6)
- moved U4 11.1 mm to (69.3, 64.7)
- moved J6 10.8 mm to (84.5, 187.9), turned to 180 degrees
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Connections:
- J2 pad 1: Net-(J2-Pad1) -> /enSTW
- J2 pad 2: Net-(J2-Pad2) -> /enDEC
- J3 pad 1: /enSTW -> /loadIR
- J3 pad 2: /enDEC -> /enAkku
- J3 pad 3: /Takt -> /clrMPC
- J4 pad 1: /loadIR -> GND
- J4 pad 2: /enAkku -> VCC
- J7 pad 1: Net-(J7-Pad1) -> /enAkku
- J7 pad 4: /enAkku -> Net-(J7-Pad4)
- J9 pad 1: /loadIR -> Net-(J9-Pad1)
- J9 pad 4: Net-(J9-Pad4) -> /loadIR
- U2 pad 3: Net-(J7-Pad3) -> Net-(J7-Pad2)
- U2 pad 4: Net-(J7-Pad2) -> Net-(J7-Pad3)
- U2 pad 5: Net-(J7-Pad1) -> Net-(J7-Pad4)
- U2 pad 6: Net-(J6-Pad2) -> Net-(J6-Pad1)
- U2 pad 7: Net-(J6-Pad1) -> Net-(J6-Pad2)
- U3 pad 3: Net-(J2-Pad1) -> Net-(J1-Pad4)
- U3 pad 4: Net-(J2-Pad2) -> Net-(J1-Pad3)
- U3 pad 5: Net-(J1-Pad1) -> Net-(J1-Pad2)
- U3 pad 6: Net-(J1-Pad2) -> Net-(J1-Pad1)
- U6 pad 4: Net-(J9-Pad4) -> Net-(J9-Pad1)
- U6 pad 5: Net-(J9-Pad3) -> Net-(J9-Pad2)
- U6 pad 6: Net-(J9-Pad2) -> Net-(J9-Pad3)
- U6 pad 8: Net-(J8-Pad2) -> Net-(J8-Pad1)
- U6 pad 9: Net-(J8-Pad1) -> Net-(J8-Pad2)
- U7 pad 12: Net-(J7-Pad3) -> Net-(J7-Pad2)
- U7 pad 15: Net-(J7-Pad1) -> Net-(J7-Pad4)
- U7 pad 16: Net-(J6-Pad1) -> Net-(J6-Pad2)
- U7 pad 5: Net-(J6-Pad2) -> Net-(J6-Pad1)
- U7 pad 6: Net-(J7-Pad2) -> Net-(J7-Pad3)
- U8 pad 15: Net-(J9-Pad3) -> Net-(J9-Pad2)
- U8 pad 19: Net-(J8-Pad1) -> Net-(J8-Pad2)
- U8 pad 2: Net-(J8-Pad2) -> Net-(J8-Pad1)
- U8 pad 5: Net-(J9-Pad2) -> Net-(J9-Pad3)
- U8 pad 6: Net-(J9-Pad4) -> Net-(J9-Pad1)
Routing:
- net VCC: track 639.1 -> 415.2 mm, vias 3 -> 0
- net GND: track 336.4 -> 468.5 mm, vias 4 -> 5
- net /clrMPC: track 118.5 -> 0.00 mm
- net /Takt: track 83.5 -> 0.00 mm
- net Net-(U3-Pad11): track 79.4 -> 0.00 mm, vias 4 -> 0
- net Net-(U3-Pad12): track 76.2 -> 0.00 mm, vias 3 -> 0
- net Net-(J2-Pad1): track 75.1 -> 0.00 mm
- net Net-(U3-Pad14): track 75.0 -> 0.00 mm
- net Net-(U3-Pad13): track 74.6 -> 0.00 mm, vias 3 -> 0
- net Net-(J2-Pad2): track 72.9 -> 0.00 mm
- net Net-(U5-Pad7): track 0.00 -> 69.1 mm
- net /enSTW: track 67.8 -> 0.00 mm, vias 3 -> 0
- net Net-(J1-Pad3): track 0.00 -> 59.8 mm
- net Net-(D23-Pad2): track 0.00 -> 59.4 mm
- net Net-(D21-Pad2): track 1.21 -> 58.8 mm
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Other:
- board text removed: "~enAkku"
- board text removed: "~enCU"
- board text removed: "~loadIR"

Commit message: Steuerwerk fertig außer Diodenmatrix
Parts:
- added C9: 100u, Capacitor_THT:CP_Radial_D8.0mm_P2.50mm, F.Cu at (62.3, 37.4)
- D1, D10, D13, D4, D6, D8: footprint LEDs:LED_D3.0mm -> LED_THT:LED_D3.0mm
- D11, D12, D14, D15, D16, D2, D22, D29, D3, D32, D34, D36, D41, D5, D7, D9: footprint LEDs:LED_D1.8mm_W1.8mm_H2.4mm_Horizontal_O1.27mm_Z1.6mm -> LED_THT:LED_D3.0mm
- R1, R10, R12, R4, R6, R8: value R -> 330
- R16: value R -> 1k
- moved D17 224.8 mm to (254.7, 71.6)
- moved D19 224.8 mm to (254.9, 79.5)
- moved D21 224.8 mm to (253.4, 64.7)
- moved D23 224.8 mm to (250.4, 58.6)
- moved D27 224.8 mm to (164.5, 100.8)
- moved D31 224.8 mm to (167.9, 96.7)
- moved D35 224.8 mm to (179.2, 91.1)
- moved D37 224.8 mm to (175.6, 79.2)
- moved D39 224.8 mm to (175.2, 83.0)
- moved D46 224.8 mm to (241.3, 50.8)
- moved D52 224.8 mm to (202.2, 90.1)
- moved D53 224.8 mm to (194.5, 93.7)
- moved D58 224.8 mm to (203.1, 101.3)
- moved D60 224.8 mm to (209.2, 98.3)
- moved D63 224.8 mm to (189.9, 93.7)
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Connections:
- net Net-(D17-Pad1) renamed /v0
- net Net-(D17-Pad2) renamed /h3
- net Net-(D18-Pad2) renamed /h10
- net Net-(D19-Pad2) renamed /h11
- net Net-(D20-Pad2) renamed /h14
- net Net-(D21-Pad2) renamed /h2
- net Net-(D23-Pad1) renamed /v2
- net Net-(D23-Pad2) renamed /h1
- net Net-(D25-Pad2) renamed /h4
- net Net-(D26-Pad2) renamed /h8
- net Net-(D27-Pad2) renamed /h13
- net Net-(D30-Pad1) renamed /v3
- net Net-(D30-Pad2) renamed /h6
- net Net-(D33-Pad1) renamed /v4
- net Net-(D33-Pad2) renamed /h5
- net Net-(D35-Pad1) renamed /v5
- net Net-(D35-Pad2) renamed /h9
- net Net-(D37-Pad1) renamed /v6
- net Net-(D39-Pad1) renamed /v7
- net Net-(D42-Pad1) renamed /v8
- net Net-(D43-Pad1) renamed /v9
- net Net-(D43-Pad2) renamed /h0
- net Net-(D46-Pad1) renamed /v10
- net Net-(D47-Pad1) renamed /v11
- net Net-(D51-Pad2) renamed /h7
- net Net-(D56-Pad2) renamed /h12
- net Net-(D59-Pad1) renamed /v12
- net Net-(D61-Pad1) renamed /v13
- net Net-(RP1-Pad8) renamed /v14
- net Net-(RP1-Pad9) renamed /v15
- net Net-(U5-Pad7) renamed /h15
- D21 pad 1: Net-(D21-Pad1) -> /v1
- R16 pad 1: Net-(D21-Pad1) -> Net-(Q1-Pad1)
- R16 pad 2: Net-(Q1-Pad1) -> /v1
- RP2 pad 3: Net-(D21-Pad1) -> /v1
- U3 pad 9: Net-(D21-Pad1) -> /v1
- U7 pad 3: Net-(D21-Pad1) -> /v1
Routing:
- net VCC: track 415.2 -> 601.6 mm
- net /Takt: track 0.00 -> 171.2 mm
- net /enSTW: track 0.00 -> 157.6 mm
- net /loadIR: track 0.00 -> 148.6 mm
- net /clrMPC: track 0.00 -> 146.1 mm
- net /v1: track 0.00 -> 134.9 mm
- net /enAkku: track 0.00 -> 118.2 mm
- net /v15: track 0.00 -> 90.4 mm
- net /v14: track 0.00 -> 79.9 mm
- net Net-(U3-Pad11): track 0.00 -> 75.6 mm, vias 0 -> 1
- net Net-(J6-Pad2): track 0.00 -> 73.5 mm
- net Net-(U3-Pad12): track 0.00 -> 73.1 mm, vias 0 -> 1
- net Net-(U3-Pad13): track 0.00 -> 70.1 mm, vias 0 -> 1
- net Net-(U3-Pad14): track 0.00 -> 69.4 mm
- net Net-(J8-Pad2): track 0.00 -> 69.3 mm
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
Commit message: Steuerwerk fast fertig TODO: Beschriftung überarbeiten
Parts:
- removed the D47 at (186.1, 38.1)
- added D11: Led_Small, bonsai:LED_Diodenmatrix, F.Cu at (123.2, 68.0)
- D10: renamed from D17; footprint LED_THT:LED_D3.0mm -> bonsai:LED_Diodenmatrix
- D12: renamed from D25; footprint LED_THT:LED_D3.0mm -> bonsai:LED_Diodenmatrix
- D13: renamed from D37; footprint LED_THT:LED_D3.0mm -> bonsai:LED_Diodenmatrix
- D14: renamed from D48; footprint LED_THT:LED_D1.8mm_W3.3mm_H2.4mm -> bonsai:LED_Diodenmatrix
- D15: renamed from D33; footprint LED_THT:LED_D3.0mm -> bonsai:LED_Diodenmatrix
- D16: renamed from D49; footprint LED_THT:LED_D1.8mm_W3.3mm_H2.4mm -> bonsai:LED_Diodenmatrix
- D17: renamed from D59; footprint LED_THT:LED_D1.8mm_W3.3mm_H2.4mm -> bonsai:LED_Diodenmatrix
- D18: renamed from D30; footprint LED_THT:LED_D3.0mm -> bonsai:LED_Diodenmatrix
- D19: renamed from D39; footprint LED_THT:LED_D3.0mm -> bonsai:LED_Diodenmatrix
- D20: renamed from D50; footprint LED_THT:LED_D1.8mm_W3.3mm_H2.4mm -> bonsai:LED_Diodenmatrix
- D21: renamed from D51; footprint LED_THT:LED_D1.8mm_W3.3mm_H2.4mm -> bonsai:LED_Diodenmatrix
- D22: renamed from D26; footprint LED_THT:LED_D3.0mm -> bonsai:LED_Diodenmatrix
- D23: renamed from D38; footprint LED_THT:LED_D3.0mm -> bonsai:LED_Diodenmatrix
- D24: renamed from D52; footprint LED_THT:LED_D1.8mm_W3.3mm_H2.4mm -> bonsai:LED_Diodenmatrix
- D25: renamed from D35; footprint LED_THT:LED_D3.0mm -> bonsai:LED_Diodenmatrix
- D26: renamed from D53; footprint LED_THT:LED_D1.8mm_W3.3mm_H2.4mm -> bonsai:LED_Diodenmatrix
- D27: renamed from D63; footprint tg_foodprint:LED_D1.8mm_W3.3mm_H2.4mmBonsai -> bonsai:LED_Diodenmatrix
- D28: renamed from D18; footprint LED_THT:LED_D3.0mm -> bonsai:LED_Diodenmatrix
- D29: renamed from D31; footprint LED_THT:LED_D3.0mm -> bonsai:LED_Diodenmatrix
- D3: renamed from D23; footprint LED_THT:LED_D3.0mm -> bonsai:LED_Diodenmatrix
- D30: renamed from D40; footprint LED_THT:LED_D3.0mm -> bonsai:LED_Diodenmatrix
- D31: renamed from D54; footprint LED_THT:LED_D1.8mm_W3.3mm_H2.4mm -> bonsai:LED_Diodenmatrix
- D32: renamed from D19; footprint LED_THT:LED_D3.0mm -> bonsai:LED_Diodenmatrix
- D33: renamed from D42; footprint LED_THT:LED_D1.8mm_W3.3mm_H2.4mm -> bonsai:LED_Diodenmatrix
- D34: renamed from D55; footprint LED_THT:LED_D1.8mm_W3.3mm_H2.4mm -> bonsai:LED_Diodenmatrix
- D35: renamed from D56; footprint LED_THT:LED_D1.8mm_W3.3mm_H2.4mm -> bonsai:LED_Diodenmatrix
- D36: renamed from D60; footprint LED_THT:LED_D1.8mm_W3.3mm_H2.4mm -> bonsai:LED_Diodenmatrix
- D37: renamed from D27; footprint LED_THT:LED_D3.0mm -> bonsai:LED_Diodenmatrix
- D38: renamed from D57; footprint LED_THT:LED_D1.8mm_W3.3mm_H2.4mm -> bonsai:LED_Diodenmatrix
- D39: renamed from D20; footprint LED_THT:LED_D3.0mm -> bonsai:LED_Diodenmatrix
- D4: renamed from D43; footprint LED_THT:LED_D1.8mm_W3.3mm_H2.4mm -> bonsai:LED_Diodenmatrix
- D40: renamed from D28; footprint LED_THT:LED_D3.0mm -> bonsai:LED_Diodenmatrix
- D41: renamed from D58; footprint LED_THT:LED_D1.8mm_W3.3mm_H2.4mm -> bonsai:LED_Diodenmatrix
- D42: renamed from D61; footprint LED_THT:LED_D1.8mm_W3.3mm_H2.4mm -> bonsai:LED_Diodenmatrix
- D5: renamed from D44; footprint LED_THT:LED_D1.8mm_W3.3mm_H2.4mm -> bonsai:LED_Diodenmatrix
- D6: renamed from D46; footprint LED_THT:LED_D1.8mm_W3.3mm_H2.4mm -> bonsai:LED_Diodenmatrix
- D7: renamed from D21; footprint LED_THT:LED_D3.0mm -> bonsai:LED_Diodenmatrix
- D8: renamed from D24; footprint LED_THT:LED_D3.0mm -> bonsai:LED_Diodenmatrix
- D9: renamed from D45; footprint LED_THT:LED_D1.8mm_W3.3mm_H2.4mm -> bonsai:LED_Diodenmatrix
- moved D32 174.5 mm to (81.4, 98.5), turned to 225 degrees
- moved D10 173.4 mm to (81.3, 68.0), turned to 225 degrees
- moved D39 173.2 mm to (81.3, 109.9), turned to 225 degrees
- moved D28 171.7 mm to (81.3, 94.6), turned to 225 degrees
- moved D7 168.3 mm to (85.1, 64.2), turned to 225 degrees
- moved D3 161.4 mm to (88.9, 60.4), turned to 225 degrees
- moved D9 130.2 mm to (115.6, 64.2), turned to 225 degrees
- moved D6 122.3 mm to (119.4, 60.4), turned to 225 degrees
- moved D17 85.5 mm to (127.1, 75.6), turned to 225 degrees
- moved D40 82.7 mm to (89.0, 109.9), turned to 225 degrees
- moved D36 82.3 mm to (127.0, 102.3), turned to 225 degrees
- moved D42 81.9 mm to (130.8, 109.9), turned to 225 degrees
- moved D4 81.7 mm to (115.6, 56.6), turned to 225 degrees
- moved D34 80.4 mm to (123.2, 98.5), turned to 225 degrees
- moved D41 80.3 mm to (123.2, 109.9), turned to 225 degrees
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- renumbered C9 to C1, C1 to C2, C2 to C3, C3 to C4, C4 to C5, C5 to C6, C6 to C7, C7 to C8, C8 to C9, D13 to D1, D62 to D2, D4 to D43, D6 to D44, D8 to D45, D10 to D46, D1 to D47, D2 to D48, D3 to D49, D5 to D50, D7 to D51, D9 to D52, D11 to D53, D12 to D54, D14 to D55, D15 to D56, D16 to D57, D22 to D58, D29 to D59, D32 to D60, D34 to D61, D36 to D62, D41 to D63, J4 to J2, J2 to J3, J3 to J4, J6 to J5, J7 to J6, J8 to J7, J9 to J8, R12 to R1, R5 to R10, R7 to R11, R9 to R12, R11 to R13, R13 to R14, R14 to R15, R15 to R16, R19 to R18, R21 to R19, R16 to R2, R24 to R20, R26 to R21, R28 to R22, R30 to R23, R4 to R3, R6 to R4, R8 to R5, R10 to R6, R1 to R7, R2 to R8, R3 to R9, RP2 to RP1, RP1 to RP2, U3 to U1, U4 to U2, U5 to U3, U9 to U4, U7 to U5, U8 to U6, U2 to U7, U6 to U8
Routing:
- net Net-(D58-Pad2): track 0.00 -> 2.54 mm
