File: Steuerwerk.sch (KiCad schematic (older format))
At the start: 115 parts, among them J1 2PinTerminalBlocktg, J10 2PinTerminalBlocktg, J11 2PinTerminalBlocktg, J12 2PinTerminalBlocktg, J2 2PinTerminalBlocktg, J3 3PinTerminalBlocktg, J4 3PinTerminalBlocktg, J5 2PinTerminalBlocktg, J6 2PinTerminalBlocktg, J7 2PinTerminalBlocktg, J8 2PinTerminalBlocktg, J9 2PinTerminalBlocktg, Q1 Q_PNP_BCE, U2 74541, U3 74LS161, U4 74LS138, U5 74LS138, U6 74541, U7 74LS374, U8 74LS374, U9 74ls240

Commit message: redesign Steuerwerk angefangen
Parts:
- removed J10, J11, J12, J6, J7, J8, J9: 2PinTerminalBlocktg, 2PinTerminalBlocktg, symbol allBonsaiSymbolLibs:2PinTerminalBlocktg-2PinTerminalBlocktg
- added U? (x6): 74240, symbol Bonsai:74240
- D17, D18, D19, D20, D21, D23, D24, D25, D26, D27, D28, D30, D31, D33, D35, D37, D38, D39, D40: footprint tg_foodprint:LED_D1.8mm_W3.3mm_H2.4mmBonsai -> LED_THT:LED_D3.0mm
- D42, D43, D44, D45, D46, D47, D48, D49, D50, D51, D52, D53, D54, D55, D56, D57, D58, D59, D60, D61: footprint tg_foodprint:LED_D1.8mm_W3.3mm_H2.4mmBonsai -> LED_THT:LED_D1.8mm_W3.3mm_H2.4mm
- U9: footprint (none) -> Package_DIP:DIP-20_W7.62mm_Socket_LongPads
Connections:
- wire segments 422 -> 417

Commit message: vor Umbau 74541 im Schaltplan
Parts:
- removed U9: 74ls240, Package_DIP:DIP-20_W7.62mm_Socket_LongPads, symbol allBonsaiSymbolLibs:74ls240
- U9: renamed from U?; footprint (none) -> Package_DIP:DIP-20_W7.62mm_Socket_LongPads
Connections:
- wire segments 417 -> 413
Changed lines of the file:
@@
-$EndComp
-$Comp
-L allBonsaiSymbolLibs:R-device R1
-U 1 1 58103C09
-P 600 6400
-F 0 "R1" V 680 6400 50  0000 C CNN
-F 1 "R" V 600 6400 50  0000 C CNN
-F 2 "Resistors_ThroughHole:R_Axial_DIN0207_L6.3mm_D2.5mm_P10.16mm_Horizontal" V 530 6400 50  0001 C CNN
-F 3 "" H 600 6400 50  0000 C CNN
-	1    600  6400
-	-1   0    0    1
 $EndComp
 $Comp
 L allBonsaiSymbolLibs:LED_Small-device D1
 U 1 1 58103D59
-P 600 6050
-F 0 "D1" V 554 6128 50  0000 L CNN
-F 1 "LED" V 645 6128 50  0000 L CNN
-F 2 "LEDs:LED_D3.0mm" H 600 6050 50  0001 C CNN
-F 3 "" H 600 6050 50  0000 C CNN
-	1    600  6050
-	0    1    1    0
+P 900 6300
+F 0 "D1" V 854 6378 50  0000 L CNN
+F 1 "LED" V 945 6378 50  0000 L CNN
+F 2 "LEDs:LED_D3.0mm" H 900 6300 50  0001 C CNN
+F 3 "" H 900 6300 50  0000 C CNN
+	1    900  6300
+	0    -1   -1   0
 $EndComp
 $Comp
 L power:GND #PWR01
 U 1 1 5810923B
-P 600 5850
-F 0 "#PWR01" H 600 5600 50  0001 C CNN
-F 1 "GND" H 600 5700 50  0000 C CNN
-F 2 "" H 600 5850 50  0000 C CNN
-F 3 "" H 600 5850 50  0000 C CNN
-	1    600  5850
-	-1   0    0    1
+P 900 6400
+F 0 "#PWR01" H 900 6150 50  0001 C CNN
+F 1 "GND" H 900 6250 50  0000 C CNN
+F 2 "" H 900 6400 50  0000 C CNN
+F 3 "" H 900 6400 50  0000 C CNN
+	1    900  6400
+	1    0    0    -1
 $EndComp
 Text Label 6650 7500 0    60   ~ 0
@@
 	3250 900  3400 900
 Wire Wire Line
-	600  6250 600  6150
-Wire Wire Line
-	600  5950 600  5850
-Wire Wire Line
 	4000 600  3950 600
 Wire Wire Line
@@
 Wire Wire Line
 	850  7100 1850 7100
-Wire Wire Line
-	600  6550 900  6550
 Wire Wire Line
 	2100 5350 2100 5850
@@
 Text Label 850  6700 0    60   ~ 0
 clrMPC
-$Comp
-L allBonsaiSymbolLibs:74ls240 U9
-U 1 1 5C91C679
-P -1650 5950
-F 0 "U9" H -1650 6425 50  0000 C CNN
-F 1 "74ls240" H -1650 6334 50  0000 C CNN
-F 2 "Package_DIP:DIP-20_W7.62mm_Socket_LongPads" H -1650 5950 50  0001 C CNN
-F 3 "" H -1650 5950 50  0001 C CNN
-	1    -1650 5950
-	0    1    1    0
-$EndComp
-Wire Wire Line
-	900  6550 900  5900
 Wire Wire Line
 	2500 6700 2550 6700
@@
 Wire Wire Line
 	900  5250 1500 5250
-$Comp
-L Bonsai:74240 U?
+Wire Wire Line
+	3100 3200 3100 3350
+Wire Wire Line
+	3400 3350 3400 3200
+$Comp
+L power:VCC #PWR0106
+U 1 1 5FDB9685
+P 8700 5400
+F 0 "#PWR0106" H 8700 5250 50  0001 C CNN
+F 1 "VCC" H 8717 5573 50  0000 C CNN
+F 2 "" H 8700 5400 50  0001 C CNN
+F 3 "" H 8700 5400 50  0001 C CNN
+	1    8700 5400
+	1    0    0    -1
+$EndComp
+$Comp
+L power:GND #PWR0107
+U 1 1 5FDB9DFF
+P 8700 6200
+F 0 "#PWR0107" H 8700 5950 50  0001 C CNN
+F 1 "GND" H 8705 6027 50  0000 C CNN
+F 2 "" H 8700 6200 50  0001 C CNN
+F 3 "" H 8700 6200 50  0001 C CNN
+	1    8700 6200
+	1    0    0    -1
+$EndComp
+$Comp
+L power:GND #PWR0108
+U 1 1 5FDBB4CB
+P 8150 6200
+F 0 "#PWR0108" H 8150 5950 50  0001 C CNN
+F 1 "GND" H 8155 6027 50  0000 C CNN
+F 2 "" H 8150 6200 50  0001 C CNN
+F 3 "" H 8150 6200 50  0001 C CNN
+	1    8150 6200
+	1    0    0    -1
+$EndComp
+Wire Wire Line
+	8150 6200 8150 5750
+Connection ~ 8150 5750
+Wire Wire Line
+	8150 5750 8150 5650
+$Comp
+L Bonsai:74240 U9
+U 1 1 5FC0A796
+P 900 5550
+F 0 "U9" V 750 5550 50  0000 L CNN
+F 1 "74240" V 900 5650 50  0000 L CNN
+F 2 "Package_DIP:DIP-20_W7.62mm_Socket_LongPads" H 1050 5450 50  0001 C CNN
+F 3 "" H 1050 5450 50  0001 C CNN
+	1    900  5550
+	0    1    1    0
+$EndComp
+$Comp
+L Bonsai:74240 U9
+U 9 1 5FDB5555
+P 8500 5900
+F 0 "U9" H 8778 6046 50  0000 L CNN
+F 1 "74240" H 8778 5955 50  0000 L CNN
+F 2 "Package_DIP:DIP-20_W7.62mm_Socket_LongPads" H 8650 5800 50  0001 C CNN
+F 3 "" H 8650 5800 50  0001 C CNN
+	9    8500 5900
+	1    0    0    -1
+$EndComp
+$Comp
+L Bonsai:74240 U9
+U 5 1 5FD4D2EC
+P 3400 3650
+F 0 "U9" V 3250 3700 50  0000 L CNN
+F 1 "74240" V 3400 3750 50  0000 L CNN
+F 2 "Package_DIP:DIP-20_W7.62mm_Socket_LongPads" H 3550 3550 50  0001 C CNN
+F 3 "" H 3550 3550 50  0001 C CNN
+	5    3400 3650
+	0    1    1    0
+$EndComp
+$Comp
+L Bonsai:74240 U9
+U 7 1 5FCAADFB
+P 2800 3650
+F 0 "U9" V 2650 3650 50  0000 L CNN
+F 1 "74240" V 2870 3778 50  0001 L CNN
+F 2 "Package_DIP:DIP-20_W7.62mm_Socket_LongPads" H 2950 3550 50  0001 C CNN
+F 3 "" H 2950 3550 50  0001 C CNN
+	7    2800 3650
+	0    1    1    0
+$EndComp
+$Comp
+L Bonsai:74240 U9
 U 8 1 5FC75D3B
 P 2500 3650
-F 0 "U?" V 2479 3778 50  0000 L CNN
-F 1 "74240" V 2570 3778 50  0000 L CNN
-F 2 "" H 2650 3550 50  0001 C CNN
+F 0 "U9" V 2350 3650 50  0000 L CNN
+F 1 "74240" V 2570 3778 50  0001 L CNN
+F 2 "Package_DIP:DIP-20_W7.62mm_Socket_LongPads" H 2650 3550 50  0001 C CNN
 F 3 "" H 2650 3550 50  0001 C CNN
 	8    2500 3650
@@
 $EndComp
 $Comp
-L Bonsai:74240 U?
-U 7 1 5FCAADFB
-P 2800 3650
-F 0 "U?" V 2779 3778 50  0000 L CNN
-F 1 "74240" V 2870 3778 50  0000 L CNN
-F 2 "" H 2950 3550 50  0001 C CNN
-F 3 "" H 2950 3550 50  0001 C CNN
-	7    2800 3650
-	0    1    1    0
-$EndComp
-$Comp
-L Bonsai:74240 U?
+L Bonsai:74240 U9
 U 6 1 5FCDFED6
 P 3100 3650
-F 0 "U?" V 3079 3778 50  0000 L CNN
-F 1 "74240" V 3170 3778 50  0000 L CNN
-F 2 "" H 3250 3550 50  0001 C CNN
+F 0 "U9" V 2950 3700 50  0000 L CNN
+F 1 "74240" V 3170 3778 50  0001 L CNN
+F 2 "Package_DIP:DIP-20_W7.62mm_Socket_LongPads" H 3250 3550 50  0001 C CNN
 F 3 "" H 3250 3550 50  0001 C CNN
 	6    3100 3650
 	0    1    1    0
 $EndComp
-Wire Wire Line
-	3100 3200 3100 3350
-$Comp
-L Bonsai:74240 U?
-U 5 1 5FD4D2EC
-P 3400 3650
-F 0 "U?" V 3379 3778 50  0000 L CNN
-F 1 "74240" V 3470 3778 50  0000 L CNN
-F 2 "" H 3550 3550 50  0001 C CNN
-F 3 "" H 3550 3550 50  0001 C CNN
-	5    3400 3650
-	0    1    1    0
-$EndComp
-Wire Wire Line
-	3400 3350 3400 3200
-$Comp
-L Bonsai:74240 U?
-U 9 1 5FDB5555
-P -650 5450
-F 0 "U?" H -372 5596 50  0000 L CNN
-F 1 "74240" H -372 5505 50  0000 L CNN
-F 2 "" H -500 5350 50  0001 C CNN
-F 3 "" H -500 5350 50  0001 C CNN
-	9    -650 5450
-	1    0    0    -1
-$EndComp
-$Comp
-L power:VCC #PWR?
-U 1 1 5FDB9685
-P -450 4950
-F 0 "#PWR?" H -450 4800 50  0001 C CNN
-F 1 "VCC" H -433 5123 50  0000 C CNN
-F 2 "" H -450 4950 50  0001 C CNN
-F 3 "" H -450 4950 50  0001 C CNN
-	1    -450 4950
-	1    0    0    -1
-$EndComp
-$Comp
-L power:GND #PWR?
-U 1 1 5FDB9DFF
-P -450 5750
-F 0 "#PWR?" H -450 5500 50  0001 C CNN
-F 1 "GND" H -445 5577 50  0000 C CNN
-F 2 "" H -450 5750 50  0001 C CNN
-F 3 "" H -450 5750 50  0001 C CNN
-	1    -450 5750
-	1    0    0    -1
-$EndComp
-$Comp
-L power:GND #PWR?
-U 1 1 5FDBB4CB
-P -1000 5750
-F 0 "#PWR?" H -1000 5500 50  0001 C CNN
-F 1 "GND" H -995 5577 50  0000 C CNN
-F 2 "" H -1000 5750 50  0001 C CNN
-F 3 "" H -1000 5750 50  0001 C CNN
-	1    -1000 5750
-	1    0    0    -1
-$EndComp
-Wire Wire Line
-	-1000 5750 -1000 5300
-Connection ~ -1000 5300
-Wire Wire Line
-	-1000 5300 -1000 5200
+$Comp
+L allBonsaiSymbolLibs:R-device R1
+U 1 1 58103C09
+P 900 6050
+F 0 "R1" V 980 6050 50  0000 C CNN
+F 1 "R" V 900 6050 50  0000 C CNN
+F 2 "Resistors_ThroughHole:R_Axial_DIN0207_L6.3mm_D2.5mm_P10.16mm_Horizontal" V 830 6050 50  0001 C CNN
+F 3 "" H 900 6050 50  0000 C CNN
+	1    900  6050
+	1    0    0    -1
+$EndComp
 Wire Bus Line
 	4850 900  6600 900
 Wire Bus Line
 	6950 900  8700 900
-$Comp
-L allBonsaiSymbolLibs:74ls240 U9
-U 5 1 5CA9B1C1
-P 700 4000
-F 0 "U9" V 654 4338 50  0000 L CNN
-F 1 "74ls240" V 745 4338 50  0000 L CNN
-F 2 "Package_DIP:DIP-20_W7.62mm_Socket_LongPads" H 700 4000 50  0001 C CNN
-F 3 "" H 700 4000 50  0001 C CNN
-	5    700  4000
-	0    1    1    0
-$EndComp
-$Comp
-L allBonsaiSymbolLibs:74ls240 U9
-U 8 1 5CCD7140
-P -2200 4000
-F 0 "U9" V -2246 4338 50  0000 L CNN
-F 1 "74ls240" V -2155 4338 50  0000 L CNN
-F 2 "Package_DIP:DIP-20_W7.62mm_Socket_LongPads" H -2200 4000 50  0001 C CNN
-F 3 "" H -2200 4000 50  0001 C CNN
-	8    -2200 4000
-	0    1    1    0
-$EndComp
-$Comp
-L allBonsaiSymbolLibs:74ls240 U9
-U 7 1 5CCD50DA
-P -1200 4000
-F 0 "U9" V -1246 4338 50  0000 L CNN
-F 1 "74ls240" V -1155 4338 50  0000 L CNN
-F 2 "Package_DIP:DIP-20_W7.62mm_Socket_LongPads" H -1200 4000 50  0001 C CNN
-F 3 "" H -1200 4000 50  0001 C CNN
-	7    -1200 4000
-	0    1    1    0
-$EndComp
-$Comp
-L allBonsaiSymbolLibs:74ls240 U9
-U 6 1 5CCD3F05
-P -300 4000
-F 0 "U9" V -346 4338 50  0000 L CNN
-F 1 "74ls240" V -255 4338 50  0000 L CNN
-F 2 "Package_DIP:DIP-20_W7.62mm_Socket_LongPads" H -300 4000 50  0001 C CNN
-F 3 "" H -300 4000 50  0001 C CNN
-	6    -300 4000
-	0    1    1    0
-$EndComp
-$Comp
-L Bonsai:74240 U?
-U 1 1 5FC0A796
-P 900 5550
-F 0 "U?" V 879 5678 50  0000 L CNN
-F 1 "74240" V 970 5678 50  0000 L CNN
-F 2 "" H 1050 5450 50  0001 C CNN
-F 3 "" H 1050 5450 50  0001 C CNN
-	1    900  5550
-	0    1    1    0
-$EndComp
 $EndSCHEMATC

Commit message: Steuerwerk: beide 74541 umgebaut
Parts:
- removed U2, U6: 74541, Housings_DIP:DIP-20_W7.62mm_Socket_LongPads, symbol allBonsaiSymbolLibs:74541
- added U2, U6: 74541, Package_DIP:DIP-20_W7.62mm_Socket_LongPads, symbol Bonsai:74541
Connections:
- wire segments 413 -> 411

Commit message: Steuerwerk vor Entfernen der Busse
Connections:
- wire segments 411 -> 429
- no-connect marks 2 -> 1

Commit message: weitergemacht
Parts:
- added J6, J8: Conn_01x02, Connector_Molex:Molex_KK-254_AE-6410-02A_1x02_P2.54mm_Vertical, symbol Connector_Generic:Conn_01x02
- added J7, J9: Conn_01x04, Connector_Molex:Molex_KK-254_AE-6410-04A_1x04_P2.54mm_Vertical, symbol Connector_Generic:Conn_01x04
- R11, R13, R14, R15, R17, R19, R2, R21, R24, R26, R28, R3, R30, R5, R7, R9: value R -> 330
Connections:
- net labels removed: 1, 10, 11, 12, 13, 14, 15, 16, 2, 3, 4, 5, 6, 7, 8, 9, a1, a2, a3, a4, a5, a6, a7, a8, b1, b2, b3, b4, b5, b6, b7, b8
- wire segments 429 -> 436

Commit message: Steuerwerk weitergemacht
Parts:
- removed J1, J2, J5: 2PinTerminalBlocktg, 2PinTerminalBlocktg, symbol allBonsaiSymbolLibs:2PinTerminalBlocktg-2PinTerminalBlocktg
- removed J3, J4: 3PinTerminalBlocktg, 3PinTerminalBlocktg, symbol allBonsaiSymbolLibs:3PinTerminalBlocktg-3PinTerminalBlocktg
- added C7, C8: 100n, Capacitor_THT:C_Disc_D10.0mm_W2.5mm_P5.00mm, symbol allBonsaiSymbolLibs:C_Small
- added J1: Conn_01x04, Connector_Molex:Molex_KK-254_AE-6410-04A_1x04_P2.54mm_Vertical, symbol Connector_Generic:Conn_01x04
- added J2, J3: Conn_01x03, Connector_Molex:Molex_KK-254_AE-6410-03A_1x03_P2.54mm_Vertical, symbol Connector_Generic:Conn_01x03
- added J4: Conn_01x02, Connector_Molex:Molex_KK-254_AE-6410-02A_1x02_P2.54mm_Vertical, symbol Connector_Generic:Conn_01x02
- C1, C2, C3, C4, C5, C6: footprint Capacitors_ThroughHole:C_Disc_D10.0mm_W2.5mm_P5.00mm -> Capacitor_THT:C_Disc_D10.0mm_W2.5mm_P5.00mm
- R1, R10, R12, R4, R6, R8: value R -> 330
- R16: value R -> 1k
Connections:
- wire segments 436 -> 442
Other:
- note added: "Mikroprogrammzähler \nMPC"
- note added: "Steuersignale"
- note added: "vom Befehlesdecoder"
- note removed: "vom_Befehle-decoder"

Commit message: Steuerwerk fertig außer Diodenmatrix
Parts:
- added C9: 100u, Capacitor_THT:CP_Radial_D8.0mm_P2.50mm, symbol Device:CP
- D1, D10, D13, D4, D6, D8: footprint LEDs:LED_D3.0mm -> LED_THT:LED_D3.0mm
- D11, D12, D14, D15, D16, D2, D22, D29, D3, D32, D34, D36, D41, D5, D7, D9: footprint LEDs:LED_D1.8mm_W1.8mm_H2.4mm_Horizontal_O1.27mm_Z1.6mm -> LED_THT:LED_D3.0mm
Connections:
- net labels added: h0, h1, h10, h11, h12, h13, h14, h15, h2, h3, h4, h5, h6, h7, h8, h9, v0, v1, v10, v11, v12, v13, v14, v15, v2, v3, v4, v5, v6, v7, v8, v9
- wire segments 442 -> 446

Commit message: Steuerwerk fast fertig TODO: Beschriftung überarbeiten
Parts:
- D10: renamed from D17; footprint LED_THT:LED_D3.0mm -> bonsai:LED_Diodenmatrix
- D11: renamed from D47; footprint LED_THT:LED_D1.8mm_W3.3mm_H2.4mm -> bonsai:LED_Diodenmatrix
- D12: renamed from D25; footprint LED_THT:LED_D3.0mm -> bonsai:LED_Diodenmatrix
- D13: renamed from D37; footprint LED_THT:LED_D3.0mm -> bonsai:LED_Diodenmatrix
- D14: renamed from D48; footprint LED_THT:LED_D1.8mm_W3.3mm_H2.4mm -> bonsai:LED_Diodenmatrix
- D15: renamed from D33; footprint LED_THT:LED_D3.0mm -> bonsai:LED_Diodenmatrix
- D16: renamed from D49; footprint LED_THT:LED_D1.8mm_W3.3mm_H2.4mm -> bonsai:LED_Diodenmatrix
- D17: renamed from D59; footprint LED_THT:LED_D1.8mm_W3.3mm_H2.4mm -> bonsai:LED_Diodenmatrix
- D18: renamed from D30; footprint LED_THT:LED_D3.0mm -> bonsai:LED_Diodenmatrix
- D19: renamed from D39; footprint LED_THT:LED_D3.0mm -> bonsai:LED_Diodenmatrix
- D20: renamed from D50; footprint LED_THT:LED_D1.8mm_W3.3mm_H2.4mm -> bonsai:LED_Diodenmatrix
- D21: renamed from D51; footprint LED_THT:LED_D1.8mm_W3.3mm_H2.4mm -> bonsai:LED_Diodenmatrix
- D22: renamed from D26; footprint LED_THT:LED_D3.0mm -> bonsai:LED_Diodenmatrix
- D23: renamed from D38; footprint LED_THT:LED_D3.0mm -> bonsai:LED_Diodenmatrix
- D24: renamed from D52; footprint LED_THT:LED_D1.8mm_W3.3mm_H2.4mm -> bonsai:LED_Diodenmatrix
- D25: renamed from D35; footprint LED_THT:LED_D3.0mm -> bonsai:LED_Diodenmatrix
- D26: renamed from D53; footprint LED_THT:LED_D1.8mm_W3.3mm_H2.4mm -> bonsai:LED_Diodenmatrix
- D27: renamed from D63; footprint tg_foodprint:LED_D1.8mm_W3.3mm_H2.4mmBonsai -> bonsai:LED_Diodenmatrix
- D28: renamed from D18; footprint LED_THT:LED_D3.0mm -> bonsai:LED_Diodenmatrix
- D29: renamed from D31; footprint LED_THT:LED_D3.0mm -> bonsai:LED_Diodenmatrix
- D3: renamed from D23; footprint LED_THT:LED_D3.0mm -> bonsai:LED_Diodenmatrix
- D30: renamed from D40; footprint LED_THT:LED_D3.0mm -> bonsai:LED_Diodenmatrix
- D31: renamed from D54; footprint LED_THT:LED_D1.8mm_W3.3mm_H2.4mm -> bonsai:LED_Diodenmatrix
- D32: renamed from D19; footprint LED_THT:LED_D3.0mm -> bonsai:LED_Diodenmatrix
- D33: renamed from D42; footprint LED_THT:LED_D1.8mm_W3.3mm_H2.4mm -> bonsai:LED_Diodenmatrix
- D34: renamed from D55; footprint LED_THT:LED_D1.8mm_W3.3mm_H2.4mm -> bonsai:LED_Diodenmatrix
- D35: renamed from D56; footprint LED_THT:LED_D1.8mm_W3.3mm_H2.4mm -> bonsai:LED_Diodenmatrix
- D36: renamed from D60; footprint LED_THT:LED_D1.8mm_W3.3mm_H2.4mm -> bonsai:LED_Diodenmatrix
- D37: renamed from D27; footprint LED_THT:LED_D3.0mm -> bonsai:LED_Diodenmatrix
- D38: renamed from D57; footprint LED_THT:LED_D1.8mm_W3.3mm_H2.4mm -> bonsai:LED_Diodenmatrix
- D39: renamed from D20; footprint LED_THT:LED_D3.0mm -> bonsai:LED_Diodenmatrix
- D4: renamed from D43; footprint LED_THT:LED_D1.8mm_W3.3mm_H2.4mm -> bonsai:LED_Diodenmatrix
- D40: renamed from D28; footprint LED_THT:LED_D3.0mm -> bonsai:LED_Diodenmatrix
- D41: renamed from D58; footprint LED_THT:LED_D1.8mm_W3.3mm_H2.4mm -> bonsai:LED_Diodenmatrix
- D42: renamed from D61; footprint LED_THT:LED_D1.8mm_W3.3mm_H2.4mm -> bonsai:LED_Diodenmatrix
- D5: renamed from D44; footprint LED_THT:LED_D1.8mm_W3.3mm_H2.4mm -> bonsai:LED_Diodenmatrix
- D6: renamed from D46; footprint LED_THT:LED_D1.8mm_W3.3mm_H2.4mm -> bonsai:LED_Diodenmatrix
- D7: renamed from D21; footprint LED_THT:LED_D3.0mm -> bonsai:LED_Diodenmatrix
- D8: renamed from D24; footprint LED_THT:LED_D3.0mm -> bonsai:LED_Diodenmatrix
- D9: renamed from D45; footprint LED_THT:LED_D1.8mm_W3.3mm_H2.4mm -> bonsai:LED_Diodenmatrix
- renumbered C9 to C1, C1 to C2, C2 to C3, C3 to C4, C4 to C5, C5 to C6, C6 to C7, C7 to C8, C8 to C9, D13 to D1, D62 to D2, D4 to D43, D6 to D44, D8 to D45, D10 to D46, D1 to D47, D2 to D48, D3 to D49, D5 to D50, D7 to D51, D9 to D52, D11 to D53, D12 to D54, D14 to D55, D15 to D56, D16 to D57, D22 to D58, D29 to D59, D32 to D60, D34 to D61, D36 to D62, D41 to D63, J4 to J2, J2 to J3, J3 to J4, J6 to J5, J7 to J6, J8 to J7, J9 to J8, R12 to R1, R5 to R10, R7 to R11, R9 to R12, R11 to R13, R13 to R14, R14 to R15, R15 to R16, R19 to R18, R21 to R19, R16 to R2, R24 to R20, R26 to R21, R28 to R22, R30 to R23, R4 to R3, R6 to R4, R8 to R5, R10 to R6, R1 to R7, R2 to R8, R3 to R9, RP2 to RP1, RP1 to RP2, U3 to U1, U4 to U2, U5 to U3, U9 to U4, U7 to U5, U8 to U6, U2 to U7, U6 to U8
Connections:
- wire segments 446 -> 449
- no-connect marks 1 -> 2
