File: Steuerwerk.sch (KiCad schematic (older format))
At the start: 114 parts, among them J1 Conn_01x04, J2 Conn_01x02, J3 Conn_01x03, J4 Conn_01x03, J5 Conn_01x02, J6 Conn_01x04, J7 Conn_01x02, J8 Conn_01x04, Q1 Q_PNP_BCE, U1 74LS161, U2 74LS138, U3 74LS138, U4 74240, U5 74LS374, U6 74LS374, U7 74541, U8 74541

Commit message: Steuerwerk: - Sperrbereiche für die Köpfe der Befestigungsschrauben hinzugefügt - Beschriftung (Silkscreen) auf der Platinenoberseite bearbeitet
Parts:
- R1, R10, R11, R12, R13, R14, R15, R16, R17, R18, R19, R2, R20, R21, R22, R23, R3, R4, R5, R6, R7, R8, R9: footprint Resistors_ThroughHole:R_Axial_DIN0207_L6.3mm_D2.5mm_P10.16mm_Horizontal -> Resistor_THT:R_Axial_DIN0207_L6.3mm_D2.5mm_P10.16mm_Horizontal
Changed lines of the file:
@@
 F 0 "R3" H 3320 5146 50  0000 L CNN
 F 1 "330" H 3320 5055 50  0000 L CNN
-F 2 "Resistors_ThroughHole:R_Axial_DIN0207_L6.3mm_D2.5mm_P10.16mm_Horizontal" V 3180 5100 50  0001 C CNN
+F 2 "Resistor_THT:R_Axial_DIN0207_L6.3mm_D2.5mm_P10.16mm_Horizontal" V 3180 5100 50  0001 C CNN
 F 3 "" H 3250 5100 50  0000 C CNN
 	1    3250 5100
@@
 F 0 "R4" H 3620 5146 50  0000 L CNN
 F 1 "330" H 3620 5055 50  0000 L CNN
-F 2 "Resistors_ThroughHole:R_Axial_DIN0207_L6.3mm_D2.5mm_P10.16mm_Horizontal" V 3480 5100 50  0001 C CNN
+F 2 "Resistor_THT:R_Axial_DIN0207_L6.3mm_D2.5mm_P10.16mm_Horizontal" V 3480 5100 50  0001 C CNN
 F 3 "" H 3550 5100 50  0000 C CNN
 	1    3550 5100
@@
 F 0 "R5" H 3920 5146 50  0000 L CNN
 F 1 "330" H 3920 5055 50  0000 L CNN
-F 2 "Resistors_ThroughHole:R_Axial_DIN0207_L6.3mm_D2.5mm_P10.16mm_Horizontal" V 3780 5100 50  0001 C CNN
+F 2 "Resistor_THT:R_Axial_DIN0207_L6.3mm_D2.5mm_P10.16mm_Horizontal" V 3780 5100 50  0001 C CNN
 F 3 "" H 3850 5100 50  0000 C CNN
 	1    3850 5100
@@
 F 0 "R6" H 4220 5146 50  0000 L CNN
 F 1 "330" H 4220 5055 50  0000 L CNN
-F 2 "Resistors_ThroughHole:R_Axial_DIN0207_L6.3mm_D2.5mm_P10.16mm_Horizontal" V 4080 5100 50  0001 C CNN
+F 2 "Resistor_THT:R_Axial_DIN0207_L6.3mm_D2.5mm_P10.16mm_Horizontal" V 4080 5100 50  0001 C CNN
 F 3 "" H 4150 5100 50  0000 C CNN
 	1    4150 5100
@@
 F 0 "R8" H 2970 7996 50  0001 L CNN
 F 1 "330" H 2970 7905 50  0001 L CNN
-F 2 "Resistors_ThroughHole:R_Axial_DIN0207_L6.3mm_D2.5mm_P10.16mm_Horizontal" V 2830 7950 50  0001 C CNN
+F 2 "Resistor_THT:R_Axial_DIN0207_L6.3mm_D2.5mm_P10.16mm_Horizontal" V 2830 7950 50  0001 C CNN
 F 3 "" H 2900 7950 50  0000 C CNN
 	1    2900 7950
@@
 F 0 "R9" H 3270 7996 50  0001 L CNN
 F 1 "330" H 3270 7905 50  0001 L CNN
-F 2 "Resistors_ThroughHole:R_Axial_DIN0207_L6.3mm_D2.5mm_P10.16mm_Horizontal" V 3130 7950 50  0001 C CNN
+F 2 "Resistor_THT:R_Axial_DIN0207_L6.3mm_D2.5mm_P10.16mm_Horizontal" V 3130 7950 50  0001 C CNN
 F 3 "" H 3200 7950 50  0000 C CNN
 	1    3200 7950
@@
 F 0 "R10" H 3570 7996 50  0001 L CNN
 F 1 "330" H 3570 7905 50  0001 L CNN
-F 2 "Resistors_ThroughHole:R_Axial_DIN0207_L6.3mm_D2.5mm_P10.16mm_Horizontal" V 3430 7950 50  0001 C CNN
+F 2 "Resistor_THT:R_Axial_DIN0207_L6.3mm_D2.5mm_P10.16mm_Horizontal" V 3430 7950 50  0001 C CNN
 F 3 "" H 3500 7950 50  0000 C CNN
 	1    3500 7950
@@
 F 0 "R11" H 3870 7996 50  0001 L CNN
 F 1 "330" H 3870 7905 50  0001 L CNN
-F 2 "Resistors_ThroughHole:R_Axial_DIN0207_L6.3mm_D2.5mm_P10.16mm_Horizontal" V 3730 7950 50  0001 C CNN
+F 2 "Resistor_THT:R_Axial_DIN0207_L6.3mm_D2.5mm_P10.16mm_Horizontal" V 3730 7950 50  0001 C CNN
 F 3 "" H 3800 7950 50  0000 C CNN
 	1    3800 7950
@@
 F 0 "R12" H 4170 7996 50  0001 L CNN
 F 1 "330" H 4170 7905 50  0001 L CNN
-F 2 "Resistors_ThroughHole:R_Axial_DIN0207_L6.3mm_D2.5mm_P10.16mm_Horizontal" V 4030 7950 50  0001 C CNN
+F 2 "Resistor_THT:R_Axial_DIN0207_L6.3mm_D2.5mm_P10.16mm_Horizontal" V 4030 7950 50  0001 C CNN
 F 3 "" H 4100 7950 50  0000 C CNN
 	1    4100 7950
@@
 F 0 "R13" H 4470 7996 50  0001 L CNN
 F 1 "330" H 4470 7905 50  0001 L CNN
-F 2 "Resistors_ThroughHole:R_Axial_DIN0207_L6.3mm_D2.5mm_P10.16mm_Horizontal" V 4330 7950 50  0001 C CNN
+F 2 "Resistor_THT:R_Axial_DIN0207_L6.3mm_D2.5mm_P10.16mm_Horizontal" V 4330 7950 50  0001 C CNN
 F 3 "" H 4400 7950 50  0000 C CNN
 	1    4400 7950
@@
 F 0 "R14" H 4770 7996 50  0001 L CNN
 F 1 "330" H 4770 7905 50  0001 L CNN
-F 2 "Resistors_ThroughHole:R_Axial_DIN0207_L6.3mm_D2.5mm_P10.16mm_Horizontal" V 4630 7950 50  0001 C CNN
+F 2 "Resistor_THT:R_Axial_DIN0207_L6.3mm_D2.5mm_P10.16mm_Horizontal" V 4630 7950 50  0001 C CNN
 F 3 "" H 4700 7950 50  0000 C CNN
 	1    4700 7950
@@
 F 0 "R15" H 5070 7996 50  0001 L CNN
 F 1 "330" H 5070 7905 50  0001 L CNN
-F 2 "Resistors_ThroughHole:R_Axial_DIN0207_L6.3mm_D2.5mm_P10.16mm_Horizontal" V 4930 7950 50  0001 C CNN
+F 2 "Resistor_THT:R_Axial_DIN0207_L6.3mm_D2.5mm_P10.16mm_Horizontal" V 4930 7950 50  0001 C CNN
 F 3 "" H 5000 7950 50  0000 C CNN
 	1    5000 7950
@@
 F 0 "R16" H 5370 7996 50  0001 L CNN
 F 1 "330" H 5370 7905 50  0001 L CNN
-F 2 "Resistors_ThroughHole:R_Axial_DIN0207_L6.3mm_D2.5mm_P10.16mm_Horizontal" V 5230 7950 50  0001 C CNN
+F 2 "Resistor_THT:R_Axial_DIN0207_L6.3mm_D2.5mm_P10.16mm_Horizontal" V 5230 7950 50  0001 C CNN
 F 3 "" H 5300 7950 50  0000 C CNN
 	1    5300 7950
@@
 F 0 "R17" H 5670 7996 50  0001 L CNN
 F 1 "330" H 5670 7905 50  0001 L CNN
-F 2 "Resistors_ThroughHole:R_Axial_DIN0207_L6.3mm_D2.5mm_P10.16mm_Horizontal" V 5530 7950 50  0001 C CNN
+F 2 "Resistor_THT:R_Axial_DIN0207_L6.3mm_D2.5mm_P10.16mm_Horizontal" V 5530 7950 50  0001 C CNN
 F 3 "" H 5600 7950 50  0000 C CNN
 	1    5600 7950
@@
 F 0 "R18" H 5970 7996 50  0001 L CNN
 F 1 "330" H 5970 7905 50  0001 L CNN
-F 2 "Resistors_ThroughHole:R_Axial_DIN0207_L6.3mm_D2.5mm_P10.16mm_Horizontal" V 5830 7950 50  0001 C CNN
+F 2 "Resistor_THT:R_Axial_DIN0207_L6.3mm_D2.5mm_P10.16mm_Horizontal" V 5830 7950 50  0001 C CNN
 F 3 "" H 5900 7950 50  0000 C CNN
 	1    5900 7950
@@
 F 0 "R19" H 6270 7996 50  0001 L CNN
 F 1 "330" H 6270 7905 50  0001 L CNN
-F 2 "Resistors_ThroughHole:R_Axial_DIN0207_L6.3mm_D2.5mm_P10.16mm_Horizontal" V 6130 7950 50  0001 C CNN
+F 2 "Resistor_THT:R_Axial_DIN0207_L6.3mm_D2.5mm_P10.16mm_Horizontal" V 6130 7950 50  0001 C CNN
 F 3 "" H 6200 7950 50  0000 C CNN
 	1    6200 7950
@@
 F 0 "R20" H 6570 7996 50  0001 L CNN
 F 1 "330" H 6570 7905 50  0001 L CNN
-F 2 "Resistors_ThroughHole:R_Axial_DIN0207_L6.3mm_D2.5mm_P10.16mm_Horizontal" V 6430 7950 50  0001 C CNN
+F 2 "Resistor_THT:R_Axial_DIN0207_L6.3mm_D2.5mm_P10.16mm_Horizontal" V 6430 7950 50  0001 C CNN
 F 3 "" H 6500 7950 50  0000 C CNN
 	1    6500 7950
@@
 F 0 "R21" H 6870 7996 50  0001 L CNN
 F 1 "330" H 6870 7905 50  0001 L CNN
-F 2 "Resistors_ThroughHole:R_Axial_DIN0207_L6.3mm_D2.5mm_P10.16mm_Horizontal" V 6730 7950 50  0001 C CNN
+F 2 "Resistor_THT:R_Axial_DIN0207_L6.3mm_D2.5mm_P10.16mm_Horizontal" V 6730 7950 50  0001 C CNN
 F 3 "" H 6800 7950 50  0000 C CNN
 	1    6800 7950
@@
 F 0 "R22" H 7170 7996 50  0001 L CNN
 F 1 "330" H 7170 7905 50  0001 L CNN
-F 2 "Resistors_ThroughHole:R_Axial_DIN0207_L6.3mm_D2.5mm_P10.16mm_Horizontal" V 7030 7950 50  0001 C CNN
+F 2 "Resistor_THT:R_Axial_DIN0207_L6.3mm_D2.5mm_P10.16mm_Horizontal" V 7030 7950 50  0001 C CNN
 F 3 "" H 7100 7950 50  0000 C CNN
 	1    7100 7950
@@
 F 0 "R23" H 7470 7996 50  0001 L CNN
 F 1 "330" H 7600 7950 50  0000 L CNN
-F 2 "Resistors_ThroughHole:R_Axial_DIN0207_L6.3mm_D2.5mm_P10.16mm_Horizontal" V 7330 7950 50  0001 C CNN
+F 2 "Resistor_THT:R_Axial_DIN0207_L6.3mm_D2.5mm_P10.16mm_Horizontal" V 7330 7950 50  0001 C CNN
 F 3 "" H 7400 7950 50  0000 C CNN
 	1    7400 7950
@@
 L allBonsaiSymbolLibs:LED_Small-device D3
 U 1 1 5836CDE4
-P 6150 2300
-F 0 "D3" H 6100 2425 50  0001 L CNN
-F 1 "Led_Small" H 5975 2200 50  0001 L CNN
-F 2 "bonsai:LED_Diodenmatrix" V 6150 2300 50  0001 C CNN
-F 3 "" V 6150 2300 50  0000 C CNN
-	1    6150 2300
+P 6150 2400
+F 0 "D3" H 6100 2525 50  0001 L CNN
+F 1 "Led_Small" H 5975 2300 50  0001 L CNN
+F 2 "bonsai:LED_Diodenmatrix" V 6150 2400 50  0001 C CNN
+F 3 "" V 6150 2400 50  0000 C CNN
+	1    6150 2400
 	1    0    0    -1
 $EndComp
@@
 	5800 2500 5800 2550
 Connection ~ 6050 2450
-Wire Wire Line
-	6050 2300 6050 2450
 Connection ~ 6050 2550
 Wire Wire Line
@@
 	5750 3950 5750 4600
 Connection ~ 6000 2500
-Connection ~ 6250 2300
-Wire Wire Line
-	6250 2300 6250 2500
 Connection ~ 6250 2500
 Wire Wire Line
@@
 F 0 "R7" V 1780 7000 50  0000 C CNN
 F 1 "330" V 1700 7000 50  0000 C CNN
-F 2 "Resistors_ThroughHole:R_Axial_DIN0207_L6.3mm_D2.5mm_P10.16mm_Horizontal" V 1630 7000 50  0001 C CNN
+F 2 "Resistor_THT:R_Axial_DIN0207_L6.3mm_D2.5mm_P10.16mm_Horizontal" V 1630 7000 50  0001 C CNN
 F 3 "" H 1700 7000 50  0000 C CNN
 	1    1700 7000
@@
 	5850 2200 5850 1900
 Wire Wire Line
-	6250 2200 6250 2300
-Wire Wire Line
 	6500 2150 5900 2150
 Wire Wire Line
@@
 F 0 "R2" H 6070 1296 50  0000 L CNN
 F 1 "1k" H 6070 1205 50  0000 L CNN
-F 2 "Resistors_ThroughHole:R_Axial_DIN0207_L6.3mm_D2.5mm_P10.16mm_Horizontal" V 5930 1250 50  0001 C CNN
+F 2 "Resistor_THT:R_Axial_DIN0207_L6.3mm_D2.5mm_P10.16mm_Horizontal" V 5930 1250 50  0001 C CNN
 F 3 "" H 6000 1250 50  0000 C CNN
 	1    6000 1250
@@
 F 0 "R1" V 6180 950 50  0000 C CNN
 F 1 "330" V 6100 950 50  0000 C CNN
-F 2 "Resistors_ThroughHole:R_Axial_DIN0207_L6.3mm_D2.5mm_P10.16mm_Horizontal" V 6030 950 50  0001 C CNN
+F 2 "Resistor_THT:R_Axial_DIN0207_L6.3mm_D2.5mm_P10.16mm_Horizontal" V 6030 950 50  0001 C CNN
 F 3 "" H 6100 950 50  0000 C CNN
 	1    6100 950
@@
 	2250 2350 2600 2350
 Connection ~ 2250 2250
+Connection ~ 6250 2400
+Wire Wire Line
+	6250 2400 6250 2500
+Wire Wire Line
+	6050 2400 6050 2450
+Wire Wire Line
+	6250 2200 6250 2400
 $EndSCHEMATC

Commit message: viele Kleinigkeiten
Parts:
- D2: footprint Diodes_ThroughHole:D_A-405_P10.16mm_Horizontal -> Diode_THT:D_A-405_P10.16mm_Horizontal
- Q1: footprint TO_SOT_Packages_THT:TO-92_Molded_Narrow -> Package_TO_SOT_THT:TO-92_Inline_Wide
- RP1, RP2: footprint Housings_SIP:SIP9_Housing_BigPads -> Package_SIP:SIP9_Housing_BigPads
- U1, U2, U3: footprint Housings_DIP:DIP-16_W7.62mm_Socket_LongPads -> Package_DIP:DIP-16_W7.62mm_Socket_LongPads
- U5: footprint Housings_DIP:DIP-20_W7.62mm_Socket_LongPads -> Package_DIP:DIP-20_W7.62mm_Socket_LongPads
- U6: footprint tg_foodprint:DIP-20_W7.62mm_Socket_LongPadstg -> Package_DIP:DIP-20_W7.62mm_Socket_LongPads
Changed lines of the file:
@@
 F 0 "U3" H 4950 3850 50  0000 C CNN
 F 1 "74LS138" H 4900 3750 50  0000 C CNN
-F 2 "Housings_DIP:DIP-16_W7.62mm_Socket_LongPads" H 4950 3750 50  0001 C CNN
+F 2 "Package_DIP:DIP-16_W7.62mm_Socket_LongPads" H 4950 3750 50  0001 C CNN
 F 3 "" H 4950 3750 50  0000 C CNN
 	1    4950 3750
@@
 F 0 "D2" V 11851 2278 50  0000 L CNN
 F 1 "D" V 11942 2278 50  0000 L CNN
-F 2 "Diodes_ThroughHole:D_A-405_P10.16mm_Horizontal" V 12041 2278 60  0001 L CNN
+F 2 "Diode_THT:D_A-405_P10.16mm_Horizontal" V 12041 2278 60  0001 L CNN
 F 3 "" H 11950 2200 60  0000 C CNN
 	1    11950 2200
@@
 F 0 "U5" V 6200 5550 50  0000 R CNN
 F 1 "74LS374" V 6300 5550 50  0000 R CNN
-F 2 "Housings_DIP:DIP-20_W7.62mm_Socket_LongPads" H 6250 5300 50  0001 C CNN
+F 2 "Package_DIP:DIP-20_W7.62mm_Socket_LongPads" H 6250 5300 50  0001 C CNN
 F 3 "" H 6250 5300 50  0000 C CNN
 	1    6250 5300
@@
 F 0 "RP1" V 5950 1300 50  0000 L CNN
 F 1 "R_PACK8BUSSED" H 6028 1708 50  0001 L CNN
-F 2 "Housings_SIP:SIP9_Housing_BigPads" H 6028 1609 60  0001 L CNN
+F 2 "Package_SIP:SIP9_Housing_BigPads" H 6028 1609 60  0001 L CNN
 F 3 "" H 5900 1750 60  0000 C CNN
 	1    5900 1700
@@
 F 0 "U6" V 8300 5500 50  0000 R CNN
 F 1 "74LS374" V 8400 5550 50  0000 R CNN
-F 2 "tg_foodprint:DIP-20_W7.62mm_Socket_LongPadstg" V 8441 4671 50  0001 R CNN
+F 2 "Package_DIP:DIP-20_W7.62mm_Socket_LongPads" V 8441 4671 50  0001 R CNN
 F 3 "" H 8350 5300 50  0000 C CNN
 	1    8350 5300
@@
 F 0 "RP2" V 8050 1300 50  0000 L CNN
 F 1 "R_PACK8BUSSED" H 8128 1708 50  0001 L CNN
-F 2 "Housings_SIP:SIP9_Housing_BigPads" H 8128 1609 60  0001 L CNN
+F 2 "Package_SIP:SIP9_Housing_BigPads" H 8128 1609 60  0001 L CNN
 F 3 "" H 8000 1750 60  0000 C CNN
 	1    8000 1700
@@
 F 0 "U2" H 4950 2800 50  0000 C CNN
 F 1 "74LS138" H 4900 2700 50  0000 C CNN
-F 2 "Housings_DIP:DIP-16_W7.62mm_Socket_LongPads" H 4950 2700 50  0001 C CNN
+F 2 "Package_DIP:DIP-16_W7.62mm_Socket_LongPads" H 4950 2700 50  0001 C CNN
 F 3 "" H 4950 2700 50  0000 C CNN
 	1    4950 2700
@@
 F 0 "Q1" H 6950 1300 50  0001 R CNN
 F 1 "Q_PNP_BCE" H 7250 1200 50  0001 R CNN
-F 2 "TO_SOT_Packages_THT:TO-92_Molded_Narrow" H 6850 1350 50  0001 C CNN
+F 2 "Package_TO_SOT_THT:TO-92_Inline_Wide" H 6850 1350 50  0001 C CNN
 F 3 "" H 6650 1250 50  0000 C CNN
 	1    6650 1250
@@
 F 0 "U1" H 3250 2400 50  0000 C CNN
 F 1 "74LS161" H 3250 2300 50  0000 C CNN
-F 2 "Housings_DIP:DIP-16_W7.62mm_Socket_LongPads" H 3300 2150 50  0001 C CNN
+F 2 "Package_DIP:DIP-16_W7.62mm_Socket_LongPads" H 3300 2150 50  0001 C CNN
 F 3 "" H 3300 2150 50  0001 C CNN
 	1    3300 2150

Commit message: Steuerwerk: Verbinder für die beiden unbenutzten Steuersignale eingebaut
Parts:
- added J9: Conn_01x02, Connector_Molex:Molex_KK-254_AE-6410-02A_1x02_P2.54mm_Vertical, symbol Connector_Generic:Conn_01x02
Connections:
- wire segments 449 -> 457
Changed lines of the file:
@@
 Wire Wire Line
 	6000 4150 5850 4150
-Connection ~ 6000 2300
 Connection ~ 8400 4000
 Wire Wire Line
@@
 Wire Wire Line
 	5550 2450 6050 2450
-Wire Wire Line
-	5550 2350 7900 2350
 Wire Wire Line
 	4200 2550 4350 2550
@@
 $EndComp
 Wire Wire Line
-	7100 7150 7100 7000
+	7100 7150 7100 7100
 Wire Wire Line
 	6800 6950 6800 7100
@@
 $EndComp
 Wire Wire Line
-	5500 2300 5500 1250
-Wire Wire Line
-	5500 2300 6000 2300
-Wire Wire Line
 	3850 4150 4100 4150
 Wire Wire Line
@@
 Connection ~ 3750 4000
 NoConn ~ 3900 2150
-Wire Wire Line
-	6000 2300 6000 2500
 Wire Wire Line
 	1950 1650 2600 1650
@@
 $EndComp
 Wire Wire Line
-	7400 7050 7400 7150
+	7400 7050 7400 7100
 $Comp
 L Bonsai:74541 U7
@@
 	5600 1900 5700 1900
 Wire Wire Line
-	6000 2250 6000 2300
-Wire Wire Line
 	5750 1900 5750 2600
 Wire Wire Line
 	6000 2250 5800 2250
 Wire Wire Line
-	5800 2250 5800 1900
+	5800 2250 5800 2200
 Wire Wire Line
 	6250 2200 5850 2200
@@
 Wire Wire Line
 	5900 2150 5900 1900
-Wire Wire Line
-	6500 2150 6500 2900
 Wire Wire Line
 	6750 2100 5950 2100
@@
 Wire Wire Line
 	6250 2200 6250 2400
+Wire Wire Line
+	5550 2350 7900 2350
+Wire Wire Line
+	6500 2150 6500 2900
+Wire Wire Line
+	5800 2200 5500 2200
+Connection ~ 5800 2200
+Wire Wire Line
+	5800 2200 5800 1900
+Wire Wire Line
+	5500 2200 5500 1250
+Wire Wire Line
+	6000 2250 6000 2500
+$Comp
+L Connector_Generic:Conn_01x02 J9
+U 1 1 5FB0DD94
+P 7350 8900
+F 0 "J9" V 7268 8712 50  0000 R CNN
+F 1 "Conn_01x02" V 7313 8712 50  0001 R CNN
+F 2 "Connector_Molex:Molex_KK-254_AE-6410-02A_1x02_P2.54mm_Vertical" H 7350 8900 50  0001 C CNN
+F 3 "~" H 7350 8900 50  0001 C CNN
+	1    7350 8900
+	0    1    1    0
+$EndComp
+Wire Wire Line
+	7100 7100 7250 7100
+Wire Wire Line
+	7250 7100 7250 8700
+Connection ~ 7100 7100
+Wire Wire Line
+	7100 7100 7100 7000
+Wire Wire Line
+	7400 7100 7550 7100
+Wire Wire Line
+	7550 7100 7550 8550
+Wire Wire Line
+	7550 8550 7350 8550
+Wire Wire Line
+	7350 8550 7350 8700
+Connection ~ 7400 7100
+Wire Wire Line
+	7400 7100 7400 7150
 $EndSCHEMATC

Commit message: Steuerwerk: Platzhalter für LEDs eingefügt
Parts:
- added D100, D101, D102, D103, D104, D105, D106, D107, D108, D109, D110, D111, D112, D113, D114, D115, D116, D117, D118, D64, D65, D66, D67, D68, D69, D70, D71, D72, D73, D74, D75, D76, D77, D78, D79, D80, D81, D82, D83, D84, D85, D86, D87, D88, D89, D90, D91, D92, D93, D94, D95, D96, D97, D98, D99: bonsai_Led_Small_Platzhalter, bonsai:LED_Diodenmatrix_Platzhalter, symbol Bonsai:bonsai_Led_Small_Platzhalter
Connections:
- wire segments 457 -> 615

Commit message: Steuerwerk: weitere Platzhalterdioden eingebaut
Parts:
- added D119, D120, D121, D122, D123, D124, D125, D126, D127, D128, D129, D130, D131, D132, D133, D134, D135, D136, D137, D138, D139, D140, D141, D142, D143, D144, D145, D146, D147, D148, D149, D150, D151, D152, D153, D154, D155, D156, D157, D158, D159, D160, D161, D162, D163, D164, D165, D166, D167, D168, D169, D170, D171, D172: bonsai_Led_Small_Platzhalter, bonsai:LED_Diodenmatrix_Platzhalter, symbol Bonsai:bonsai_Led_Small_Platzhalter
Connections:
- wire segments 615 -> 772

Commit message: Steuerwerk: alle Diodenplatzhalter eingebaut
Parts:
- added D173, D174, D175, D176, D177, D178, D179, D180, D181, D182, D183, D184, D185, D186, D187, D188, D189, D190, D191, D192, D193, D194, D195, D196, D197, D198, D199, D200, D201, D202, D203, D204, D205, D206, D207, D208, D209, D210, D211, D212, D213, D214, D215, D216, D217, D218, D219, D220, D221, D222, D223, D224, D225, D226, D227, D228, D229, D230, D231, D232, D233, D234, D235, D236, D237, D238, D239, D240, D241, D242, D243, D244, D245, D246, D247, D248, D249, D250, D251, D252, D253, D254, D255, D256, D257, D258, D259, D260, D261, D262, D263, D264, D265, D266, D267, D268, D269, D270, D271, D272, D273, D274, D275, D276, D277, D278, D279: bonsai_Led_Small_Platzhalter, bonsai:LED_Diodenmatrix_Platzhalter, symbol Bonsai:bonsai_Led_Small_Platzhalter
Connections:
- wire segments 772 -> 1093
- no-connect marks 2 -> 1

Commit message: Steuerwerk rev 2.0
Parts:
- added unit 4 of U4
- added unit 3 of U4
- added unit 2 of U4
Connections:
- net labels added: CLK, ~clrMPC, ~enCU, ~enDEC, ~readR, ~writeAccu
- net labels removed: Takt, clrMPC, enAkku, enDEC, enSTW, loadIR
- wire segments 1093 -> 1097
- no-connect marks 1 -> 4
Changed lines of the file:
@@
 $EndComp
 Text Label 1650 5750 0    60   ~ 0
-Takt
-Text Label 1750 5850 0    60   ~ 0
-enDEC
+CLK
+Text Label 1650 5850 0    60   ~ 0
+~enDEC
 Text Label 1700 8050 0    60   ~ 0
-enAkku
+~writeAccu
 Text Label 1700 8150 0    60   ~ 0
-loadIR
+~readR
 $Comp
 L power:VCC #PWR06
@@
 Wire Wire Line
 	4150 3400 4350 3400
-Connection ~ 4100 1750
 Wire Wire Line
-	4100 1750 4100 3500
-Connection ~ 4050 1850
-Wire Wire Line
-	4050 1850 4050 3600
+	4050 1850 4050 2550
 Wire Wire Line
 	5550 4100 5800 4100
@@
 	5550 2450 5800 2450
 Wire Wire Line
-	4200 2550 4350 2550
-Wire Wire Line
-	4200 1850 4200 2550
-Wire Wire Line
-	4300 2450 4350 2450
-Wire Wire Line
-	4300 1750 4300 2450
-Wire Wire Line
-	4350 1650 4350 2350
-Wire Wire Line
 	8550 4450 9600 4450
 Wire Wire Line
@@
 Wire Wire Line
 	6800 3500 7050 3500
-Wire Wire Line
-	4100 1750 4300 1750
-Wire Wire Line
-	4050 1850 4200 1850
 $Comp
 L power:GND #PWR08
@@
 vom Befehlesdecoder
 Text Label 1650 6000 0    60   ~ 0
-enSTW
+~enCU
 Wire Wire Line
 	1650 6200 1650 5950
@@
 Connection ~ 4000 3900
 Wire Wire Line
-	4150 1650 4350 1650
-Wire Wire Line
 	3900 1650 4150 1650
-Connection ~ 4150 1650
 Connection ~ 4150 3400
 Connection ~ 2400 7950
 Text Label 1700 7950 0    60   ~ 0
-clrMPC
+~clrMPC
 Wire Wire Line
 	4000 1950 4000 3050
 Wire Wire Line
-	4150 1650 4150 3400
+	4150 1650 4150 2350
 Wire Wire Line
 	4350 3050 4000 3050
@@
 Wire Wire Line
 	9400 4100 9650 4100
+Connection ~ 4050 2550
+Wire Wire Line
+	4050 2550 4050 3600
+Wire Wire Line
+	4050 2550 4350 2550
+Wire Wire Line
+	4350 2350 4150 2350
+Connection ~ 4150 2350
+Wire Wire Line
+	4150 2350 4150 3400
+Wire Wire Line
+	4100 1750 4100 2450
+Connection ~ 4100 2450
+Wire Wire Line
+	4100 2450 4100 3500
+Wire Wire Line
+	4100 2450 4350 2450
+$Comp
+L Bonsai:74240 U4
+U 4 1 6088CDDE
+P 14000 6700
+F 0 "U4" V 13850 6750 50  0000 L CNN
+F 1 "74240" V 14000 6800 50  0000 L CNN
+F 2 "Package_DIP:DIP-20_W7.62mm_Socket_LongPads" H 14150 6600 50  0001 C CNN
+F 3 "" H 14150 6600 50  0001 C CNN
+	4    14000 6700
+	0    1    1    0
+$EndComp
+$Comp
+L Bonsai:74240 U4
+U 3 1 6088E591
+P 13650 6700
+F 0 "U4" V 13500 6750 50  0000 L CNN
+F 1 "74240" V 13650 6800 50  0001 L CNN
+F 2 "Package_DIP:DIP-20_W7.62mm_Socket_LongPads" H 13800 6600 50  0001 C CNN
+F 3 "" H 13800 6600 50  0001 C CNN
+	3    13650 6700
+	0    1    1    0
+$EndComp
+$Comp
+L Bonsai:74240 U4
+U 2 1 6088F09D
+P 13300 6700
+F 0 "U4" V 13150 6750 50  0000 L CNN
+F 1 "74240" V 13300 6800 50  0001 L CNN
+F 2 "Package_DIP:DIP-20_W7.62mm_Socket_LongPads" H 13450 6600 50  0001 C CNN
+F 3 "" H 13450 6600 50  0001 C CNN
+	2    13300 6700
+	0    1    1    0
+$EndComp
+Wire Wire Line
+	14000 6350 14000 6400
+Wire Wire Line
+	13650 6400 13650 6350
+Connection ~ 13650 6350
+Wire Wire Line
+	13650 6350 14000 6350
+NoConn ~ 14000 7050
+NoConn ~ 13650 7050
+NoConn ~ 13300 7050
+$Comp
+L power:VCC #PWR0101
+U 1 1 6125D521
+P 13650 6250
+F 0 "#PWR0101" H 13650 6100 50  0001 C CNN
+F 1 "VCC" H 13667 6423 50  0000 C CNN
+F 2 "" H 13650 6250 50  0001 C CNN
+F 3 "" H 13650 6250 50  0001 C CNN
+	1    13650 6250
+	1    0    0    -1
+$EndComp
+Wire Wire Line
+	13650 6250 13650 6350
+Wire Wire Line
+	13650 6350 13300 6350
+Wire Wire Line
+	13300 6350 13300 6400
 $EndSCHEMATC

Commit message: Steuerwerk und Befehle bearbeitet
Parts:
- D1: symbol allBonsaiSymbolLibs:LED-device -> Device:LED_Small_ALT
- D10, D11, D12, D13, D14, D15, D16, D17, D18, D19, D20, D21, D22, D23, D24, D25, D26, D27, D28, D29, D3, D30, D31, D32, D33, D34, D35, D36, D37, D38, D39, D4, D40, D41, D42, D47, D48, D49, D5, D50, D51, D52, D53, D54, D55, D56, D57, D58, D59, D6, D60, D61, D62, D63, D7, D8, D9: symbol allBonsaiSymbolLibs:LED_Small-device -> Device:LED_Small_ALT
- D43, D44, D45, D46: symbol allBonsaiSymbolLibs:LED-device -> Device:LED_ALT
Connections:
- wire segments 1097 -> 1106
