File: Steuerwerk.sch (KiCad schematic (older format))
At the start: 331 parts, among them J1 Conn_01x04, J2 Conn_01x02, J3 Conn_01x03, J4 Conn_01x03, J5 Conn_01x02, J6 Conn_01x04, J7 Conn_01x02, J8 Conn_01x04, J9 Conn_01x02, Q1 Q_PNP_BCE, U1 74LS161, U2 74LS138, U3 74LS138, U4 74240, U5 74LS374, U6 74LS374, U7 74541, U8 74541

Commit message: Steuerwerk: keine verstecken Pins mehr; alle Pins explizit im Schaltplan angeschossen
Connections:
- wire segments 1106 -> 1117
Other:
- note added: "Mikroprogramm-\nzähler \nMPC"
- note removed: "Mikroprogrammzähler \nMPC"
