File: Befehle.sch (KiCad schematic (older format))
At the start: 60 parts, among them J1 2PinTerminalBlocktg, J2 2PinTerminalBlocktg, J3 3PinTerminalBlocktg, J4 2PinTerminalBlocktg, J5 2PinTerminalBlocktg, P1 CONN_02X10, P2 CONN_02X10, U1 74LS14, U2 74540, U3 7400, U4 74HCT02, U5 74LS541, U6 74LS373, U7 74LS139, U8 74LS540

Commit message: Befehle: vor Umbau der Diodenmatrix im Schalplan
Connections:
- net labels added: AB0, AB1, AB2, AB3, AB4, AB5, AB6, AB7
- net labels removed: y1, y2, y3, y4, y5, y6, y7, y8
- wire segments 316 -> 281

Commit message: Befehle: Schaltplan bearbeitet
Parts:
- added C3, C4, C5, C6, C7, C8: 100n, Capacitor_THT:C_Disc_D10.0mm_W2.5mm_P5.00mm, symbol allBonsaiSymbolLibs:C_Small
- added C9: CP, Capacitor_THT:CP_Radial_D8.0mm_P2.50mm, symbol Device:CP
- added D23, D24, D25, D26, D27, D28, D29, D30, D31, D32: bonsai_Led_Small_Platzhalter, bonsai:LED_Diodenmatrix_Platzhalter, symbol Bonsai:bonsai_Led_Small_Platzhalter
- C1, C2: footprint Capacitors_ThroughHole:C_Disc_D10.0mm_W2.5mm_P5.00mm -> Capacitor_THT:C_Disc_D10.0mm_W2.5mm_P5.00mm
- D11, D12, D15, D16, D19, D20: footprint allBonsaiFootprintsLibs:Diode_D1.8mm_W3.3mm_H2.4mmBonsai -> bonsai:LED_Diodenmatrix
- U2: footprint Housings_DIP:DIP-20_W7.62mm_Socket_LongPads -> allBonsaiFootprintsLibs:DIP-20_W7.62mm_Socket_LongPadstg
Connections:
- wire segments 281 -> 300

Commit message: Befehle: Schaltplan geändert
Parts:
- added unit 9 of U2
- U2: symbol allBonsaiSymbolLibs:74540 -> Bonsai:74540
- U4: footprint allBonsaiFootprintsLibs:DIP-14_W7.62mm_Socket_LongPadstg -> Package_DIP:DIP-14_W7.62mm_Socket_LongPads
Connections:
- wire segments 300 -> 299
Other:
- note added: "0"
- note added: "7"

Commit message: Steuerwerk und Befehle bearbeitet
Parts:
- removed J1, J2, J4, J5: 2PinTerminalBlocktg, 2PinTerminalBlocktg, symbol allBonsaiSymbolLibs:2PinTerminalBlocktg-2PinTerminalBlocktg
- removed J3: 3PinTerminalBlocktg, 3PinTerminalBlocktg, symbol allBonsaiSymbolLibs:3PinTerminalBlocktg-3PinTerminalBlocktg
- removed P1, P2: CONN_02X10, allBonsaiFootprintsLibs:Pin_Header_Straight_2x10_Pitch2.00mmBonsai.pretty, symbol allBonsaiSymbolLibs:Conn_02x10_Counter_Clockwise-conn
- removed R7: 1k, Resistors_ThroughHole:R_Axial_DIN0207_L6.3mm_D2.5mm_P10.16mm_Horizontal, symbol allBonsaiSymbolLibs:R-device
- removed U3: 7400, allBonsaiFootprintsLibs:DIP-14_W7.62mm_Socket_LongPadstg, symbol allBonsaiSymbolLibs:7400
- removed U4: 74HCT02, Package_DIP:DIP-14_W7.62mm_Socket_LongPads, symbol allBonsaiSymbolLibs:74HCT02
- added C10: 100n, Capacitor_THT:C_Disc_D10.0mm_W2.5mm_P5.00mm, symbol allBonsaiSymbolLibs:C_Small
- added J1, J4: Conn_02x10_Odd_Even, Connector_PinHeader_2.54mm:PinHeader_2x10_P2.54mm_Vertical, symbol Connector_Generic:Conn_02x10_Odd_Even
- added J2, J5: Conn_01x02, Connector_Molex:Molex_KK-254_AE-6410-02A_1x02_P2.54mm_Vertical, symbol Connector_Generic:Conn_01x02
- added J3: Conn_01x04, Connector_Molex:Molex_KK-254_AE-6410-04A_1x04_P2.54mm_Vertical, symbol Connector_Generic:Conn_01x04
- added J6: Conn_01x03, Connector_Molex:Molex_KK-254_AE-6410-03A_1x03_P2.54mm_Vertical, symbol Connector_Generic:Conn_01x03
- added U7: 7402, Package_DIP:DIP-14_W7.62mm_Socket_LongPads, symbol 74xx_IEEE:7402
- added U8: 7408, Package_DIP:DIP-14_W7.62mm_Socket_LongPads, symbol 74xx_IEEE:7408
- added U9: 7400, Package_DIP:DIP-14_W7.62mm_Socket_LongPads, symbol 74xx_IEEE:7400
- D1: renamed from D5; footprint LEDs:LED_D3.0mm -> LED_THT:LED_D3.0mm; symbol allBonsaiSymbolLibs:Led_Small -> Device:LED_Small_ALT
- D10: renamed from D15; symbol allBonsaiSymbolLibs:Led_Small -> Device:LED_Small_ALT
- D13: renamed from D12; symbol allBonsaiSymbolLibs:Led_Small -> Device:LED_Small_ALT
- D17: renamed from D2; footprint LEDs:LED_D3.0mm -> LED_THT:LED_D3.0mm; symbol allBonsaiSymbolLibs:Led_Small -> Device:LED_Small_ALT
- D19: renamed from D16; symbol allBonsaiSymbolLibs:Led_Small -> Device:LED_Small_ALT
- D2: renamed from D6; footprint LEDs:LED_D3.0mm -> LED_THT:LED_D3.0mm; symbol allBonsaiSymbolLibs:Led_Small -> Device:LED_Small_ALT
- D24: renamed from D19; symbol allBonsaiSymbolLibs:Led_Small -> Device:LED_Small_ALT
- D25: renamed from D20; symbol allBonsaiSymbolLibs:Led_Small -> Device:LED_Small_ALT
- D26: renamed from D4; footprint LEDs:LED_D3.0mm -> LED_THT:LED_D3.0mm
- D27: renamed from D7; footprint LEDs:LED_D3.0mm -> LED_THT:LED_D3.0mm
- D28: renamed from D17; footprint LEDs:LED_D3.0mm -> LED_THT:LED_D3.0mm
- D29: renamed from D21; footprint LEDs:LED_D3.0mm -> LED_THT:LED_D3.0mm
- D3: renamed from D8; footprint LEDs:LED_D3.0mm -> LED_THT:LED_D3.0mm; symbol allBonsaiSymbolLibs:Led_Small -> Device:LED_Small_ALT
- D30: renamed from D3; footprint LEDs:LED_D3.0mm -> LED_THT:LED_D3.0mm; symbol allBonsaiSymbolLibs:Led_Small -> Device:LED_Small_ALT
- D31: renamed from D1; footprint LEDs:LED_D3.0mm -> LED_THT:LED_D3.0mm; symbol allBonsaiSymbolLibs:Led_Small -> Device:LED_Small_ALT
- D32: renamed from D22; footprint Diodes_ThroughHole:D_DO-41_SOD81_P10.16mm_Horizontal -> Diode_THT:D_A-405_P10.16mm_Horizontal
- D4: renamed from D9; footprint LEDs:LED_D3.0mm -> LED_THT:LED_D3.0mm; symbol allBonsaiSymbolLibs:Led_Small -> Device:LED_Small_ALT
- D5: renamed from D10; footprint LEDs:LED_D3.0mm -> LED_THT:LED_D3.0mm; symbol allBonsaiSymbolLibs:Led_Small -> Device:LED_Small_ALT
- D6: renamed from D13; footprint LEDs:LED_D3.0mm -> LED_THT:LED_D3.0mm; symbol allBonsaiSymbolLibs:Led_Small -> Device:LED_Small_ALT
- D7: renamed from D14; footprint LEDs:LED_D3.0mm -> LED_THT:LED_D3.0mm; symbol allBonsaiSymbolLibs:Led_Small -> Device:LED_Small_ALT
- D8: renamed from D18; footprint LEDs:LED_D3.0mm -> LED_THT:LED_D3.0mm; symbol allBonsaiSymbolLibs:Led_Small -> Device:LED_Small_ALT
- D9: renamed from D11; symbol allBonsaiSymbolLibs:Led_Small -> Device:LED_Small_ALT
- R1: renamed from R10; footprint Resistors_ThroughHole:R_Axial_DIN0207_L6.3mm_D2.5mm_P10.16mm_Horizontal -> Resistor_THT:R_Axial_DIN0207_L6.3mm_D2.5mm_P10.16mm_Horizontal
- R10: renamed from R5; footprint Resistors_ThroughHole:R_Axial_DIN0207_L6.3mm_D2.5mm_P10.16mm_Horizontal -> Resistor_THT:R_Axial_DIN0207_L6.3mm_D2.5mm_P10.16mm_Horizontal
- R11: renamed from R4; footprint Resistors_ThroughHole:R_Axial_DIN0207_L6.3mm_D2.5mm_P10.16mm_Horizontal -> Resistor_THT:R_Axial_DIN0207_L6.3mm_D2.5mm_P10.16mm_Horizontal
- R12: renamed from R9; footprint Resistors_ThroughHole:R_Axial_DIN0207_L6.3mm_D2.5mm_P10.16mm_Horizontal -> Resistor_THT:R_Axial_DIN0207_L6.3mm_D2.5mm_P10.16mm_Horizontal
- R13: renamed from R12; footprint Resistors_ThroughHole:R_Axial_DIN0207_L6.3mm_D2.5mm_P10.16mm_Horizontal -> Resistor_THT:R_Axial_DIN0207_L6.3mm_D2.5mm_P10.16mm_Horizontal
- R14: renamed from R20; footprint Resistors_ThroughHole:R_Axial_DIN0207_L6.3mm_D2.5mm_P10.16mm_Horizontal -> Resistor_THT:R_Axial_DIN0207_L6.3mm_D2.5mm_P10.16mm_Horizontal
- R15: renamed from R24; footprint Resistors_ThroughHole:R_Axial_DIN0207_L6.3mm_D2.5mm_P10.16mm_Horizontal -> Resistor_THT:R_Axial_DIN0207_L6.3mm_D2.5mm_P10.16mm_Horizontal
- R16: renamed from R8; footprint Resistors_ThroughHole:R_Axial_DIN0207_L6.3mm_D2.5mm_P10.16mm_Horizontal -> Resistor_THT:R_Axial_DIN0207_L6.3mm_D2.5mm_P10.16mm_Horizontal
- R17: renamed from R2; footprint Resistors_ThroughHole:R_Axial_DIN0207_L6.3mm_D2.5mm_P10.16mm_Horizontal -> Resistor_THT:R_Axial_DIN0207_L6.3mm_D2.5mm_P10.16mm_Horizontal
- R18: renamed from R3; footprint Resistors_ThroughHole:R_Axial_DIN0207_L6.3mm_D2.5mm_P10.16mm_Horizontal -> Resistor_THT:R_Axial_DIN0207_L6.3mm_D2.5mm_P10.16mm_Horizontal
- R19: renamed from R6; footprint Resistors_ThroughHole:R_Axial_DIN0207_L6.3mm_D2.5mm_P10.16mm_Horizontal -> Resistor_THT:R_Axial_DIN0207_L6.3mm_D2.5mm_P10.16mm_Horizontal
- R2: renamed from R11; footprint Resistors_ThroughHole:R_Axial_DIN0207_L6.3mm_D2.5mm_P10.16mm_Horizontal -> Resistor_THT:R_Axial_DIN0207_L6.3mm_D2.5mm_P10.16mm_Horizontal
- R3: renamed from R13; footprint Resistors_ThroughHole:R_Axial_DIN0207_L6.3mm_D2.5mm_P10.16mm_Horizontal -> Resistor_THT:R_Axial_DIN0207_L6.3mm_D2.5mm_P10.16mm_Horizontal
- R4: renamed from R14; footprint Resistors_ThroughHole:R_Axial_DIN0207_L6.3mm_D2.5mm_P10.16mm_Horizontal -> Resistor_THT:R_Axial_DIN0207_L6.3mm_D2.5mm_P10.16mm_Horizontal
- R5: renamed from R15; footprint Resistors_ThroughHole:R_Axial_DIN0207_L6.3mm_D2.5mm_P10.16mm_Horizontal -> Resistor_THT:R_Axial_DIN0207_L6.3mm_D2.5mm_P10.16mm_Horizontal
- R6: renamed from R16; footprint Resistors_ThroughHole:R_Axial_DIN0207_L6.3mm_D2.5mm_P10.16mm_Horizontal -> Resistor_THT:R_Axial_DIN0207_L6.3mm_D2.5mm_P10.16mm_Horizontal
- R7: renamed from R18; footprint Resistors_ThroughHole:R_Axial_DIN0207_L6.3mm_D2.5mm_P10.16mm_Horizontal -> Resistor_THT:R_Axial_DIN0207_L6.3mm_D2.5mm_P10.16mm_Horizontal
- R8: renamed from R21; footprint Resistors_ThroughHole:R_Axial_DIN0207_L6.3mm_D2.5mm_P10.16mm_Horizontal -> Resistor_THT:R_Axial_DIN0207_L6.3mm_D2.5mm_P10.16mm_Horizontal
- R9: renamed from R1; footprint Resistors_ThroughHole:R_Axial_DIN0207_L6.3mm_D2.5mm_P10.16mm_Horizontal -> Resistor_THT:R_Axial_DIN0207_L6.3mm_D2.5mm_P10.16mm_Horizontal
- RP1: footprint Resistors_ThroughHole:R_Array_SIP5 -> Resistor_THT:R_Array_SIP5
- U1: footprint allBonsaiFootprintsLibs:DIP-14_W7.62mm_Socket_LongPadstg -> Package_DIP:DIP-14_W7.62mm_Socket_LongPads
- U2: renamed from U5; footprint allBonsaiFootprintsLibs:DIP-20_W7.62mm_Socket_LongPadstg -> Package_DIP:DIP-20_W7.62mm_LongPads
- U3: renamed from U8; footprint allBonsaiFootprintsLibs:DIP-20_W7.62mm_Socket_LongPadstg -> Package_DIP:DIP-20_W7.62mm_LongPads
- U4: renamed from U7; footprint allBonsaiFootprintsLibs:DIP-16_W7.62mm_Socket_LongPadstg -> Package_DIP:DIP-16_W7.62mm_Socket_LongPads
- U5: renamed from U6; footprint allBonsaiFootprintsLibs:DIP-20_W7.62mm_Socket_LongPadstg -> Package_DIP:DIP-20_W7.62mm_LongPads
- U6: renamed from U2; footprint allBonsaiFootprintsLibs:DIP-20_W7.62mm_Socket_LongPadstg -> Package_DIP:DIP-20_W7.62mm_LongPads
- renumbered C9 to C1, C1 to C2, C2 to C3, C3 to C4, C4 to C5, C5 to C6, C6 to C7, C7 to C8, C8 to C9, D24 to D11, D25 to D12, D26 to D14, D27 to D15, D28 to D16, D23 to D18, D29 to D20, D30 to D21, D31 to D22, D32 to D23
Connections:
- net labels added: DB0, DB1, DB2, DB3, DB4, DB5, DB6, DB7, a0, b0, b1, h0, h1, h2, h3, is0, v0, v1, v2, v3, ~incPC, ~incPCz, ~is0_&_incPCz, ~upPC
- net labels removed: 0, 1, 2, 3, a8, d1, d2, d3, d4, d44, d5, d6, d7
- wire segments 299 -> 311
Other:
- note added: "Adressbus"
- note added: "Datenbus"
- note added: "Nullentdeckungslogik"
- note added: "ungenutzte Gatter"
- note removed: "0"
- note removed: "7"

Commit message: Befehle: An der Platine weitergearbeitet
Parts:
- removed J6: Conn_01x03, Connector_Molex:Molex_KK-254_AE-6410-03A_1x03_P2.54mm_Vertical, symbol Connector_Generic:Conn_01x03
- added J6: Conn_01x04, Connector_Molex:Molex_KK-254_AE-6410-04A_1x04_P2.54mm_Vertical, symbol Connector_Generic:Conn_01x04
- U8: symbol 74xx_IEEE:7408 -> Bonsai:7408
Connections:
- net labels added: ~readIR, ~writeIR
- net labels removed: enableR, incPC, loadIR, upPC
- wire segments 311 -> 317
Other:
- note added: "Befehlsregister\n(Instruction Register IR)"
- note added: "Signal für den PC"
- note added: "Steuersignale\nvom Steuerwerk"
Changed lines of the file:
@@
 $EndComp
 Text GLabel 1200 4000 0    60   Input ~ 0
-enableR
+~writeIR
 $Comp
 L power:GND #PWR05
@@
 	1    0    0    -1
 $EndComp
-Text GLabel 1600 7350 0    60   Input ~ 0
-loadIR
 $Comp
 L allBonsaiSymbolLibs:R-device R11
 U 1 1 582B55B4
-P 1800 7050
-F 0 "R11" V 1700 7050 50  0000 C CNN
-F 1 "4,7k" V 1800 7050 50  0000 C CNN
-F 2 "Resistor_THT:R_Axial_DIN0207_L6.3mm_D2.5mm_P10.16mm_Horizontal" H 1450 7250 50  0001 C CNN
-F 3 "" H 1800 7050 50  0000 C CNN
-	1    1800 7050
+P 1350 7050
+F 0 "R11" V 1250 7050 50  0000 C CNN
+F 1 "4,7k" V 1350 7050 50  0000 C CNN
+F 2 "Resistor_THT:R_Axial_DIN0207_L6.3mm_D2.5mm_P10.16mm_Horizontal" H 1000 7250 50  0001 C CNN
+F 3 "" H 1350 7050 50  0000 C CNN
+	1    1350 7050
 	1    0    0    1
 $EndComp
@@
 L power:VCC #PWR010
 U 1 1 582B5718
-P 1800 6800
-F 0 "#PWR010" H 1800 6650 50  0001 C CNN
-F 1 "VCC" H 1800 6950 50  0000 C CNN
-F 2 "" H 1800 6800 50  0000 C CNN
-F 3 "" H 1800 6800 50  0000 C CNN
-	1    1800 6800
+P 1350 6800
+F 0 "#PWR010" H 1350 6650 50  0001 C CNN
+F 1 "VCC" H 1350 6950 50  0000 C CNN
+F 2 "" H 1350 6800 50  0000 C CNN
+F 3 "" H 1350 6800 50  0000 C CNN
+	1    1350 6800
 	1    0    0    -1
 $EndComp
@@
 L allBonsaiSymbolLibs:R-device R16
 U 1 1 582B6652
-P 2950 7550
-F 0 "R16" V 2950 7550 50  0000 C CNN
-F 1 "330" V 2850 7550 50  0000 C CNN
-F 2 "Resistor_THT:R_Axial_DIN0207_L6.3mm_D2.5mm_P10.16mm_Horizontal" H 3300 7300 50  0001 C CNN
-F 3 "" H 2950 7550 50  0000 C CNN
-	1    2950 7550
+P 2250 7550
+F 0 "R16" V 2250 7550 50  0000 C CNN
+F 1 "330" V 2150 7550 50  0000 C CNN
+F 2 "Resistor_THT:R_Axial_DIN0207_L6.3mm_D2.5mm_P10.16mm_Horizontal" H 2600 7300 50  0001 C CNN
+F 3 "" H 2250 7550 50  0000 C CNN
+	1    2250 7550
 	-1   0    0    1
 $EndComp
@@
 L Device:LED_Small_ALT D30
 U 1 1 582B68A1
-P 2950 7850
-F 0 "D30" H 2950 7993 50  0000 C CNN
-F 1 "LED" H 2950 7736 50  0001 C CNN
-F 2 "LED_THT:LED_D3.0mm" H 2950 7700 50  0001 C CNN
-F 3 "" V 2950 7850 50  0000 C CNN
-	1    2950 7850
+P 2250 7850
+F 0 "D30" H 2250 7993 50  0000 C CNN
+F 1 "LED" H 2250 7736 50  0001 C CNN
+F 2 "LED_THT:LED_D3.0mm" H 2250 7700 50  0001 C CNN
+F 3 "" V 2250 7850 50  0000 C CNN
+	1    2250 7850
 	0    -1   -1   0
 $EndComp
@@
 L power:GND #PWR016
 U 1 1 582B6B6B
-P 2950 8000
-F 0 "#PWR016" H 2950 7750 50  0001 C CNN
-F 1 "GND" H 2950 7850 50  0000 C CNN
-F 2 "" H 2950 8000 50  0000 C CNN
-F 3 "" H 2950 8000 50  0000 C CNN
-	1    2950 8000
+P 2250 8000
+F 0 "#PWR016" H 2250 7750 50  0001 C CNN
+F 1 "GND" H 2250 7850 50  0000 C CNN
+F 2 "" H 2250 8000 50  0000 C CNN
+F 3 "" H 2250 8000 50  0000 C CNN
+	1    2250 8000
 	1    0    0    -1
 $EndComp
@@
 	4250 4300 4150 4400
 Entry Wire Line
-	4150 4300 4050 4400
-Entry Wire Line
-	4050 4300 3950 4400
-Entry Wire Line
 	3950 4300 3850 4400
 Entry Wire Line
@@
 Text Label 3950 3550 3    60   ~ 0
 a3
-Text Label 4050 5400 3    60   ~ 0
+Text Label 3850 5400 3    60   ~ 0
 a4
-Text Label 3850 5400 3    60   ~ 0
-a2
-Text Label 3950 5400 3    60   ~ 0
+Text Label 4250 5400 3    60   ~ 0
 a3
-Text Label 3750 5400 3    60   ~ 0
-a1
 Text Label 3650 5400 3    60   ~ 0
 a0
@@
 Entry Wire Line
 	3650 8250 3550 8350
-Text Label 4350 7050 1    60   ~ 0
+Text Label 4050 7050 1    60   ~ 0
 DB7
-Text Label 4250 7050 1    60   ~ 0
+Text Label 3950 7050 1    60   ~ 0
 DB6
 Text Label 4150 7050 1    60   ~ 0
 DB5
-Text Label 4050 7050 1    60   ~ 0
+Text Label 3850 7050 1    60   ~ 0
 DB4
-Text Label 3950 7050 1    60   ~ 0
+Text Label 4250 7050 1    60   ~ 0
 DB3
-Text Label 3850 7050 1    60   ~ 0
-DB2
-Text Label 3750 7050 1    60   ~ 0
-DB1
 Text Label 4250 2100 1    60   ~ 0
 AB6
@@
 L Bonsai:74540 U6
 U 7 1 5A287D96
-P 2500 7350
-F 0 "U6" H 2600 7450 60  0000 C CNN
-F 1 "74540" H 2650 7200 60  0000 C CNN
-F 2 "Package_DIP:DIP-20_W7.62mm_LongPads" H 2650 7200 60  0001 C CNN
-F 3 "" H 2650 7200 60  0001 C CNN
-	7    2500 7350
+P 1800 7350
+F 0 "U6" H 1900 7450 60  0000 C CNN
+F 1 "74540" H 1950 7200 60  0000 C CNN
+F 2 "Package_DIP:DIP-20_W7.62mm_LongPads" H 1950 7200 60  0001 C CNN
+F 3 "" H 1950 7200 60  0001 C CNN
+	7    1800 7350
 	1    0    0    -1
 $EndComp
@@
 	1    0    0    -1
 $EndComp
-Text GLabel 1100 5800 2    60   Input ~ 0
-enableR
-Text GLabel 1100 5900 2    60   Input ~ 0
-loadIR
+Text GLabel 2050 14600 2    60   Input ~ 0
+~readIR
 Wire Wire Line
 	1200 4000 1250 4000
@@
 Connection ~ 5200 11800
 Wire Wire Line
-	1600 7350 1800 7350
-Wire Wire Line
-	1800 7350 1800 7200
-Connection ~ 1800 7350
+	1150 7350 1350 7350
+Wire Wire Line
+	1350 7350 1350 7200
+Connection ~ 1350 7350
 Wire Wire Line
 	6800 3550 6800 4200
@@
 	4250 6950 4250 8250
 Wire Wire Line
-	2950 7700 2950 7750
-Wire Wire Line
-	2950 7950 2950 8000
+	2250 7700 2250 7750
+Wire Wire Line
+	2250 7950 2250 8000
 Wire Wire Line
 	6100 1650 6200 1650
@@
 Connection ~ 7700 14100
 Wire Wire Line
-	1100 5800 1000 5800
-Wire Wire Line
-	1000 5900 1100 5900
+	2050 14400 2000 14400
+Wire Wire Line
+	1800 14600 2050 14600
 $Comp
 L power:GND #PWR011
@@
 Wire Wire Line
 	8100 14100 8500 14100
-Text Label 4350 5400 3    60   ~ 0
-b1
-Text Label 4250 5400 3    60   ~ 0
+Text Label 3950 5400 3    60   ~ 0
 b0
 Text Label 4150 5400 3    60   ~ 0
@@
 Connection ~ 6100 1650
 Wire Wire Line
-	1800 7350 2150 7350
+	1350 7350 1450 7350
 Wire Wire Line
 	2650 3200 2400 3200
@@
 $EndComp
 Wire Wire Line
-	1800 6800 1800 6900
-Wire Wire Line
-	2800 7350 2950 7350
-Wire Wire Line
-	2950 7400 2950 7350
+	1350 6800 1350 6900
+Wire Wire Line
+	2100 7350 2250 7350
+Wire Wire Line
+	2250 7400 2250 7350
 Wire Wire Line
 	4150 4400 4150 5550
@@
 	1750 11400 1850 11500
 $Comp
-L 74xx_IEEE:7408 U8
+L Bonsai:7408 U8
 U 1 1 5FFF8FCE
 P 3850 10000
@@
 $EndComp
 $Comp
-L 74xx_IEEE:7408 U8
+L Bonsai:7408 U8
 U 3 1 5FFFB7C2
 P 3850 11150
@@
 $EndComp
 $Comp
-L 74xx_IEEE:7408 U8
+L Bonsai:7408 U8
 U 2 1 5FFFC51C
 P 5050 10600
@@
 Connection ~ 10500 14100
 Wire Wire Line
-	2950 7350 4550 7350
+	2250 7350 4550 7350
 Wire Wire Line
 	4550 6950 4550 7350
-Connection ~ 2950 7350
+Connection ~ 2250 7350
 Wire Wire Line
 	3150 4000 4550 4000
@@
 Wire Wire Line
 	8550 12650 8550 11900
-$Comp
-L Connector_Generic:Conn_01x03 J6
-U 1 1 5FC323D8
-P 1600 14600
-F 0 "J6" H 1518 14275 50  0000 C CNN
-F 1 "Conn_01x03" H 1518 14366 50  0000 C CNN
-F 2 "Connector_Molex:Molex_KK-254_AE-6410-03A_1x03_P2.54mm_Vertical" H 1600 14600 50  0001 C CNN
-F 3 "~" H 1600 14600 50  0001 C CNN
-	1    1600 14600
-	-1   0    0    1
-$EndComp
-Text GLabel 2000 14700 2    60   Input ~ 0
-upPC
-Text GLabel 2000 14500 2    60   Input ~ 0
-incPC
-Text GLabel 2000 14600 2    60   Input ~ 0
-incPCz
-Wire Wire Line
-	2000 14700 1800 14700
-Wire Wire Line
-	1800 14500 2000 14500
-Wire Wire Line
-	1800 14600 2000 14600
+Text GLabel 2000 15550 2    60   Input ~ 0
+~upPC
+Text GLabel 2050 14200 2    60   Input ~ 0
+~incPC
+Text GLabel 2050 14000 2    60   Input ~ 0
+~incPCz
+Wire Wire Line
+	2000 15550 1800 15550
 Wire Wire Line
 	1250 4000 1250 3900
@@
 L Connector_Generic:Conn_01x02 J2
 U 1 1 5FD023A3
-P 800 5900
-F 0 "J2" H 718 5575 50  0000 C CNN
-F 1 "Conn_01x02" H 718 5666 50  0000 C CNN
-F 2 "Connector_Molex:Molex_KK-254_AE-6410-02A_1x02_P2.54mm_Vertical" H 800 5900 50  0001 C CNN
-F 3 "~" H 800 5900 50  0001 C CNN
-	1    800  5900
+P 1600 15550
+F 0 "J2" H 1518 15225 50  0000 C CNN
+F 1 "Conn_01x02" H 1518 15316 50  0000 C CNN
+F 2 "Connector_Molex:Molex_KK-254_AE-6410-02A_1x02_P2.54mm_Vertical" H 1600 15550 50  0001 C CNN
+F 3 "~" H 1600 15550 50  0001 C CNN
+	1    1600 15550
 	-1   0    0    1
 $EndComp
@@
 DB7
 Wire Wire Line
-	3950 4400 3950 5550
-Wire Wire Line
-	4050 4400 4050 5550
-Wire Wire Line
-	4250 5550 4250 5350
-Wire Wire Line
-	4250 5350 5600 5350
-Wire Wire Line
-	4350 5550 4350 5200
-Wire Wire Line
-	4350 5200 5600 5200
-Wire Wire Line
 	1450 12850 1400 12850
 Connection ~ 1450 12850
@@
 Wire Wire Line
 	2350 12850 2250 12850
+Text Notes 4750 6300 0    50   ~ 0
+Befehlsregister\n(Instruction Register IR)
+$Comp
+L Connector_Generic:Conn_01x04 J6
+U 1 1 5FA7535B
+P 1600 14500
+F 0 "J6" H 1680 14492 50  0000 L CNN
+F 1 "Conn_01x04" H 1680 14401 50  0000 L CNN
+F 2 "Connector_Molex:Molex_KK-254_AE-6410-04A_1x04_P2.54mm_Vertical" H 1600 14500 50  0001 C CNN
+F 3 "~" H 1600 14500 50  0001 C CNN
+	1    1600 14500
+	-1   0    0    1
+$EndComp
+Text GLabel 2050 14400 2    60   Input ~ 0
+~writeIR
+Wire Wire Line
+	1800 14500 2000 14500
+Wire Wire Line
+	2000 14500 2000 14400
+Wire Wire Line
+	1800 14400 1950 14400
+Wire Wire Line
+	1950 14400 1950 14200
+Wire Wire Line
+	1950 14200 2050 14200
+Wire Wire Line
+	1800 14300 1900 14300
+Wire Wire Line
+	1900 14300 1900 14000
+Wire Wire Line
+	1900 14000 2050 14000
+Text Notes 1900 13850 0    50   ~ 0
+Steuersignale\nvom Steuerwerk
+Text Notes 1500 15100 0    50   ~ 0
+Signal für den PC
+Text GLabel 1150 7350 0    60   Input ~ 0
+~readIR
+Text Label 3750 5400 3    60   ~ 0
+a2
+Text Label 4350 7050 1    60   ~ 0
+DB1
+Text Label 3750 7050 1    60   ~ 0
+DB2
+Text Label 4050 5400 3    60   ~ 0
+b1
+Text Label 4350 5400 3    60   ~ 0
+a1
+Wire Wire Line
+	4350 5550 4350 4400
+Wire Wire Line
+	4250 5550 4250 4400
+Entry Wire Line
+	4350 4400 4450 4300
+Entry Wire Line
+	4250 4400 4350 4300
+Wire Wire Line
+	3950 5350 3950 5550
+Wire Wire Line
+	5600 5350 3950 5350
+Wire Wire Line
+	4050 5550 4050 5200
+Wire Wire Line
+	4050 5200 5600 5200
 Wire Bus Line
 	1750 12000 2450 12000
 Wire Bus Line
+	1750 8350 1750 12000
+Wire Bus Line
 	1850 1850 1850 2900
 Wire Bus Line
-	1750 8350 1750 12000
+	1850 1850 4250 1850
 Wire Bus Line
 	1750 8350 4250 8350
 Wire Bus Line
-	1850 1850 4250 1850
-Wire Bus Line
-	3650 4300 6700 4300
+	3750 4300 6700 4300
 $EndSCHEMATC
