File: Befehle.sch (KiCad schematic (older format))
At the start: 77 parts, among them J1 Conn_02x10_Odd_Even, J2 Conn_01x02, J3 Conn_01x04, J4 Conn_02x10_Odd_Even, J5 Conn_01x02, J6 Conn_01x04, U1 74LS14, U2 74LS541, U3 74LS540, U4 74LS139, U5 74LS373, U6 74540, U7 7402, U8 7408, U9 7400

Commit message: Befehle: Platine fertig (TODO: Kontrolle)
Parts:
- added unit 2 of U4
- added unit 5 of U6
- added unit 6 of U6
- added unit 3 of U9
- added unit 4 of U9
- U2, U3, U5, U6: footprint Package_DIP:DIP-20_W7.62mm_LongPads -> Package_DIP:DIP-20_W7.62mm_Socket_LongPads
- U9: symbol 74xx_IEEE:7400 -> Bonsai:7400
Connections:
- net labels removed: a6, a7
- wire segments 317 -> 322
Changed lines of the file:
@@
 F 0 "U5" V 4150 6300 50  0000 C CNN
 F 1 "74LS373" V 4250 6300 50  0000 C CNN
-F 2 "Package_DIP:DIP-20_W7.62mm_LongPads" V 4150 6250 50  0001 C CNN
+F 2 "Package_DIP:DIP-20_W7.62mm_Socket_LongPads" V 4150 6250 50  0001 C CNN
 F 3 "" H 4150 6250 50  0000 C CNN
 	1    4150 6250
@@
 F 0 "U2" H 4150 2084 50  0000 C CNN
 F 1 "74LS541" H 4150 2175 50  0000 C CNN
-F 2 "Package_DIP:DIP-20_W7.62mm_LongPads" V 4350 2850 50  0001 C CNN
+F 2 "Package_DIP:DIP-20_W7.62mm_Socket_LongPads" V 4350 2850 50  0001 C CNN
 F 3 "" H 4150 2850 50  0000 C CNN
 	1    4150 2850
@@
 F 0 "U3" H 6600 2084 50  0000 C CNN
 F 1 "74LS540" H 6600 2175 50  0000 C CNN
-F 2 "Package_DIP:DIP-20_W7.62mm_LongPads" V 6800 2850 50  0001 C CNN
+F 2 "Package_DIP:DIP-20_W7.62mm_Socket_LongPads" V 6800 2850 50  0001 C CNN
 F 3 "" H 6600 2850 50  0000 C CNN
 	1    6600 2850
@@
 a2
 Text Label 6100 3550 3    60   ~ 0
-a7
+b1
 Text Label 6400 3550 3    60   ~ 0
 a4
@@
 a5
 Text Label 6200 3550 3    60   ~ 0
-a6
+b0
 Text Label 6500 3550 3    60   ~ 0
 a3
@@
 F 0 "U6" H 1900 7450 60  0000 C CNN
 F 1 "74540" H 1950 7200 60  0000 C CNN
-F 2 "Package_DIP:DIP-20_W7.62mm_LongPads" H 1950 7200 60  0001 C CNN
+F 2 "Package_DIP:DIP-20_W7.62mm_Socket_LongPads" H 1950 7200 60  0001 C CNN
 F 3 "" H 1950 7200 60  0001 C CNN
 	7    1800 7350
@@
 F 0 "U6" H 5750 10300 60  0000 C CNN
 F 1 "74540" H 5800 10050 60  0000 C CNN
-F 2 "Package_DIP:DIP-20_W7.62mm_LongPads" H 5800 10050 60  0001 C CNN
+F 2 "Package_DIP:DIP-20_W7.62mm_Socket_LongPads" H 5800 10050 60  0001 C CNN
 F 3 "" H 5800 10050 60  0001 C CNN
 	8    5650 10200
@@
 F 0 "U6" H 5400 14100 60  0000 C CNN
 F 1 "74540" H 5450 14000 60  0000 C CNN
-F 2 "Package_DIP:DIP-20_W7.62mm_LongPads" H 5550 14850 60  0001 C CNN
+F 2 "Package_DIP:DIP-20_W7.62mm_Socket_LongPads" H 5550 14850 60  0001 C CNN
 F 3 "" H 5600 13900 60  0001 C CNN
 	9    5450 14050
@@
 Wire Wire Line
 	5650 9900 5650 9850
-Text Notes 9350 1650 0    50   ~ 0
-ungenutzte Gatter
 $Comp
 L allBonsaiSymbolLibs:C_Small C10
@@
 F 0 "U6" V 9000 6800 60  0000 C CNN
 F 1 "74540" V 9150 6950 60  0000 C CNN
-F 2 "Package_DIP:DIP-20_W7.62mm_LongPads" H 9350 6550 60  0001 C CNN
+F 2 "Package_DIP:DIP-20_W7.62mm_Socket_LongPads" H 9350 6550 60  0001 C CNN
 F 3 "" H 9350 6550 60  0001 C CNN
 	1    9200 6700
@@
 F 0 "U6" V 8500 6800 60  0000 C CNN
 F 1 "74540" H 8850 6550 60  0001 C CNN
-F 2 "Package_DIP:DIP-20_W7.62mm_LongPads" H 8850 6550 60  0001 C CNN
+F 2 "Package_DIP:DIP-20_W7.62mm_Socket_LongPads" H 8850 6550 60  0001 C CNN
 F 3 "" H 8850 6550 60  0001 C CNN
 	2    8700 6700
@@
 F 0 "U6" V 8000 6800 60  0000 C CNN
 F 1 "74540" H 8350 6550 60  0001 C CNN
-F 2 "Package_DIP:DIP-20_W7.62mm_LongPads" H 8350 6550 60  0001 C CNN
+F 2 "Package_DIP:DIP-20_W7.62mm_Socket_LongPads" H 8350 6550 60  0001 C CNN
 F 3 "" H 8350 6550 60  0001 C CNN
 	3    8200 6700
@@
 F 0 "U6" V 7500 6800 60  0000 C CNN
 F 1 "74540" H 7850 6550 60  0001 C CNN
-F 2 "Package_DIP:DIP-20_W7.62mm_LongPads" H 7800 7500 60  0001 C CNN
+F 2 "Package_DIP:DIP-20_W7.62mm_Socket_LongPads" H 7800 7500 60  0001 C CNN
 F 3 "" H 7850 6550 60  0001 C CNN
 	4    7700 6700
@@
 Connection ~ 5650 10600
 $Comp
-L 74xx_IEEE:7400 U9
+L Bonsai:7400 U9
 U 1 1 5FF4C3E3
 P 7450 11700
@@
 $EndComp
 $Comp
-L 74xx_IEEE:7400 U9
+L Bonsai:7400 U9
 U 2 1 5FF6CD43
 P 5850 11800
@@
 Wire Wire Line
 	4050 5200 5600 5200
+$Comp
+L Bonsai:7400 U9
+U 3 1 5FD25346
+P 10200 3600
+F 0 "U9" H 10200 4066 50  0000 C CNN
+F 1 "7400" H 10200 3975 50  0000 C CNN
+F 2 "Package_DIP:DIP-14_W7.62mm_Socket_LongPads" H 10200 3600 50  0001 C CNN
+F 3 "" H 10200 3600 50  0001 C CNN
+	3    10200 3600
+	1    0    0    -1
+$EndComp
+$Comp
+L Bonsai:7400 U9
+U 4 1 5FD25F35
+P 10200 4300
+F 0 "U9" H 10200 4766 50  0000 C CNN
+F 1 "7400" H 10200 4675 50  0000 C CNN
+F 2 "Package_DIP:DIP-14_W7.62mm_Socket_LongPads" H 10200 4300 50  0001 C CNN
+F 3 "" H 10200 4300 50  0001 C CNN
+	4    10200 4300
+	1    0    0    -1
+$EndComp
+Wire Wire Line
+	9700 3500 9700 3700
+Wire Wire Line
+	9700 4200 9700 4400
+$Comp
+L power:VCC #PWR0101
+U 1 1 5FD8091C
+P 9700 3500
+F 0 "#PWR0101" H 9700 3350 50  0001 C CNN
+F 1 "VCC" H 9700 3650 50  0000 C CNN
+F 2 "" H 9700 3500 50  0000 C CNN
+F 3 "" H 9700 3500 50  0000 C CNN
+	1    9700 3500
+	1    0    0    -1
+$EndComp
+Connection ~ 9700 3500
+$Comp
+L power:VCC #PWR0102
+U 1 1 5FD814A1
+P 9700 4200
+F 0 "#PWR0102" H 9700 4050 50  0001 C CNN
+F 1 "VCC" H 9700 4350 50  0000 C CNN
+F 2 "" H 9700 4200 50  0000 C CNN
+F 3 "" H 9700 4200 50  0000 C CNN
+	1    9700 4200
+	1    0    0    -1
+$EndComp
+Connection ~ 9700 4200
+$Comp
+L Bonsai:74540 U6
+U 5 1 5FDF6728
+P 8700 2300
+F 0 "U6" V 8500 2400 60  0000 C CNN
+F 1 "74540" H 8850 2150 60  0001 C CNN
+F 2 "Package_DIP:DIP-20_W7.62mm_Socket_LongPads" H 8800 3100 60  0001 C CNN
+F 3 "" H 8850 2150 60  0001 C CNN
+	5    8700 2300
+	0    1    1    0
+$EndComp
+$Comp
+L Bonsai:74540 U6
+U 6 1 5FDF73E3
+P 8400 2300
+F 0 "U6" V 8200 2400 60  0000 C CNN
+F 1 "74540" H 8550 2150 60  0001 C CNN
+F 2 "Package_DIP:DIP-20_W7.62mm_Socket_LongPads" H 8500 3100 60  0001 C CNN
+F 3 "" H 8550 2150 60  0001 C CNN
+	6    8400 2300
+	0    1    1    0
+$EndComp
+Connection ~ 8400 1950
+Wire Wire Line
+	8400 1950 8700 1950
+$Comp
+L power:VCC #PWR0103
+U 1 1 5FE3BBB2
+P 8400 1950
+F 0 "#PWR0103" H 8400 1800 50  0001 C CNN
+F 1 "VCC" H 8400 2100 50  0000 C CNN
+F 2 "" H 8400 1950 50  0000 C CNN
+F 3 "" H 8400 1950 50  0000 C CNN
+	1    8400 1950
+	1    0    0    -1
+$EndComp
+$Comp
+L allBonsaiSymbolLibs:74LS139-74xx U4
+U 2 1 5FE911F7
+P 10000 1200
+F 0 "U4" H 10050 1200 50  0000 R CNN
+F 1 "74LS139" H 10150 1350 50  0000 R CNN
+F 2 "Package_DIP:DIP-16_W7.62mm_Socket_LongPads" H 9600 1200 50  0001 C CNN
+F 3 "" H 10000 1200 50  0000 C CNN
+	2    10000 1200
+	1    0    0    -1
+$EndComp
+Text Notes 8050 700  0    50   ~ 0
+ungenutzte Gatter
+Wire Wire Line
+	9150 950  9150 1100
 Wire Bus Line
 	1750 12000 2450 12000
@@
 Wire Bus Line
 	3750 4300 6700 4300
+Connection ~ 9150 1100
+Wire Wire Line
+	9150 1100 9150 1450
+$Comp
+L power:VCC #PWR0104
+U 1 1 5FEB1B47
+P 9150 950
+F 0 "#PWR0104" H 9150 800 50  0001 C CNN
+F 1 "VCC" H 9150 1100 50  0000 C CNN
+F 2 "" H 9150 950 50  0000 C CNN
+F 3 "" H 9150 950 50  0000 C CNN
+	1    9150 950
+	1    0    0    -1
+$EndComp
+Connection ~ 9150 950
 $EndSCHEMATC

Commit message: Befehle: alle versteckten Pins durch sichtbare Pins ersetzt; VCC und GND an jedem IC explizit im Schaltplan angeschlossen.
Parts:
- added unit 7 of U1
- added unit 3 of U4
- added unit 5 of U7
- added unit 5 of U8
- added unit 5 of U9
- U7: symbol 74xx_IEEE:7402 -> Bonsai:7402
- U8: symbol 74xx_IEEE:7408 -> Bonsai:7408
Connections:
- wire segments 322 -> 338

Commit message: Befehle und Steuerwerk: - Kleinkram - gerber rev 2.0 für Bestellung exportiert
Parts:
- U4: value 74LS139 -> 74HC139
- U5: value 74LS373 -> 74HCT373
- U6: value 74540 -> 74HC540
- U7: value 7402 -> 74HCT02
Connections:
- no-connect marks 0 -> 10
Changed lines of the file:
@@
 P 4150 6250
 F 0 "U5" V 4150 6300 50  0000 C CNN
-F 1 "74LS373" V 4250 6300 50  0000 C CNN
+F 1 "74HCT373" V 4250 6300 50  0000 C CNN
 F 2 "Package_DIP:DIP-20_W7.62mm_Socket_LongPads" V 4150 6250 50  0001 C CNN
 F 3 "" H 4150 6250 50  0000 C CNN
@@
 P 1800 7350
 F 0 "U6" H 1900 7450 60  0000 C CNN
-F 1 "74540" H 1950 7200 60  0000 C CNN
+F 1 "74HC540" H 1950 7200 60  0000 C CNN
 F 2 "Package_DIP:DIP-20_W7.62mm_Socket_LongPads" H 1950 7200 60  0001 C CNN
 F 3 "" H 1950 7200 60  0001 C CNN
@@
 L allBonsaiSymbolLibs:R-device R17
 U 1 1 582AA727
-P 5650 9700
-F 0 "R17" V 5650 9700 50  0000 C CNN
-F 1 "330" V 5550 9700 50  0000 C CNN
-F 2 "Resistor_THT:R_Axial_DIN0207_L6.3mm_D2.5mm_P10.16mm_Horizontal" V 5850 8900 50  0001 C CNN
-F 3 "" H 5650 9700 50  0000 C CNN
-	1    5650 9700
+P 5650 9650
+F 0 "R17" V 5650 9650 50  0000 C CNN
+F 1 "330" V 5550 9650 50  0000 C CNN
+F 2 "Resistor_THT:R_Axial_DIN0207_L6.3mm_D2.5mm_P10.16mm_Horizontal" V 5850 8850 50  0001 C CNN
+F 3 "" H 5650 9650 50  0000 C CNN
+	1    5650 9650
 	1    0    0    -1
 $EndComp
@@
 L Device:LED_Small_ALT D31
 U 1 1 582AC971
-P 5650 9400
-F 0 "D31" H 5650 9500 50  0000 C CNN
-F 1 "LED" H 5650 9286 50  0001 C CNN
-F 2 "LED_THT:LED_D3.0mm" V 5800 9400 50  0001 C CNN
-F 3 "" V 5650 9400 50  0000 C CNN
-	1    5650 9400
+P 5650 9350
+F 0 "D31" H 5650 9450 50  0000 C CNN
+F 1 "LED" H 5650 9236 50  0001 C CNN
+F 2 "LED_THT:LED_D3.0mm" V 5800 9350 50  0001 C CNN
+F 3 "" V 5650 9350 50  0000 C CNN
+	1    5650 9350
 	0    -1   -1   0
 $EndComp
@@
 L power:VCC #PWR017
 U 1 1 582B09F9
-P 5650 9250
-F 0 "#PWR017" H 5650 9100 50  0001 C CNN
-F 1 "VCC" H 5650 9400 50  0000 C CNN
-F 2 "" H 5650 9250 50  0000 C CNN
-F 3 "" H 5650 9250 50  0000 C CNN
-	1    5650 9250
-	1    0    0    -1
-$EndComp
-Wire Wire Line
-	5650 9550 5650 9500
-Wire Wire Line
-	5650 9300 5650 9250
+P 5650 9200
+F 0 "#PWR017" H 5650 9050 50  0001 C CNN
+F 1 "VCC" H 5650 9350 50  0000 C CNN
+F 2 "" H 5650 9200 50  0000 C CNN
+F 3 "" H 5650 9200 50  0000 C CNN
+	1    5650 9200
+	1    0    0    -1
+$EndComp
+Wire Wire Line
+	5650 9500 5650 9450
+Wire Wire Line
+	5650 9250 5650 9200
 $Comp
 L Bonsai:74540 U6
 U 8 1 5A2905C7
-P 5650 10200
-F 0 "U6" H 5750 10300 60  0000 C CNN
-F 1 "74540" H 5800 10050 60  0000 C CNN
-F 2 "Package_DIP:DIP-20_W7.62mm_Socket_LongPads" H 5800 10050 60  0001 C CNN
-F 3 "" H 5800 10050 60  0001 C CNN
-	8    5650 10200
+P 5650 10150
+F 0 "U6" H 5750 10250 60  0000 C CNN
+F 1 "74HC540" H 5800 10000 60  0000 C CNN
+F 2 "Package_DIP:DIP-20_W7.62mm_Socket_LongPads" H 5800 10000 60  0001 C CNN
+F 3 "" H 5800 10000 60  0001 C CNN
+	8    5650 10150
 	0    -1   -1   0
 $EndComp
@@
 P 5300 14500
 F 0 "U6" H 5200 14950 60  0000 C CNN
-F 1 "74540" H 5300 14450 60  0000 C CNN
+F 1 "74HC540" H 5300 14450 60  0000 C CNN
 F 2 "Package_DIP:DIP-20_W7.62mm_Socket_LongPads" H 5400 15300 60  0001 C CNN
 F 3 "" H 5450 14350 60  0001 C CNN
@@
 P 2650 11400
 F 0 "U7" H 2650 11600 50  0000 C CNN
-F 1 "7402" H 2650 11200 50  0000 C CNN
+F 1 "74HCT02" H 2650 11200 50  0000 C CNN
 F 2 "Package_DIP:DIP-14_W7.62mm_Socket_LongPads" H 2650 11400 50  0001 C CNN
 F 3 "" H 2650 11400 50  0001 C CNN
@@
 P 2650 10850
 F 0 "U7" H 2650 11050 50  0000 C CNN
-F 1 "7402" H 2650 10650 50  0000 C CNN
+F 1 "74HCT02" H 2650 10650 50  0000 C CNN
 F 2 "Package_DIP:DIP-14_W7.62mm_Socket_LongPads" H 2650 10850 50  0001 C CNN
 F 3 "" H 2650 10850 50  0001 C CNN
@@
 P 2650 10300
 F 0 "U7" H 2650 10450 50  0000 C CNN
-F 1 "7402" H 2650 10100 50  0000 C CNN
+F 1 "74HCT02" H 2650 10100 50  0000 C CNN
 F 2 "Package_DIP:DIP-14_W7.62mm_Socket_LongPads" H 2650 10300 50  0001 C CNN
 F 3 "" H 2650 10300 50  0001 C CNN
@@
 P 2650 9700
 F 0 "U7" H 2650 9850 50  0000 C CNN
-F 1 "7402" H 2650 9500 50  0000 C CNN
+F 1 "74HCT02" H 2650 9500 50  0000 C CNN
 F 2 "Package_DIP:DIP-14_W7.62mm_Socket_LongPads" H 2650 9700 50  0001 C CNN
 F 3 "" H 2650 9700 50  0001 C CNN
@@
 Nullentdeckungslogik
 Wire Wire Line
-	5650 9900 5650 9850
+	5650 9850 5650 9800
 $Comp
 L allBonsaiSymbolLibs:C_Small C10
@@
 P 6450 5450
 F 0 "U4" H 6500 5450 50  0000 R CNN
-F 1 "74LS139" H 6600 5600 50  0000 R CNN
+F 1 "74HC139" H 6600 5600 50  0000 R CNN
 F 2 "Package_DIP:DIP-16_W7.62mm_Socket_LongPads" H 6050 5450 50  0001 C CNN
 F 3 "" H 6450 5450 50  0000 C CNN
@@
 P 9200 6700
 F 0 "U6" V 9000 6800 60  0000 C CNN
-F 1 "74540" V 9150 6950 60  0000 C CNN
+F 1 "74HC540" V 9150 6950 60  0000 C CNN
 F 2 "Package_DIP:DIP-20_W7.62mm_Socket_LongPads" H 9350 6550 60  0001 C CNN
 F 3 "" H 9350 6550 60  0001 C CNN
@@
 P 8700 6700
 F 0 "U6" V 8500 6800 60  0000 C CNN
-F 1 "74540" H 8850 6550 60  0001 C CNN
+F 1 "74HC540" H 8850 6550 60  0001 C CNN
 F 2 "Package_DIP:DIP-20_W7.62mm_Socket_LongPads" H 8850 6550 60  0001 C CNN
 F 3 "" H 8850 6550 60  0001 C CNN
@@
 P 8200 6700
 F 0 "U6" V 8000 6800 60  0000 C CNN
-F 1 "74540" H 8350 6550 60  0001 C CNN
+F 1 "74HC540" H 8350 6550 60  0001 C CNN
 F 2 "Package_DIP:DIP-20_W7.62mm_Socket_LongPads" H 8350 6550 60  0001 C CNN
 F 3 "" H 8350 6550 60  0001 C CNN
@@
 P 7700 6700
 F 0 "U6" V 7500 6800 60  0000 C CNN
-F 1 "74540" H 7850 6550 60  0001 C CNN
+F 1 "74HC540" H 7850 6550 60  0001 C CNN
 F 2 "Package_DIP:DIP-20_W7.62mm_Socket_LongPads" H 7800 7500 60  0001 C CNN
 F 3 "" H 7850 6550 60  0001 C CNN
@@
 	5550 5700 5550 5750
 Wire Wire Line
-	5650 10600 5650 10550
+	5650 10600 5650 10500
 Wire Wire Line
 	5600 10600 5650 10600
@@
 P 8700 2300
 F 0 "U6" V 8500 2400 60  0000 C CNN
-F 1 "74540" H 8850 2150 60  0001 C CNN
+F 1 "74HC540" H 8850 2150 60  0001 C CNN
 F 2 "Package_DIP:DIP-20_W7.62mm_Socket_LongPads" H 8800 3100 60  0001 C CNN
 F 3 "" H 8850 2150 60  0001 C CNN
@@
 P 8400 2300
 F 0 "U6" V 8200 2400 60  0000 C CNN
-F 1 "74540" H 8550 2150 60  0001 C CNN
+F 1 "74HC540" H 8550 2150 60  0001 C CNN
 F 2 "Package_DIP:DIP-20_W7.62mm_Socket_LongPads" H 8500 3100 60  0001 C CNN
 F 3 "" H 8550 2150 60  0001 C CNN
@@
 P 10000 1200
 F 0 "U4" H 10050 1200 50  0000 R CNN
-F 1 "74LS139" H 10150 1350 50  0000 R CNN
+F 1 "74HC139" H 10150 1350 50  0000 R CNN
 F 2 "Package_DIP:DIP-16_W7.62mm_Socket_LongPads" H 9600 1200 50  0001 C CNN
 F 3 "" H 10000 1200 50  0000 C CNN
@@
 P 3100 15500
 F 0 "U7" H 3100 15700 50  0000 C CNN
-F 1 "7402" H 3100 15300 50  0000 C CNN
+F 1 "74HCT02" H 3100 15300 50  0000 C CNN
 F 2 "Package_DIP:DIP-14_W7.62mm_Socket_LongPads" H 3100 15500 50  0001 C CNN
 F 3 "" H 3100 15500 50  0001 C CNN
@@
 P 6300 15250
 F 0 "U4" H 6350 15250 50  0000 R CNN
-F 1 "74LS139" H 6450 15400 50  0000 R CNN
+F 1 "74HC139" H 6450 15400 50  0000 R CNN
 F 2 "Package_DIP:DIP-16_W7.62mm_Socket_LongPads" H 5900 15250 50  0001 C CNN
 F 3 "" H 6300 15250 50  0000 C CNN
@@
 Wire Wire Line
 	4550 15450 4550 15400
+NoConn ~ 10850 900
+NoConn ~ 10850 1100
+NoConn ~ 10850 1300
+NoConn ~ 10850 1500
+NoConn ~ 8400 2600
+NoConn ~ 8700 2600
+NoConn ~ 10350 2000
+NoConn ~ 10700 3600
+NoConn ~ 10700 4450
+NoConn ~ 1800 15450
 Wire Bus Line
 	1750 12000 2450 12000
