File: Akku.kicad_pcb (KiCad board)
At the start: 2 copper layers, 100 x 160 mm, 51 parts, among them J1 +/- Stecker, J2 load/up, J3 down/en/clear, P7 CONN_02X10, P8 CONN_02X10, P9 CONN_02X10, SW1 UP_Bonsai_SWITCH_INV, SW2 DOWN_Bonsai_SWITCH_INV, SW3 CLR_Bonsai_SWITCH_INV, U1 74HC14, U2 7400, U4 7408, U5 74LS193, U6 74LS541, U7 74LS193, U8 74LS540

Commit message: Akku: Bauteilwerte ergänzt
Parts:
- C1, C2, C3: value C -> 100n
- R12: value R -> 470
- R13, R15, R16, R17, R18, R19, R20, R21: value R -> 330
- R14: value R -> 150
- R2, R3: value R -> 4k7
Connections:
- D7 pad 1: GND -> Net-(D7-Pad1)
- RPB1 pad 2: (no net) -> RPB1
- SW1 pad 6: (no net) -> Net-(SW1-Pad6)
- SW2 pad 6: (no net) -> Net-(SW2-Pad6)
- U5 pad 12: (no net) -> Net-(U5-Pad12)
- U5 pad 13: (no net) -> Net-(U5-Pad13)

Commit message: Akku: Schaltungen zum entprellen der Taster gleichartig angeordnet
Parts:
- R10, R11, R9: value R -> 150

Commit message: Backup vor Umbennung von Netzen
Parts:
- removed G***: LOGO, allBonsaiFootprintsLibs:agi5
- moved D1 0.64 mm to (64.1, 119.4)
Connections:
- net /a0 renamed /B0
- net /a1 renamed /B1
- net /a2 renamed /B2
- net /a3 renamed /B3
- net /a4 renamed /B4
- net /a5 renamed /B5
- net /a6 renamed /B6
- net /a7 renamed /B7
- D7 pad 1: Net-(D7-Pad1) -> GND
Routing:
- net GND: track 655.5 -> 656.1 mm

Commit message: Akku/PC: Schaltplan mit Bussen gezeichnet; Netze der Busse sinnvoll benannt
Connections:
- net Net-(U5-Pad2) renamed /Bi5
- net Net-(U5-Pad3) renamed /Bi4
- net Net-(U5-Pad6) renamed /Bi6
- net Net-(U5-Pad7) renamed /Bi7
- net Net-(U6-Pad6) renamed /Bi3
- net Net-(U6-Pad7) renamed /Bi2
- net Net-(U6-Pad8) renamed /Bi1
- net Net-(U6-Pad9) renamed /Bi0
- P7 pad 12: /B7 -> /B0
- P7 pad 13: /B6 -> /B1
- P7 pad 14: /B5 -> /B2
- P7 pad 15: /B4 -> /B3
- P7 pad 16: /B3 -> /B4
- P7 pad 17: /B2 -> /B5
- P7 pad 18: /B1 -> /B6
- P7 pad 19: /B0 -> /B7
- P8 pad 12: /B7 -> /B0
- P8 pad 13: /B6 -> /B1
- P8 pad 14: /B5 -> /B2
- P8 pad 15: /B4 -> /B3
- P8 pad 16: /B3 -> /B4
- P8 pad 17: /B2 -> /B5
- P8 pad 18: /B1 -> /B6
- P8 pad 19: /B0 -> /B7
- P9 pad 12: /B7 -> /B0
- P9 pad 13: /B6 -> /B1
- P9 pad 14: /B5 -> /B2
- P9 pad 15: /B4 -> /B3
- P9 pad 16: /B3 -> /B4
- P9 pad 17: /B2 -> /B5
- P9 pad 18: /B1 -> /B6
- P9 pad 19: /B0 -> /B7
- U5 pad 1: /B2 -> /B5
- U5 pad 10: /B1 -> /B6
- U5 pad 15: /B3 -> /B4
- U5 pad 9: /B0 -> /B7
- U6 pad 11: /B7 -> /B0
- U6 pad 12: /B6 -> /B1
- U6 pad 13: /B5 -> /B2
- U6 pad 14: /B4 -> /B3
- U6 pad 15: /B3 -> /B4
- U6 pad 16: /B2 -> /B5
- U6 pad 17: /B1 -> /B6
- U6 pad 18: /B0 -> /B7
- U7 pad 1: /B6 -> /B1
- U7 pad 10: /B5 -> /B2
- U7 pad 15: /B7 -> /B0
- U7 pad 9: /B4 -> /B3
Routing:
- net /B7: track 303.7 -> 204.4 mm
- net /B0: track 204.4 -> 303.7 mm
- net /B6: track 302.3 -> 215.7 mm
- net /B1: track 215.7 -> 302.3 mm
- net /B4: track 262.0 -> 246.2 mm
- net /B3: track 246.2 -> 262.0 mm
- net /B5: track 272.5 -> 268.1 mm
- net /B2: track 268.1 -> 272.5 mm

Commit message: Akku/PC: Schaltplan aufgeräumt
Connections:
- net CLR renamed /clr
- net Net-(U1-Pad11) renamed /up_i
- net Net-(U1-Pad13) renamed /down_i
- net Net-(U5-Pad4) renamed /downCarry
- net Net-(U5-Pad5) renamed /upCarry
- net RPB4 renamed /~load

Commit message: Steuerwerk 2.0 gerber exportiert
Parts:
- U1, U2, U4: footprint Housings_DIP:DIP-14_W7.62mm_LongPads -> Package_DIP:DIP-14_W7.62mm_Socket_LongPads
- U5, U7: footprint Housings_DIP:DIP-16_W7.62mm_LongPads -> Package_DIP:DIP-16_W7.62mm_Socket_LongPads
- U6, U8: footprint Housings_DIP:DIP-20_W7.62mm_LongPads -> Package_DIP:DIP-20_W7.62mm_Socket_LongPads

Commit message: Akku weitergebaut
Parts:
- removed RPB1: R_PACK4BUSSED, tg_locallibs:R_Array_SIP5
- added J2: Conn_01x02, Connector_Molex:Molex_KK-254_AE-6410-02A_1x02_P2.54mm_Vertical, F.Cu at (53.8, 72.6)
- added J3: Conn_01x04, Connector_Molex:Molex_KK-254_AE-6410-04A_1x04_P2.54mm_Vertical, F.Cu at (146.1, 209.0)
- added J4: Conn_01x02, Connector_Molex:Molex_KK-254_AE-6410-02A_1x02_P2.54mm_Vertical, F.Cu at (146.1, 223.5)
- added R1: 4k7, Resistor_THT:R_Axial_DIN0207_L6.3mm_D2.5mm_P10.16mm_Horizontal, F.Cu at (146.8, 182.8)
- added R4: 4k7, Resistor_THT:R_Axial_DIN0207_L6.3mm_D2.5mm_P10.16mm_Horizontal, F.Cu at (146.8, 186.8)
- added R5: 4k7, Resistor_THT:R_Axial_DIN0207_L6.3mm_D2.5mm_P10.16mm_Horizontal, F.Cu at (146.8, 190.9)
- SW1: value UP_Bonsai_SWITCH_INV -> Digitast; footprint allBonsaiFootprintsLibs:SW_PUSH_LCD_E3_SAxxxx_tg_V2 -> bonsai:Switch_Digitast
- SW2: value DOWN_Bonsai_SWITCH_INV -> Digitast; footprint allBonsaiFootprintsLibs:SW_PUSH_LCD_E3_SAxxxx_tg_V2 -> bonsai:Switch_Digitast
- SW3: value CLR_Bonsai_SWITCH_INV -> Digitast; footprint allBonsaiFootprintsLibs:SW_PUSH_LCD_E3_SAxxxx_tg_V2 -> bonsai:Switch_Digitast
Connections:
- net RPB2 renamed ^down
- net RPB3 renamed ^up
- SW1 pad 6: Net-(SW1-Pad6) -> (no net)
- SW2 pad 6: Net-(SW2-Pad6) -> (no net)
- SW3 pad 6: GND -> (no net)
Routing:
- net ^up: track 82.8 -> 77.7 mm
- net GND: track 656.1 -> 652.4 mm

Commit message: Akku weitergebaut
Parts:
- removed the J2 at (134.1, 208.5)
- removed the J3 at (134.1, 221.7)
- removed P7, P8, P9: CONN_02X10, allBonsaiFootprintsLibs:Pin_Header_Straight_2x10_Pitch2.00mmBonsai.pretty
- added J5: Conn_02x10_Odd_Even, Connector_PinHeader_2.54mm:PinHeader_2x10_P2.54mm_Vertical, F.Cu at (45.7, 90.2)
- added J6: Conn_02x10_Odd_Even, Connector_PinHeader_2.54mm:PinHeader_2x10_P2.54mm_Vertical, F.Cu at (127.0, 82.5)
- D1, D2, D3, D7: footprint LEDs:LED_D5.0mm_FlatTop -> LED_THT:LED_D3.0mm
- D10, D11, D12, D4, D5, D6, D8, D9: footprint LEDs:LED-3MM -> LED_THT:LED_D3.0mm
- J1: value +/- Stecker -> Conn_02x10_Odd_Even; footprint 2PinTerminalBlocktg -> Connector_PinHeader_2.54mm:PinHeader_2x10_P2.54mm_Vertical
- R10, R11, R12, R13, R14, R15, R16, R17, R18, R19, R2, R20, R21, R3, R9: footprint Resistors_ThroughHole:R_Axial_DIN0207_L6.3mm_D2.5mm_P10.16mm_Horizontal -> Resistor_THT:R_Axial_DIN0207_L6.3mm_D2.5mm_P10.16mm_Horizontal
- moved J1 77.1 mm to (132.1, 90.2)
Connections:
- J1 pad 1: VCC -> GND
Routing:
- net /B6: track 215.7 -> 210.1 mm
Other:
- net class Power: clearance 0.3 -> 0.2
- rule pad_to_mask_clearance: 0.2 -> 0.08
- rule solder_mask_min_width: 0.25 -> 0.254
- rule trace_min: 0.2 -> 0.15
