File: Akku.kicad_pcb (KiCad board)
At the start: 2 copper layers, 100 x 160 mm, 52 parts, among them J1 Conn_02x10_Odd_Even, J2 Conn_01x02, J3 Conn_01x04, J4 Conn_01x02, J5 Conn_02x10_Odd_Even, J6 Conn_02x10_Odd_Even, SW1 Digitast, SW2 Digitast, SW3 Digitast, U1 74HC14, U2 7400, U4 7408, U5 74LS193, U6 74LS541, U7 74LS193, U8 74LS540

Commit message: akku weitergebaut
Parts:
- added C4: CP, Capacitor_THT:CP_Radial_D8.0mm_P2.50mm, F.Cu at (162.3, 164.8)
- added C5: 100n, Capacitor_THT:C_Disc_D10.0mm_W2.5mm_P5.00mm, F.Cu at (150.3, 158.0)
- added C6: 100n, Capacitor_THT:C_Disc_D10.0mm_W2.5mm_P5.00mm, F.Cu at (150.3, 162.1)
- added C7: 100n, Capacitor_THT:C_Disc_D10.0mm_W2.5mm_P5.00mm, F.Cu at (161.9, 158.0)
- added C8: 100n, Capacitor_THT:C_Disc_D10.0mm_W2.5mm_P5.00mm, F.Cu at (150.3, 166.1)
- C1, C2, C3: footprint allBonsaiFootprintsLibs:C_Disc_D10.0mm_W2.5mm_P5.00mm -> Capacitor_THT:C_Disc_D10.0mm_W2.5mm_P5.00mm
- D13: footprint Pin_Headers:D_DO-41_SOD81_P10.16mm_Horizontal -> Diode_THT:D_A-405_P10.16mm_Horizontal
- moved D13 127.7 mm to (176.8, 167.4), turned to 0 degrees
Connections:
- D13 pad 1: GND -> VCC
- D13 pad 2: VCC -> GND

Commit message: Akku/PC Layout angefangen
Parts:
- removed the REF** at (139.7, 237.5)
- added J7: Conn_01x02, Connector_Molex:Molex_KK-254_AE-6410-02A_1x02_P2.54mm_Vertical, F.Cu at (139.7, 191.8)
- added J8: Conn_01x02, Connector_Molex:Molex_KK-254_AE-6410-02A_1x02_P2.54mm_Vertical, F.Cu at (139.7, 183.5)
- added REF**: EuroBoard160mmX100mm_holes_keepout, bonsai:EuroBoard160mmX100mm_holes_keepout, F.Cu at (45.7, 48.3)
- added RN1: R_Network08, Resistor_THT:R_Array_SIP9, F.Cu at (62.9, 61.6)
- U2: value 7400 -> 74HC00
- U4: value 7408 -> 74HC08
- moved D13 151.1 mm to (76.2, 54.6)
- moved C4 144.6 mm to (68.0, 55.2)
- moved R14 116.2 mm to (56.5, 95.9), turned to 0 degrees
- moved C8 99.1 mm to (64.8, 116.1), turned to 90 degrees
- moved R9 97.7 mm to (66.7, 99.7), turned to 180 degrees
- moved C6 88.9 mm to (64.8, 137.8), turned to 270 degrees
- moved C5 66.7 mm to (98.4, 116.1), turned to 90 degrees
- moved C7 66.6 mm to (98.4, 137.8), turned to 270 degrees
- moved J4 48.7 mm to (139.7, 175.3)
- moved R10 47.8 mm to (124.5, 161.9)
- moved J3 47.5 mm to (139.7, 161.9)
- moved R11 43.4 mm to (121.3, 161.9)
- moved R5 42.2 mm to (130.8, 151.8), turned to 270 degrees
- moved R4 39.9 mm to (127.6, 151.8), turned to 270 degrees
- moved U7 37.1 mm to (120.0, 136.5)
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Connections:
- net Net-(U1-Pad4) renamed /~write_i
- net ^enable renamed /~write
- J3 pad 1: /~load -> /~inc
- J3 pad 2: ^up -> /~dec
- J3 pad 3: ^down -> /~load
- R1 pad 2: ^up -> /~inc
- R5 pad 2: ^down -> /~dec
- U4 pad 10: (no net) -> VCC
- U4 pad 12: ^up -> /~inc
- U4 pad 2: ^down -> /~dec
- U4 pad 4: (no net) -> VCC
- U4 pad 5: (no net) -> VCC
- U4 pad 6: (no net) -> Net-(U4-Pad6)
- U4 pad 8: (no net) -> Net-(U4-Pad8)
- U4 pad 9: (no net) -> VCC
Routing:
- net VCC: track 787.2 -> 264.9 mm, vias 4 -> 1
- net GND: track 652.4 -> 394.1 mm, vias 11 -> 0
- net /~write_i: track 209.1 -> 8.67 mm
- net Net-(D7-Pad2): track 144.8 -> 0.00 mm
- net /clr: track 125.0 -> 0.00 mm, vias 3 -> 0
- net Net-(D1-Pad2): track 122.7 -> 0.00 mm
- net /~write: track 111.0 -> 0.00 mm
- net /down_i: track 114.3 -> 11.1 mm, vias 2 -> 0
- net /~load: track 116.1 -> 16.4 mm, vias 4 -> 0
- net /B1: track 302.3 -> 205.5 mm, vias 6 -> 1
- net /up_i: track 106.6 -> 12.2 mm, vias 2 -> 0
- net /B0: track 303.7 -> 215.7 mm, vias 4 -> 1
- net /B5: track 268.1 -> 180.8 mm, vias 6 -> 1
- net ^down: track 81.1 -> 0.00 mm
- net ^up: track 77.7 -> 0.00 mm, vias 2 -> 0
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Other:
- board text removed: "+"
- board text removed: "-"

Commit message: Akku Board weiter
Parts:
- moved R1 46.4 mm to (118.7, 195.6), turned to 90 degrees
- moved R5 46.4 mm to (115.6, 195.6), turned to 90 degrees
- moved R4 44.2 mm to (121.9, 195.6), turned to 90 degrees
- moved R3 21.0 mm to (104.1, 195.6)
- moved R11 19.6 mm to (140.3, 157.5)
- moved R12 17.5 mm to (125.1, 185.4), turned to 270 degrees
- moved R2 14.0 mm to (108.0, 195.6)
- moved R10 12.9 mm to (136.5, 157.5)
- moved C1 3.18 mm to (79.4, 173.9)
- moved C3 3.18 mm to (104.8, 173.9)
- moved SW1 3.18 mm to (70.5, 193.0)
- moved SW2 3.18 mm to (84.5, 193.0)
- moved SW3 3.18 mm to (98.4, 193.0)
- moved U1 3.18 mm to (108.6, 175.3)
- moved U2 3.18 mm to (58.4, 175.3)
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Routing:
- net VCC: track 264.9 -> 555.1 mm, vias 1 -> 2
- net GND: track 394.1 -> 616.2 mm
- net Net-(R9-Pad2): track 0.00 -> 136.5 mm
- net Net-(R14-Pad1): track 0.00 -> 135.7 mm, vias 0 -> 1
- net /~write_i: track 8.67 -> 136.5 mm, vias 0 -> 1
- net /~load: track 16.4 -> 132.1 mm
- net /~inc: track 5.71 -> 116.0 mm
- net /clr: track 0.00 -> 102.6 mm
- net /down_i: track 11.1 -> 106.7 mm, vias 0 -> 2
- net /~write: track 0.00 -> 70.2 mm
- net /~dec: track 11.1 -> 74.2 mm
- net /up_i: track 12.2 -> 61.2 mm, vias 0 -> 1
- net Net-(U2-Pad11): track 0.00 -> 42.7 mm
- net RPA4: track 0.00 -> 42.5 mm
- net RPA2: track 0.00 -> 36.6 mm
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
Commit message: Akku Layout weitergemacht
Parts:
- moved D1 8.89 mm to (75.6, 88.9)
- moved D12 4.58 mm to (134.0, 91.4)
- moved R21 4.58 mm to (134.0, 94.0)
- moved D10 4.58 mm to (123.8, 91.4)
- moved D11 4.58 mm to (128.9, 91.4)
- moved D8 4.58 mm to (113.7, 91.4)
- moved D9 4.58 mm to (118.7, 91.4)
- moved R17 4.58 mm to (113.7, 94.0)
- moved R18 4.58 mm to (118.7, 94.0)
- moved R19 4.58 mm to (123.8, 94.0)
- moved R20 4.58 mm to (128.9, 94.0)
- moved D4 4.58 mm to (98.4, 91.4)
- moved D5 4.58 mm to (103.5, 91.4)
- moved D6 4.58 mm to (108.6, 91.4)
- moved R13 4.58 mm to (98.4, 94.0)
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Routing:
- net GND: track 616.2 -> 625.9 mm
- net Net-(R17-Pad2): track 10.8 -> 6.24 mm
- net VCC: track 555.1 -> 559.5 mm
- net Net-(R15-Pad2): track 13.5 -> 9.83 mm
- net Net-(R18-Pad2): track 9.75 -> 6.24 mm
- net Net-(R16-Pad2): track 11.9 -> 8.41 mm
- net Net-(R13-Pad2): track 16.2 -> 13.9 mm
- net Net-(D1-Pad2): track 11.5 -> 13.5 mm
- net Net-(D2-Pad2): track 7.29 -> 5.39 mm
- net /B7: track 207.6 -> 209.4 mm
- net /B6: track 220.2 -> 221.8 mm
- net Net-(R19-Pad2): track 9.84 -> 8.41 mm
- net Net-(D7-Pad2): track 8.19 -> 6.77 mm
- net /B5: track 180.8 -> 182.1 mm
- net Net-(R14-Pad1): track 135.7 -> 134.5 mm
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Other:
- board text added: "0"
- board text added: "1"
- board text added: "2"
- board text added: "3"
- board text added: "4"
- board text added: "5"
- board text added: "6"
- board text added: "7"
- board text added: "DEC"
- board text added: "INC"
- board text added: "clr"
- board text added: "decrease"
- board text added: "increase"
- board text added: "rev 2.0"
- board text added: "~dec"
- board text added: "~inc"
- board text added: "~write"
- board text removed: "DOWN"
- board text removed: "UP"
- board text removed: "clear"
- board text removed: "~down"
- board text removed: "~en"
- board text removed: "~up"

Commit message: EinTaktReset
Other:
- board text added: "+"
- board text added: "-"
