File: Akku.kicad_pcb (KiCad board)
At the start: 2 copper layers, 100 x 160 mm, 60 parts, among them J1 Conn_02x10_Odd_Even, J2 Conn_01x02, J3 Conn_01x04, J4 Conn_01x02, J5 Conn_02x10_Odd_Even, J6 Conn_02x10_Odd_Even, J7 Conn_01x02, J8 Conn_01x02, SW1 Digitast, SW2 Digitast, SW3 Digitast, U1 74HC14, U2 74HC00, U4 74HC08, U5 74LS193, U6 74LS541, U7 74LS193, U8 74LS540

Commit message: viele kleine Änderungen
Connections:
- net /~load renamed /~read
- J4 pad 2: Net-(J4-Pad2) -> /clr
- J7 pad 1: Net-(J7-Pad1) -> /~inc
Routing:
- net /clr: track 102.6 -> 105.1 mm
- net /~inc: track 116.7 -> 119.3 mm
Other:
- net class Default: via_dia 0.6 -> 0.8
- net class Power: via_dia 0.6 -> 0.8
- net class smal: via_dia 0.6 -> 0.8
- rule trace_min: 0.15 -> 0.4
- rule via_min_drill: 0.3 -> 0.4
- rule via_min_size: 0.4 -> 0.8
- board text added: "JLCJLCJLCJLC"
- board text added: "~read"
- board text removed: "~load"
