File: Akku.sch (KiCad schematic (older format))
At the start: 49 parts, among them J1 +/- Stecker, J2 load/up, J3 down/en/clear, P7 CONN_02X10, P8 CONN_02X10, P9 CONN_02X10, SW1 UP_Bonsai_SWITCH_INV, SW2 DOWN_Bonsai_SWITCH_INV, SW3 CLR_Bonsai_SWITCH_INV, U1 74HC14, U2 7400, U4 7408, U5 74LS193, U6 74LS541, U7 74LS193, U8 74LS540

Commit message: Akku: Bauteilwerte ergänzt
Parts:
- C1, C2, C3: value C -> 100n
- R12: value R -> 470
- R13, R15, R16, R17, R18, R19, R20, R21: value R -> 330
- R14: value R -> 150
- R2, R3: value R -> 4k7
Connections:
- net labels added: ^up
- net labels removed: VDD, VSS, ûp
- wire segments 264 -> 263

Commit message: Akku: Schaltungen zum entprellen der Taster gleichartig angeordnet
Parts:
- R10, R11, R9: value R -> 150
Connections:
- wire segments 263 -> 267
Changed lines of the file:
@@
 P 3650 2250
 F 0 "R9" H 3720 2296 50  0000 L CNN
-F 1 "R" H 3720 2205 50  0000 L CNN
+F 1 "150" H 3720 2205 50  0000 L CNN
 F 2 "Resistors_ThroughHole:R_Axial_DIN0207_L6.3mm_D2.5mm_P10.16mm_Horizontal" V 3580 2250 50  0001 C CNN
 F 3 "" H 3650 2250 50  0000 C CNN
@@
 $EndComp
 $Comp
-L allBonsaiSymbolLibs:7400 U2
-U 4 1 580F5956
-P 2650 5000
-F 0 "U2" H 2650 5050 50  0000 C CNN
-F 1 "7400" H 2650 4900 50  0000 C CNN
-F 2 "Housings_DIP:DIP-14_W7.62mm_LongPads" H 2650 5000 50  0001 C CNN
-F 3 "" H 2650 5000 50  0000 C CNN
-	4    2650 5000
-	1    0    0    -1
-$EndComp
-$Comp
-L allBonsaiSymbolLibs:7400 U2
-U 1 1 580F5818
-P 2650 4200
-F 0 "U2" H 2650 4250 50  0000 C CNN
-F 1 "7400" H 2650 4100 50  0000 C CNN
-F 2 "Housings_DIP:DIP-14_W7.62mm_LongPads" H 2650 4200 50  0001 C CNN
-F 3 "" H 2650 4200 50  0000 C CNN
-	1    2650 4200
-	1    0    0    -1
-$EndComp
-$Comp
-L allBonsaiSymbolLibs:SWITCH_INV-bonsai SW1
-U 1 1 58100CBF
-P 1400 4600
-F 0 "SW1" H 1200 4750 50  0000 C CNN
-F 1 "UP_Bonsai_SWITCH_INV" H 1250 4450 50  0000 C CNN
-F 2 "allBonsaiFootprintsLibs:SW_PUSH_LCD_E3_SAxxxx_tg_V2" H 1400 4600 50  0001 C CNN
-F 3 "" H 1400 4600 50  0000 C CNN
-	1    1400 4600
-	1    0    0    1
-$EndComp
-$Comp
 L power:GND #PWR04
 U 1 1 58100E67
-P 900 4600
-F 0 "#PWR04" H 900 4350 50  0001 C CNN
-F 1 "GND" H 900 4450 50  0000 C CNN
-F 2 "" H 900 4600 50  0000 C CNN
-F 3 "" H 900 4600 50  0000 C CNN
-	1    900  4600
+P 650 4850
+F 0 "#PWR04" H 650 4600 50  0001 C CNN
+F 1 "GND" H 650 4700 50  0000 C CNN
+F 2 "" H 650 4850 50  0000 C CNN
+F 3 "" H 650 4850 50  0000 C CNN
+	1    650  4850
 	1    0    0    -1
 $EndComp
@@
 P 5850 3900
 F 0 "R11" V 5930 3900 50  0000 C CNN
-F 1 "R" V 5850 3900 50  0000 C CNN
+F 1 "150" V 5850 3900 50  0000 C CNN
 F 2 "Resistors_ThroughHole:R_Axial_DIN0207_L6.3mm_D2.5mm_P10.16mm_Horizontal" V 5780 3900 50  0001 C CNN
 F 3 "" H 5850 3900 50  0000 C CNN
@@
 L power:GND #PWR05
 U 1 1 58103EBB
-P 900 6650
-F 0 "#PWR05" H 900 6400 50  0001 C CNN
-F 1 "GND" H 900 6500 50  0000 C CNN
-F 2 "" H 900 6650 50  0000 C CNN
-F 3 "" H 900 6650 50  0000 C CNN
-	1    900  6650
+P 650 6450
+F 0 "#PWR05" H 650 6200 50  0001 C CNN
+F 1 "GND" H 650 6300 50  0000 C CNN
+F 2 "" H 650 6450 50  0000 C CNN
+F 3 "" H 650 6450 50  0000 C CNN
+	1    650  6450
 	1    0    0    -1
 $EndComp
@@
 Wire Wire Line
 	2050 6650 2050 6450
-Wire Wire Line
-	1900 4100 1900 4500
-Wire Wire Line
-	1900 5100 1900 4700
-Wire Wire Line
-	3250 4700 3250 5000
-Wire Wire Line
-	2050 4300 2050 4500
 Connection ~ 1300 3000
 Wire Wire Line
@@
 	4950 4050 4850 4050
 Wire Wire Line
-	2050 4500 2650 4500
-Wire Wire Line
-	2650 4500 2650 4700
-Wire Wire Line
-	2650 4700 3250 4700
-Wire Wire Line
-	3250 4200 3250 4650
-Wire Wire Line
-	3250 4650 2050 4650
-Wire Wire Line
-	2050 4650 2050 4900
-Wire Wire Line
-	1900 4100 2050 4100
+	1800 5250 1900 5250
 Wire Wire Line
 	7600 3100 4650 3100
@@
 P 5650 6200
 F 0 "R10" V 5730 6200 50  0000 C CNN
-F 1 "R" V 5650 6200 50  0000 C CNN
+F 1 "150" V 5650 6200 50  0000 C CNN
 F 2 "Resistors_ThroughHole:R_Axial_DIN0207_L6.3mm_D2.5mm_P10.16mm_Horizontal" V 5580 6200 50  0001 C CNN
 F 3 "" H 5650 6200 50  0000 C CNN
@@
 	0    1    1    0
 $EndComp
-Text GLabel 1900 5100 3    50   Input ~ 0
+Text GLabel 1800 4250 0    50   Input ~ 0
 RPA2
 Text GLabel 1900 5850 1    50   Input ~ 0
@@
 	1900 5850 2050 5850
 Wire Wire Line
-	1900 5100 2050 5100
-Text GLabel 1900 4100 0    50   Input ~ 0
+	1800 4250 1900 4250
+Text GLabel 1800 5250 0    50   Input ~ 0
 RPA1
 Text GLabel 2950 3800 0    50   Input ~ 0
@@
 Wire Wire Line
 	10350 5750 10450 5750
-Wire Wire Line
-	3250 4700 3550 4700
-Wire Wire Line
-	3550 4150 3550 4700
-Connection ~ 3250 4700
 $Comp
 L power:GND #PWR0103
@@
 	1000 1400 1200 1400
 Wire Wire Line
-	900  6650 900  6350
+	650  6350 900  6350
+$Comp
+L allBonsaiSymbolLibs:SWITCH_INV-bonsai SW1
+U 1 1 5F89E939
+P 1400 4750
+F 0 "SW1" H 1200 4900 50  0000 C CNN
+F 1 "UP_Bonsai_SWITCH_INV" H 1250 4600 50  0000 C CNN
+F 2 "allBonsaiFootprintsLibs:SW_PUSH_LCD_E3_SAxxxx_tg_V2" H 1400 4750 50  0001 C CNN
+F 3 "" H 1400 4750 50  0000 C CNN
+	1    1400 4750
+	1    0    0    -1
+$EndComp
+$Comp
+L allBonsaiSymbolLibs:7400 U2
+U 4 1 580F5956
+P 2650 4350
+F 0 "U2" H 2650 4400 50  0000 C CNN
+F 1 "7400" H 2650 4250 50  0000 C CNN
+F 2 "Housings_DIP:DIP-14_W7.62mm_LongPads" H 2650 4350 50  0001 C CNN
+F 3 "" H 2650 4350 50  0000 C CNN
+	4    2650 4350
+	1    0    0    1
+$EndComp
+$Comp
+L allBonsaiSymbolLibs:7400 U2
+U 1 1 580F5818
+P 2650 5150
+F 0 "U2" H 2650 5200 50  0000 C CNN
+F 1 "7400" H 2650 5050 50  0000 C CNN
+F 2 "Housings_DIP:DIP-14_W7.62mm_LongPads" H 2650 5150 50  0001 C CNN
+F 3 "" H 2650 5150 50  0000 C CNN
+	1    2650 5150
+	1    0    0    1
+$EndComp
+Wire Wire Line
+	1900 4650 1900 4250
+Connection ~ 1900 4250
+Wire Wire Line
+	1900 4250 2050 4250
+Wire Wire Line
+	1900 4850 1900 5250
+Connection ~ 1900 5250
+Wire Wire Line
+	1900 5250 2050 5250
+Wire Wire Line
+	3250 4350 3450 4350
+Wire Wire Line
+	3450 4350 3450 4150
+Wire Wire Line
+	3450 4150 3550 4150
+Wire Wire Line
+	3250 5150 3250 4850
+Wire Wire Line
+	3250 4850 2050 4650
+Wire Wire Line
+	2050 4650 2050 4450
+Wire Wire Line
+	3250 4350 3250 4650
+Wire Wire Line
+	3250 4650 2050 4850
+Wire Wire Line
+	2050 4850 2050 5050
+Connection ~ 3250 4350
+Connection ~ 3250 5950
+Wire Wire Line
+	900  4750 650  4750
+Wire Wire Line
+	650  4750 650  4850
+Wire Wire Line
+	650  6450 650  6350
 Wire Bus Line
 	6000 600  7400 600

Commit message: Backup vor Umbennung von Netzen
Connections:
- net labels added: B0, B1, B2, B3, B4, B5, B6, B7
- net labels removed: a0, a1, a2, a3, a4, a5, a6, a7
- wire segments 267 -> 264
Other:
- note added: "Bit 3..0"
- note added: "Bit 7..4"
- note added: "Datenbus (Akku) / Adressbus (PC)"

Commit message: Akku/PC: Schaltplan mit Bussen gezeichnet; Netze der Busse sinnvoll benannt
Connections:
- net labels added: Bi0, Bi1, Bi2, Bi3, Bi4, Bi5, Bi6, Bi7
- wire segments 264 -> 235

Commit message: Akku/PC: Schaltplan aufgeräumt
Connections:
- net labels added: clr, downCarry, down_i, upCarry, up_i, ~load
- net labels removed: CLR, RPB4, ^load
- wire segments 235 -> 221
Other:
- note added: "Verzögerung des ~Write~ - Signals\num 2 Gatter-Laufzeiten,\num bei einem Wechsel der Steuersignale\ngleichzeitiges Schreiben auf\nden Bus zu vermeiden"
- note added: "nur bestücken \nbei PC"
- note added: "nur bestücken\nbei Akku"
- note removed: "(Akku)"
- note removed: "(PC)"
- note removed: "Akku/PC - Modul"
- note removed: "Akkumulator"
- note removed: "Dezember 2017"

Commit message: Steuerwerk 2.0 gerber exportiert
Parts:
- added RN? (x3): R_Network04_Split, Resistor_THT:R_Array_SIP5, symbol Device:R_Network04_Split
- U1, U2, U4: footprint Housings_DIP:DIP-14_W7.62mm_LongPads -> Package_DIP:DIP-14_W7.62mm_Socket_LongPads
- U5, U7: footprint Housings_DIP:DIP-16_W7.62mm_LongPads -> Package_DIP:DIP-16_W7.62mm_Socket_LongPads
- U6, U8: footprint Housings_DIP:DIP-20_W7.62mm_LongPads -> Package_DIP:DIP-20_W7.62mm_Socket_LongPads
Connections:
- wire segments 221 -> 236

Commit message: Akku weitergebaut
Parts:
- removed J1: +/- Stecker, 2PinTerminalBlocktg, symbol allBonsaiSymbolLibs:2PinTerminalBlocktg-2PinTerminalBlocktg
- removed J2: load/up, 2PinTerminalBlocktg, symbol allBonsaiSymbolLibs:2PinTerminalBlocktg-2PinTerminalBlocktg
- removed J3: down/en/clear, 3PinTerminalBlocktg, symbol allBonsaiSymbolLibs:3PinTerminalBlocktg-3PinTerminalBlocktg
- removed RN? (x3): R_Network04_Split, Resistor_THT:R_Array_SIP5, symbol Device:R_Network04_Split
- removed RPB1: R_PACK4BUSSED, tg_locallibs:R_Array_SIP5, symbol allBonsaiSymbolLibs:R_PACK4BUSSED
- removed SW1: UP_Bonsai_SWITCH_INV, allBonsaiFootprintsLibs:SW_PUSH_LCD_E3_SAxxxx_tg_V2, symbol allBonsaiSymbolLibs:SWITCH_INV-bonsai
- removed SW2: DOWN_Bonsai_SWITCH_INV, allBonsaiFootprintsLibs:SW_PUSH_LCD_E3_SAxxxx_tg_V2, symbol allBonsaiSymbolLibs:SWITCH_INV-bonsai
- removed SW3: CLR_Bonsai_SWITCH_INV, allBonsaiFootprintsLibs:SW_PUSH_LCD_E3_SAxxxx_tg_V2, symbol allBonsaiSymbolLibs:SWITCH_INV-bonsai
- added J2, J4: Conn_01x02, Connector_Molex:Molex_KK-254_AE-6410-02A_1x02_P2.54mm_Vertical, symbol Connector_Generic:Conn_01x02
- added J3: Conn_01x04, Connector_Molex:Molex_KK-254_AE-6410-04A_1x04_P2.54mm_Vertical, symbol Connector_Generic:Conn_01x04
- added R1, R4, R5: 4k7, Resistor_THT:R_Axial_DIN0207_L6.3mm_D2.5mm_P10.16mm_Horizontal, symbol Device:R
- added SW1, SW2, SW3: Digitast, bonsai:Switch_Digitast, symbol Bonsai:Digitast
Connections:
- net labels removed: RPB1, RPB2, RPB3

Commit message: Akku weitergebaut
Parts:
- removed P7, P8, P9: CONN_02X10, allBonsaiFootprintsLibs:Pin_Header_Straight_2x10_Pitch2.00mmBonsai.pretty, symbol allBonsaiSymbolLibs:Conn_02x10_Counter_Clockwise-conn
- added J1, J5, J6: Conn_02x10_Odd_Even, Connector_PinHeader_2.54mm:PinHeader_2x10_P2.54mm_Vertical, symbol Connector_Generic:Conn_02x10_Odd_Even
- D1, D2, D3, D7: footprint LEDs:LED_D5.0mm_FlatTop -> LED_THT:LED_D3.0mm
- D10, D11, D12, D4, D5, D6, D8, D9: footprint LEDs:LED-3MM -> LED_THT:LED_D3.0mm
- R10, R11, R12, R13, R14, R15, R16, R17, R18, R19, R2, R20, R21, R3, R9: footprint Resistors_ThroughHole:R_Axial_DIN0207_L6.3mm_D2.5mm_P10.16mm_Horizontal -> Resistor_THT:R_Axial_DIN0207_L6.3mm_D2.5mm_P10.16mm_Horizontal
Connections:
- wire segments 236 -> 240
