File: Akku.sch (KiCad schematic (older format))
At the start: 51 parts, among them J1 Conn_02x10_Odd_Even, J2 Conn_01x02, J3 Conn_01x04, J4 Conn_01x02, J5 Conn_02x10_Odd_Even, J6 Conn_02x10_Odd_Even, SW1 Digitast, SW2 Digitast, SW3 Digitast, U1 74HC14, U2 7400, U4 7408, U5 74LS193, U6 74LS541, U7 74LS193, U8 74LS540

Commit message: akku weitergebaut
Parts:
- added C4: CP, Capacitor_THT:CP_Radial_D8.0mm_P2.50mm, symbol Device:CP
- added C5, C6, C7, C8: 100n, Capacitor_THT:C_Disc_D10.0mm_W2.5mm_P5.00mm, symbol allBonsaiSymbolLibs:C-bonsai
- C1, C2, C3: footprint allBonsaiFootprintsLibs:C_Disc_D10.0mm_W2.5mm_P5.00mm -> Capacitor_THT:C_Disc_D10.0mm_W2.5mm_P5.00mm
- D13: footprint Pin_Headers:D_DO-41_SOD81_P10.16mm_Horizontal -> Diode_THT:D_A-405_P10.16mm_Horizontal; symbol allBonsaiSymbolLibs:D-bonsai -> allBonsaiSymbolLibs:D-device
Connections:
- wire segments 240 -> 252
Changed lines of the file:
@@
 NoConn ~ 12850 5250
 NoConn ~ 12850 5100
-Connection ~ 14650 3350
-Connection ~ 14650 3050
-Wire Wire Line
-	14650 3050 14450 3050
-Wire Wire Line
-	14650 3350 14450 3350
-$Comp
-L allBonsaiSymbolLibs:C-bonsai C3
-U 1 1 5CC7F388
-P 14450 3200
-F 0 "C3" V 14138 3200 50  0000 C CNN
-F 1 "100n" V 14229 3200 50  0000 C CNN
-F 2 "allBonsaiFootprintsLibs:C_Disc_D10.0mm_W2.5mm_P5.00mm" V 14305 3200 30  0001 C CNN
-F 3 "" H 14450 3200 60  0000 C CNN
-	1    14450 3200
-	-1   0    0    1
-$EndComp
-Connection ~ 14850 3350
-Wire Wire Line
-	14850 3350 14750 3350
-Wire Wire Line
-	15000 3350 14850 3350
-$Comp
-L allBonsaiSymbolLibs:D-bonsai D13
+Connection ~ 13450 9250
+Connection ~ 13450 8950
+Connection ~ 13700 9250
+$Comp
+L allBonsaiSymbolLibs:D-device D13
 U 1 1 5CC05CEA
-P 15000 3200
-F 0 "D13" H 15000 2879 50  0000 C CNN
-F 1 "D" H 15000 2970 50  0000 C CNN
-F 2 "Pin_Headers:D_DO-41_SOD81_P10.16mm_Horizontal" H 15000 3069 60  0001 C CNN
-F 3 "" H 15000 3200 60  0000 C CNN
-	1    15000 3200
-	0    -1   -1   0
+P 12200 9100
+F 0 "D13" V 12150 9250 50  0001 C CNN
+F 1 "D" V 12250 9200 50  0001 C CNN
+F 2 "Diode_THT:D_A-405_P10.16mm_Horizontal" H 12200 8969 60  0001 C CNN
+F 3 "" H 12200 9100 60  0000 C CNN
+	1    12200 9100
+	0    1    1    0
 $EndComp
 $Comp
 L allBonsaiSymbolLibs:C-bonsai C2
 U 1 1 5CBF52E5
-P 14650 3200
-F 0 "C2" V 14338 3200 50  0000 C CNN
-F 1 "100n" V 14429 3200 50  0000 C CNN
-F 2 "allBonsaiFootprintsLibs:C_Disc_D10.0mm_W2.5mm_P5.00mm" V 14505 3200 30  0001 C CNN
-F 3 "" H 14650 3200 60  0000 C CNN
-	1    14650 3200
+P 13450 9100
+F 0 "C2" V 13138 9100 50  0001 C CNN
+F 1 "100n" V 13229 9100 50  0001 C CNN
+F 2 "Capacitor_THT:C_Disc_D10.0mm_W2.5mm_P5.00mm" V 13305 9100 30  0001 C CNN
+F 3 "" H 13450 9100 60  0000 C CNN
+	1    13450 9100
 	-1   0    0    1
 $EndComp
@@
 L allBonsaiSymbolLibs:C-bonsai C1
 U 1 1 5CBF3D2E
-P 14850 3200
-F 0 "C1" V 14538 3200 50  0000 C CNN
-F 1 "100n" V 14629 3200 50  0000 C CNN
-F 2 "allBonsaiFootprintsLibs:C_Disc_D10.0mm_W2.5mm_P5.00mm" V 14705 3200 30  0001 C CNN
-F 3 "" H 14850 3200 60  0000 C CNN
-	1    14850 3200
+P 13700 9100
+F 0 "C1" V 13388 9100 50  0001 C CNN
+F 1 "100n" V 13479 9100 50  0001 C CNN
+F 2 "Capacitor_THT:C_Disc_D10.0mm_W2.5mm_P5.00mm" V 13555 9100 30  0001 C CNN
+F 3 "" H 13700 9100 60  0000 C CNN
+	1    13700 9100
 	-1   0    0    1
 $EndComp
-Connection ~ 14850 3050
-Wire Wire Line
-	14850 3050 15000 3050
-Wire Wire Line
-	14850 3050 14850 3000
+Connection ~ 13700 8950
+Wire Wire Line
+	13700 8950 13950 8950
+Wire Wire Line
+	11800 8950 11800 8850
 $Comp
 L power:VCC #PWR025
 U 1 1 5A8A1D7F
-P 14850 3000
-F 0 "#PWR025" H 14850 2850 50  0001 C CNN
-F 1 "VCC" H 14867 3173 50  0000 C CNN
-F 2 "" H 14850 3000 50  0001 C CNN
-F 3 "" H 14850 3000 50  0001 C CNN
-	1    14850 3000
+P 11800 8850
+F 0 "#PWR025" H 11800 8700 50  0001 C CNN
+F 1 "VCC" H 11817 9023 50  0000 C CNN
+F 2 "" H 11800 8850 50  0001 C CNN
+F 3 "" H 11800 8850 50  0001 C CNN
+	1    11800 8850
 	1    0    0    -1
 $EndComp
@@
 L power:GND #PWR014
 U 1 1 5A840FE3
-P 14750 3350
-F 0 "#PWR014" H 14750 3100 50  0001 C CNN
-F 1 "GND" H 14755 3177 50  0000 C CNN
-F 2 "" H 14750 3350 50  0001 C CNN
-F 3 "" H 14750 3350 50  0001 C CNN
-	1    14750 3350
-	1    0    0    -1
-$EndComp
-Wire Wire Line
-	14650 3050 14850 3050
+P 11800 9300
+F 0 "#PWR014" H 11800 9050 50  0001 C CNN
+F 1 "GND" H 11805 9127 50  0000 C CNN
+F 2 "" H 11800 9300 50  0001 C CNN
+F 3 "" H 11800 9300 50  0001 C CNN
+	1    11800 9300
+	1    0    0    -1
+$EndComp
+Wire Wire Line
+	13450 8950 13700 8950
 Wire Wire Line
 	4250 5200 4350 5200
@@
 L Connector_Generic:Conn_01x02 J2
 U 1 1 5FDE0B19
-P 13550 3150
-F 0 "J2" H 13468 2825 50  0000 C CNN
-F 1 "Conn_01x02" H 13468 2916 50  0000 C CNN
-F 2 "Connector_Molex:Molex_KK-254_AE-6410-02A_1x02_P2.54mm_Vertical" H 13550 3150 50  0001 C CNN
-F 3 "~" H 13550 3150 50  0001 C CNN
-	1    13550 3150
+P 11450 9050
+F 0 "J2" H 11368 8725 50  0000 C CNN
+F 1 "Conn_01x02" H 11368 8816 50  0000 C CNN
+F 2 "Connector_Molex:Molex_KK-254_AE-6410-02A_1x02_P2.54mm_Vertical" H 11450 9050 50  0001 C CNN
+F 3 "~" H 11450 9050 50  0001 C CNN
+	1    11450 9050
 	-1   0    0    1
 $EndComp
@@
 Wire Wire Line
 	1150 10900 1050 10900
-Connection ~ 14750 3350
-Wire Wire Line
-	14750 3350 14650 3350
-Wire Wire Line
-	13750 3050 14450 3050
-Connection ~ 14450 3050
-Wire Wire Line
-	14450 3350 13750 3350
-Wire Wire Line
-	13750 3350 13750 3150
-Connection ~ 14450 3350
+Wire Wire Line
+	11650 8950 11800 8950
+Connection ~ 13200 8950
+Wire Wire Line
+	11650 9250 11650 9050
+Connection ~ 13200 9250
 Wire Wire Line
 	3900 8750 3900 9350
@@
 Wire Wire Line
 	7550 1700 7550 1600
+Wire Wire Line
+	13700 9250 13450 9250
+Connection ~ 11800 8950
+Wire Wire Line
+	11800 9300 11800 9250
+Wire Wire Line
+	13700 9250 13950 9250
+Connection ~ 11800 9250
+Wire Wire Line
+	11800 9250 11650 9250
+Wire Wire Line
+	11800 8950 11950 8950
+Wire Wire Line
+	13200 9250 12950 9250
+Wire Wire Line
+	13450 8950 13200 8950
+Wire Wire Line
+	13450 9250 13200 9250
+$Comp
+L allBonsaiSymbolLibs:C-bonsai C3
+U 1 1 5CC7F388
+P 13200 9100
+F 0 "C3" V 12888 9100 50  0001 C CNN
+F 1 "100n" V 12979 9100 50  0001 C CNN
+F 2 "Capacitor_THT:C_Disc_D10.0mm_W2.5mm_P5.00mm" V 13055 9100 30  0001 C CNN
+F 3 "" H 13200 9100 60  0000 C CNN
+	1    13200 9100
+	-1   0    0    1
+$EndComp
+$Comp
+L allBonsaiSymbolLibs:C-bonsai C7
+U 1 1 5FCDB8CE
+P 12950 9100
+F 0 "C7" V 12638 9100 50  0001 C CNN
+F 1 "100n" V 12729 9100 50  0001 C CNN
+F 2 "Capacitor_THT:C_Disc_D10.0mm_W2.5mm_P5.00mm" V 12805 9100 30  0001 C CNN
+F 3 "" H 12950 9100 60  0000 C CNN
+	1    12950 9100
+	-1   0    0    1
+$EndComp
+Connection ~ 12950 9250
+Wire Wire Line
+	12950 9250 12700 9250
+Connection ~ 12950 8950
+Wire Wire Line
+	12950 8950 13200 8950
+$Comp
+L allBonsaiSymbolLibs:C-bonsai C8
+U 1 1 5FCDBABE
+P 13950 9100
+F 0 "C8" V 13638 9100 50  0001 C CNN
+F 1 "100n" V 13729 9100 50  0001 C CNN
+F 2 "Capacitor_THT:C_Disc_D10.0mm_W2.5mm_P5.00mm" V 13805 9100 30  0001 C CNN
+F 3 "" H 13950 9100 60  0000 C CNN
+	1    13950 9100
+	-1   0    0    1
+$EndComp
+$Comp
+L allBonsaiSymbolLibs:C-bonsai C6
+U 1 1 5FD30308
+P 12700 9100
+F 0 "C6" V 12388 9100 50  0001 C CNN
+F 1 "100n" V 12479 9100 50  0001 C CNN
+F 2 "Capacitor_THT:C_Disc_D10.0mm_W2.5mm_P5.00mm" V 12555 9100 30  0001 C CNN
+F 3 "" H 12700 9100 60  0000 C CNN
+	1    12700 9100
+	-1   0    0    1
+$EndComp
+Connection ~ 12700 9250
+Wire Wire Line
+	12700 9250 12450 9250
+Connection ~ 12700 8950
+Wire Wire Line
+	12700 8950 12950 8950
+$Comp
+L allBonsaiSymbolLibs:C-bonsai C5
+U 1 1 5FD53DEE
+P 12450 9100
+F 0 "C5" V 12138 9100 50  0001 C CNN
+F 1 "100n" V 12229 9100 50  0001 C CNN
+F 2 "Capacitor_THT:C_Disc_D10.0mm_W2.5mm_P5.00mm" V 12305 9100 30  0001 C CNN
+F 3 "" H 12450 9100 60  0000 C CNN
+	1    12450 9100
+	-1   0    0    1
+$EndComp
+Connection ~ 12450 9250
+Wire Wire Line
+	12450 9250 12200 9250
+Connection ~ 12450 8950
+Wire Wire Line
+	12450 8950 12700 8950
+Connection ~ 12200 8950
+Wire Wire Line
+	12200 8950 12450 8950
+Connection ~ 12200 9250
+Wire Wire Line
+	12200 9250 11950 9250
+$Comp
+L Device:CP C4
+U 1 1 5FD6DC45
+P 11950 9100
+F 0 "C4" H 12068 9146 50  0001 L CNN
+F 1 "CP" H 12068 9055 50  0001 L CNN
+F 2 "Capacitor_THT:CP_Radial_D8.0mm_P2.50mm" H 11988 8950 50  0001 C CNN
+F 3 "~" H 11950 9100 50  0001 C CNN
+	1    11950 9100
+	1    0    0    -1
+$EndComp
+Connection ~ 11950 8950
+Wire Wire Line
+	11950 8950 12200 8950
+Connection ~ 11950 9250
+Wire Wire Line
+	11950 9250 11800 9250
 Wire Bus Line
 	8800 6300 11900 6300

Commit message: Akku/PC Layout angefangen
Parts:
- removed U1: 74HC14, Package_DIP:DIP-14_W7.62mm_Socket_LongPads, symbol allBonsaiSymbolLibs:4069-cmos4000
- removed U2: 7400, Package_DIP:DIP-14_W7.62mm_Socket_LongPads, symbol allBonsaiSymbolLibs:7400
- removed U4: 7408, Package_DIP:DIP-14_W7.62mm_Socket_LongPads, symbol allBonsaiSymbolLibs:74LS08-74xx
- added J7, J8: Conn_01x02, Connector_Molex:Molex_KK-254_AE-6410-02A_1x02_P2.54mm_Vertical, symbol Connector_Generic:Conn_01x02
- added RN1: R_Network08, Resistor_THT:R_Array_SIP9, symbol Device:R_Network08
- added U1: 74HC14, Package_DIP:DIP-14_W7.62mm_Socket_LongPads, symbol Bonsai:7414
- added U2: 74HC00, Package_DIP:DIP-14_W7.62mm_Socket_LongPads, symbol Bonsai:7400
- added U4: 74HC08, Package_DIP:DIP-14_W7.62mm_Socket_LongPads, symbol Bonsai:7408
- U5, U7: symbol allBonsaiSymbolLibs:74LS193 -> Bonsai:74193
Connections:
- net labels added: ~dec, ~inc, ~read, ~write, ~write_i
- net labels removed: ^down, ^enable, ^up
- wire segments 252 -> 286
- no-connect marks 2 -> 6
Other:
- note added: "Stecker für Akku und PC:"
- note added: "Stecker nur für Akku:"
- note added: "Stecker nur für PC:"
- note added: "Verzögerung des ~Write~ - Signals\num 2 Gatter-Laufzeiten,\num bei einem Wechsel der Steuersignale\nzu erreichen, dass die Daten lange genug\nauf dem Bus anliegen, so dass sie sicher\nübertragen werden"
- note added: "zu Ein/\nTakt/Reset"
- note added: "zu\nBefehle"
- note added: "zum\nSteuer-\nwerk"
- note removed: "Verzögerung des ~Write~ - Signals\num 2 Gatter-Laufzeiten,\num bei einem Wechsel der Steuersignale\ngleichzeitiges Schreiben auf\nden Bus zu vermeiden"

Commit message: viele kleine Änderungen
Connections:
- net labels removed: ~load
- wire segments 286 -> 294
- no-connect marks 6 -> 4
