File: EinTaktReset.sch (KiCad schematic (older format))
At the start: 58 parts, among them IC1 74LS624, J1 3PinTerminalBlocktg, J2 3PinTerminalBlocktg, J3 2PinTerminalBlocktg, J4 3PinTerminalBlocktg, J5 2PinTerminalBlocktg, P1 CONN_02X10, P4 CONN_02X10, SW1 SWITCH_INV, SW10 SPST, SW11 SPST, SW12 SPST, SW13 SPST, SW2 SWITCH_INV, SW3 SPST, SW4 SPST, SW5 SPST, SW6 SWITCH_INV, SW7 SPST, SW8 SPST, SW9 SPST, U1 74LS132, U2 74540En, U3 74HCT541_PWR, U4 74LS32, U5 74LS00

Commit message: Speicher Layout EinTaktReset VCO
Parts:
- removed C3: 220 µ, Capacitors_ThroughHole:CP_Radial_D8.0mm_P3.50mm, symbol allBonsaiSymbolLibs:bonsai_CP
- removed C4: 220µ, Capacitors_ThroughHole:CP_Radial_D8.0mm_P3.50mm, symbol allBonsaiSymbolLibs:bonsai_CP
- removed C5: 10n, Capacitors_ThroughHole:C_Disc_D3.0mm_W1.6mm_P2.50mm, symbol allBonsaiSymbolLibs:bonsai_C
- removed IC1: 74LS624, Housings_DIP:DIP-14_W7.62mm_Socket_LongPads, symbol allBonsaiSymbolLibs:vco_74LS624
- removed J1, J2, J4: 3PinTerminalBlocktg, 3PinTerminalBlocktg, symbol allBonsaiSymbolLibs:3PinTerminalBlocktg_3PinTerminalBlocktg
- removed J3, J5: 2PinTerminalBlocktg, 2PinTerminalBlocktg, symbol allBonsaiSymbolLibs:2PinTerminalBlocktg_2PinTerminalBlocktg
- added C10, C5: C, symbol Device:C
- added C3, C4: CP, Capacitor_THT:CP_Radial_D10.0mm_P2.50mm_P5.00mm, symbol Device:CP
- added R18, R19: 10k, Resistors_ThroughHole:R_Axial_DIN0207_L6.3mm_D2.5mm_P10.16mm_Horizontal, symbol allBonsaiSymbolLibs:device_R
- added U6: 74HC4046, Package_DIP:DIP-16_W7.62mm_Socket_LongPads, symbol Bonsai:74HC4046
- RV1: value POT -> Poti 10k
- U2: footprint (none) -> Housings_DIP:DIP-20_W7.62mm_Socket_LongPads
Connections:
- net labels added: VCC
- wire segments 291 -> 314
- no-connect marks 2 -> 7

Commit message: EinTaktReset
Parts:
- removed SW1, SW2: SWITCH_INV, tg_foodprint:SW_PUSH_LCD_E3_SAxxxx_tg_V2, symbol allBonsaiSymbolLibs:bonsai_SWITCH_INV
- removed SW3, SW4: SPST, tg_foodprint:eintakt_tg_SW_CuK_JS202011CQN_DPDT_Straight, symbol allBonsaiSymbolLibs:bonsai_SW_PUSH
- removed SW6: SWITCH_INV, tg_foodprint:eintakt_tg_SW_CuK_JS202011CQN_DPDT_Straight, symbol allBonsaiSymbolLibs:bonsai_SWITCH_INV
- removed U1: 74LS132, Housings_DIP:DIP-14_W7.62mm_Socket_LongPads, symbol allBonsaiSymbolLibs:74xx_74LS132
- removed U2: 74540En, Housings_DIP:DIP-20_W7.62mm_Socket_LongPads, symbol allBonsaiSymbolLibs:74540_74540En
- removed U4: 74LS32, Housings_DIP:DIP-14_W7.62mm_Socket_LongPads, symbol allBonsaiSymbolLibs:74xx_74LS32
- removed U5: 74LS00, Housings_DIP:DIP-14_W7.62mm_Socket_LongPads, symbol allBonsaiSymbolLibs:74xx_74LS00
- added C11: CP, Capacitor_THT:CP_Radial_D8.0mm_P2.50mm, symbol Device:CP
- added C12, C13: 100n, Capacitor_THT:C_Disc_D10.0mm_W2.5mm_P5.00mm, symbol allBonsaiSymbolLibs:bonsai_C
- added C14, C15: CP, Capacitor_THT:CP_Radial_D10.0mm_P2.50mm_P5.00mm, symbol Device:CP
- added J1, J5, J6: Conn_01x02, Connector_Molex:Molex_KK-254_AE-6410-02A_1x02_P2.54mm_Vertical, symbol Connector_Generic:Conn_01x02
- added J2, J3, J4: Conn_01x03, Connector_Molex:Molex_KK-254_AE-6410-03A_1x03_P2.54mm_Vertical, symbol Connector_Generic:Conn_01x03
- added SW1, SW2: Digitast, bonsai:Switch_Digitast, symbol Bonsai:Digitast
- added SW3, SW4, SW6: SW_SPDT, Switches-Walter:switch_100sp5, symbol Switch:SW_SPDT
- added U1: 74132, Package_DIP:DIP-14_W7.62mm_Socket_LongPads, symbol Bonsai:74132
- added U2: 74540, Package_DIP:DIP-20_W7.62mm_Socket_LongPads, symbol Bonsai:74540
- added U4: 7432, Package_DIP:DIP-14_W7.62mm_Socket_LongPads, symbol Bonsai:7432
- added U5: 7400, Package_DIP:DIP-14_W7.62mm_Socket_LongPads, symbol Bonsai:7400
- C1, C2: footprint Capacitors_ThroughHole:CP_Radial_D5.0mm_P2.00mm -> Capacitor_THT:CP_Radial_D5.0mm_P2.00mm
- C10: footprint (none) -> Capacitor_THT:C_Disc_D10.0mm_W2.5mm_P5.00mm
- C5: footprint (none) -> Capacitor_THT:C_Disc_D9.0mm_W5.0mm_P5.00mm
- C6, C7, C8, C9: footprint Capacitors_ThroughHole:C_Disc_D10.0mm_W2.5mm_P5.00mm -> Capacitor_THT:C_Disc_D10.0mm_W2.5mm_P5.00mm
- D1, D3: footprint Diodes_ThroughHole:D_DO-35_SOD27_P10.16mm_Horizontal -> Diode_THT:D_A-405_P10.16mm_Horizontal
- D2: footprint LEDs:LED_D5.0mm -> LED_THT:LED_D3.0mm
- DROT1: footprint LEDs:LED_D3.0mm -> LED_THT:LED_D3.0mm
- P1, P4: footprint tg_foodprint:Pin_Header_Straight_2x10_Pitch2.00mmBonsai.pretty -> Connector_PinHeader_2.54mm:PinHeader_2x10_P2.54mm_Vertical; symbol allBonsaiSymbolLibs:conn_Conn_02x10_Counter_Clockwise -> Connector_Generic:Conn_02x10_Odd_Even
- R1, R10, R11, R13, R16, R17, R18, R19, R2, R4, R5, R6, R8: footprint Resistors_ThroughHole:R_Axial_DIN0207_L6.3mm_D2.5mm_P10.16mm_Horizontal -> Resistor_THT:R_Axial_DIN0207_L6.3mm_D2.5mm_P10.16mm_Horizontal
- R12, R9: footprint tg_foodprint:R_Axial_DIN0207_L6.3mm_D2.5mm_P12.7mm_Horizontaltg -> Resistor_THT:R_Axial_DIN0207_L6.3mm_D2.5mm_P10.16mm_Horizontal
- R14, R15: footprint tg_bonsai_proj_spec_libs:R_Axial_DIN0207_L6.3mm_D2.5mm_P10.16mm_Horizontal -> Resistor_THT:R_Axial_DIN0207_L6.3mm_D2.5mm_P10.16mm_Horizontal
- R3: footprint tg_foodprint:R_Axial_DIN0207_L6.3mm_D2.5mm_P17.7mm_Horizontaltg -> Resistor_THT:R_Axial_DIN0207_L6.3mm_D2.5mm_P10.16mm_Horizontal
- R7: footprint tg_foodprint:R_Axial_DIN0207_L6.3mm_D2.5mm_P21.59mm_Horizontaltg -> Resistor_THT:R_Axial_DIN0207_L6.3mm_D2.5mm_P10.16mm_Horizontal
- RP1: footprint Housings_SIP:SIP9_Housing_BigPads -> Resistor_THT:R_Array_SIP9
- SW10, SW11, SW12, SW13, SW5, SW7, SW8, SW9: footprint tg_foodprint:eintakt_tg_SW_CuK_JS202011CQN_DPDT_Straight -> Switches-Walter:switch_100sp5
- U3: footprint Housings_DIP:DIP-20_W7.62mm_Socket_LongPads -> Package_DIP:DIP-20_W7.62mm_Socket_LongPads
Connections:
- net labels removed: +5V, VDD
- wire segments 314 -> 365
- no-connect marks 7 -> 11
Other:
- note added: "(bei Reset 0)"
- note added: "(bei Reset 1)"
- note added: "Hand"
- note added: "RES"
- note added: "Steuerwerk"
- note added: "Takt"
- note added: "langsam"
- note added: "schnell"
- note added: "~RES"
- note added: "~enable"

Commit message: EinTaktReset
Parts:
- C5: footprint Capacitor_THT:C_Disc_D9.0mm_W5.0mm_P5.00mm -> Capacitor_THT:CP_Axial_L30.0mm_D12.5mm_P35.00mm_Horizontal
Changed lines of the file:
@@
 F 0 "C5" H 1615 6346 50  0000 L CNN
 F 1 "C" H 1615 6255 50  0000 L CNN
-F 2 "Capacitor_THT:C_Disc_D9.0mm_W5.0mm_P5.00mm" H 1538 6150 50  0001 C CNN
+F 2 "Capacitor_THT:CP_Axial_L30.0mm_D12.5mm_P35.00mm_Horizontal" H 1538 6150 50  0001 C CNN
 F 3 "~" H 1500 6300 50  0001 C CNN
 	1    1500 6300

Commit message: viele kleine Änderungen
Parts:
- U3: value 74HCT541_PWR -> 74HC541
Connections:
- net labels added: ~auto, ~clrMPC, ~en-ln1, ~en-ln2, ~enAkku, ~loadIR
- net labels removed: auto, clrMPC, en-ln1, en-ln2, enAkku, loadIR
- wire segments 365 -> 374
- no-connect marks 11 -> 9

Commit message: Netze umbenannt
Connections:
- net labels added: ~readIR, ~writeAccu
- net labels removed: ~enAkku, ~loadIR
Changed lines of the file:
@@
 clrAkku
 Text GLabel 10450 13100 2    60   Input ~ 0
-~loadIR
+~readIR
 Text GLabel 10450 12850 2    60   Input ~ 0
-~enAkku
+~writeAccu
 Text GLabel 10450 12600 2    60   Input ~ 0
 ~clrMPC
@@
 clrAkku
 Text GLabel 10050 7700 0    60   Input ~ 0
-~loadIR
+~readIR
 Text GLabel 10050 7500 0    60   Input ~ 0
-~enAkku
+~writeAccu
 Text GLabel 10050 7300 0    60   Input ~ 0
 ~clrMPC

Commit message: EinTaktReset kleine Korrekturen
Connections:
- net labels added: contCLK, ein0, ein1, ein2, ein3, ein4, ein5, ein6, ein7, ~enCu, ~enDEC
- net labels removed: enDEC, enSTW
- wire segments 374 -> 390
Other:
- note added: "0"
- note added: "1"
- note added: "Hi-Z"
- note added: "Reset"
- note added: "aus"
- note added: "bei Reset"
- note added: "ein"
- note added: "kontinuierlicher Takt"
- note added: "sonst"

Commit message: viel Kleinkram
Parts:
- C10: value C -> 100n
- C3, C4: value CP -> 47u
- D1: value D -> 1N4148
- R17: value 10k -> 300k
- R18: value 10k -> 560
- R19: value 10k -> 3k3
Changed lines of the file:
@@
 P 1700 13600
 F 0 "D1" H 1700 13700 50  0000 C CNN
-F 1 "D" H 1700 13500 50  0000 C CNN
+F 1 "1N4148" H 1700 13500 50  0000 C CNN
 F 2 "Diode_THT:D_A-405_P10.16mm_Horizontal" H 1700 13600 50  0001 C CNN
 F 3 "" H 1700 13600 50  0001 C CNN
@@
 P 1350 8100
 F 0 "R19" H 1400 8150 39  0000 L CNN
-F 1 "10k" H 1420 8055 50  0000 L CNN
+F 1 "3k3" H 1420 8055 50  0000 L CNN
 F 2 "Resistor_THT:R_Axial_DIN0207_L6.3mm_D2.5mm_P10.16mm_Horizontal" V 1280 8100 50  0001 C CNN
 F 3 "" H 1350 8100 50  0000 C CNN
@@
 P 1350 7200
 F 0 "R18" H 1400 7250 39  0000 L CNN
-F 1 "10k" H 1420 7155 50  0000 L CNN
+F 1 "560" H 1420 7155 50  0000 L CNN
 F 2 "Resistor_THT:R_Axial_DIN0207_L6.3mm_D2.5mm_P10.16mm_Horizontal" V 1280 7200 50  0001 C CNN
 F 3 "" H 1350 7200 50  0000 C CNN
@@
 P 2950 6800
 F 0 "R17" H 3000 6850 39  0000 L CNN
-F 1 "10k" H 3020 6755 50  0000 L CNN
+F 1 "300k" H 3020 6755 50  0000 L CNN
 F 2 "Resistor_THT:R_Axial_DIN0207_L6.3mm_D2.5mm_P10.16mm_Horizontal" V 2880 6800 50  0001 C CNN
 F 3 "" H 2950 6800 50  0000 C CNN
@@
 P 2550 6300
 F 0 "C10" H 2665 6346 50  0000 L CNN
-F 1 "C" H 2665 6255 50  0000 L CNN
+F 1 "100n" H 2665 6255 50  0000 L CNN
 F 2 "Capacitor_THT:C_Disc_D10.0mm_W2.5mm_P5.00mm" H 2588 6150 50  0001 C CNN
 F 3 "~" H 2550 6300 50  0001 C CNN
@@
 P 1100 6300
 F 0 "C4" H 1218 6346 50  0000 L CNN
-F 1 "CP" H 1218 6255 50  0000 L CNN
+F 1 "47u" H 1218 6255 50  0000 L CNN
 F 2 "Capacitor_THT:CP_Radial_D10.0mm_P2.50mm_P5.00mm" H 1138 6150 50  0001 C CNN
 F 3 "~" H 1100 6300 50  0001 C CNN
@@
 P 1100 5950
 F 0 "C3" H 982 5904 50  0000 R CNN
-F 1 "CP" H 982 5995 50  0000 R CNN
+F 1 "47u" H 982 5995 50  0000 R CNN
 F 2 "Capacitor_THT:CP_Radial_D10.0mm_P2.50mm_P5.00mm" H 1138 5800 50  0001 C CNN
 F 3 "~" H 1100 5950 50  0001 C CNN
@@
 Text Notes 10500 13600 0    50   ~ 0
 1
+Text Notes 10950 12600 0    50   ~ 0
+Hi-Z
+Text Notes 10950 13350 0    50   ~ 0
+Hi-Z
+Text Notes 10950 13600 0    50   ~ 0
+Hi-Z
 Wire Bus Line
 	5950 1000 5950 1250
@@
 Wire Bus Line
 	5950 1250 8750 1250
-Text Notes 10950 12600 0    50   ~ 0
-Hi-Z
-Text Notes 10950 13350 0    50   ~ 0
-Hi-Z
-Text Notes 10950 13600 0    50   ~ 0
-Hi-Z
 $EndSCHEMATC
