File: speichermodul.kicad_pcb (KiCad board)
At the start: 2 copper layers, 100 x 160 mm, 69 parts, among them IC1 6116, J1 Conn_01x02, J2 Conn_01x02, J3 Conn_01x02, P1 CONN_3X2, P8 CONN_02X10, P9 CONN_02X10, SW1 Digitast rot, SW2 Digitast grün, U1 74HC00, U2 74HC08, U3 74HC14, U4 74HC14, U5 74LS540, U6 74LS540

Commit message: viele kleine Änderungen
Parts:
- added C9: 100n, Capacitor_THT:C_Disc_D10.0mm_W2.5mm_P5.00mm, F.Cu at (56.5, 52.7)
- moved D10 3.18 mm to (74.9, 131.4)
- moved D3 3.18 mm to (110.5, 131.4)
- moved D4 3.18 mm to (105.4, 131.4)
- moved D5 3.18 mm to (100.3, 131.4)
- moved D6 3.18 mm to (95.2, 131.4)
- moved D7 3.18 mm to (90.2, 131.4)
- moved D8 3.18 mm to (85.1, 131.4)
- moved D9 3.18 mm to (80.0, 131.4)
- moved U5 3.18 mm to (78.7, 158.8)
- moved C7 3.17 mm to (74.9, 152.4)
- moved R10 3.17 mm to (85.1, 134.6)
- moved R11 3.17 mm to (90.2, 134.6)
- moved R12 3.17 mm to (95.2, 134.6)
- moved R13 3.17 mm to (100.3, 134.6)
- moved R14 3.17 mm to (105.4, 134.6)
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Connections:
- net AUTO renamed ~AUTO
- net EN renamed ~writeEin
- net readMem renamed ~readMem
- net writeMem renamed ~writeMem
Routing:
- net GND: track 762.5 -> 776.5 mm
- net /D6: track 134.3 -> 147.0 mm
- net /D7: track 141.3 -> 154.0 mm
- net /D5: track 127.6 -> 140.0 mm
- net /D4: track 120.7 -> 129.3 mm
- net /D3: track 113.8 -> 121.6 mm
- net /D2: track 120.8 -> 127.2 mm
- net /D1: track 120.1 -> 125.3 mm
- net Net-(C9-Pad1): track 4.45 -> 8.89 mm
- net /D0: track 119.4 -> 123.7 mm
- net Net-(D1-Pad2): track 61.2 -> 57.2 mm
- net Net-(D2-Pad2): track 48.0 -> 49.8 mm
- net ~writeEin: track 168.0 -> 169.1 mm
- net VCC: track 477.5 -> 478.0 mm
Other:
- rule pad_to_mask_clearance: 0 -> 0.08
- rule solder_mask_min_width: 0.25 -> 0.254
- rule via_min_drill: 0.3 -> 0.4
- rule via_min_size: 0.4 -> 0.8
- board text added: "JLCJLCJLCJLC"
- board text added: "~auto"
- board text added: "~readMem"
- board text added: "~writeEin"
- board text added: "~writeMem"
- board text removed: "auto"
- board text removed: "enableEin"
- board text removed: "readMem"
- board text removed: "writeMem"

Commit message: viel Kleinkram
Parts:
- R7, R8: value R -> 150
Changed lines of the file:
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@@
     (descr "Resistor, Axial_DIN0207 series, Axial, Horizontal, pin pitch=10.16mm, 0.25W = 1/4W, length*diameter=6.3*2.5mm^2, http://cdn-reichelt.de/documents/datenblatt/B400/1_4W%23YAG.pdf")
     (tags "Resistor Axial_DIN0207 series Axial Horizontal pin pitch 10.16mm 0.25W = 1/4W length 6.3mm diameter 2.5mm")
-    (fp_text reference R8 (at 5.08 -2.37 90) (layer Eco2.User)
-      (effects (font (size 1 1) (thickness 0.15)))
-    )
-    (fp_text value R (at 5.08 2.37 90) (layer Eco2.User)
+    (fp_text reference R8 (at 6.985 0 90) (layer Eco2.User)
+      (effects (font (size 1 1) (thickness 0.15)))
+    )
+    (fp_text value 150 (at 3.175 0 90) (layer Eco2.User)
       (effects (font (size 1 1) (thickness 0.15)))
     )
@@
     (fp_line (start 11.21 1.5) (end 11.21 -1.5) (layer F.CrtYd) (width 0.05))
     (fp_line (start 11.21 -1.5) (end -1.05 -1.5) (layer F.CrtYd) (width 0.05))
-    (fp_text user %R (at 5.08 0 90) (layer Eco2.User)
+    (fp_text user %R (at 6.985 0 90) (layer Eco2.User) hide
       (effects (font (size 1 1) (thickness 0.15)))
     )
@@
     (descr "Resistor, Axial_DIN0207 series, Axial, Horizontal, pin pitch=10.16mm, 0.25W = 1/4W, length*diameter=6.3*2.5mm^2, http://cdn-reichelt.de/documents/datenblatt/B400/1_4W%23YAG.pdf")
     (tags "Resistor Axial_DIN0207 series Axial Horizontal pin pitch 10.16mm 0.25W = 1/4W length 6.3mm diameter 2.5mm")
-    (fp_text reference R7 (at 5.08 -2.37 90) (layer Eco2.User)
-      (effects (font (size 1 1) (thickness 0.15)))
-    )
-    (fp_text value R (at 5.08 2.37 90) (layer Eco2.User)
+    (fp_text reference R7 (at 6.985 0 90) (layer Eco2.User)
+      (effects (font (size 1 1) (thickness 0.15)))
+    )
+    (fp_text value 150 (at 3.175 0 90) (layer Eco2.User)
       (effects (font (size 1 1) (thickness 0.15)))
     )
@@
     (fp_line (start 11.21 1.5) (end 11.21 -1.5) (layer F.CrtYd) (width 0.05))
     (fp_line (start 11.21 -1.5) (end -1.05 -1.5) (layer F.CrtYd) (width 0.05))
-    (fp_text user %R (at 5.08 0 90) (layer Eco2.User)
+    (fp_text user %R (at 6.985 0 90) (layer Eco2.User) hide
       (effects (font (size 1 1) (thickness 0.15)))
     )
@@
   (segment (start 117.475 86.36) (end 115.57 86.36) (width 0.4) (layer F.Cu) (net 53))
   (segment (start 118.11 85.725) (end 117.475 86.36) (width 0.4) (layer F.Cu) (net 53))
-  (segment (start 65.405 165.735) (end 65.405 131.445) (width 0.4) (layer F.Cu) (net 82))
-  (segment (start 64.77 166.37) (end 65.405 165.735) (width 0.4) (layer F.Cu) (net 82))
-  (segment (start 65.405 127.635) (end 65.405 125.095) (width 0.4) (layer F.Cu) (net 82))
-  (segment (start 65.405 131.445) (end 65.405 127.635) (width 0.4) (layer F.Cu) (net 82))
-  (segment (start 65.405 127.635) (end 65.405 127) (width 0.4) (layer F.Cu) (net 82))
-  (segment (start 65.405 125.095) (end 68.58 121.92) (width 0.4) (layer F.Cu) (net 82))
-  (segment (start 68.58 121.92) (end 68.58 109.22) (width 0.4) (layer F.Cu) (net 82))
-  (segment (start 68.58 109.22) (end 60.96 101.6) (width 0.4) (layer F.Cu) (net 82))
-  (segment (start 60.96 101.6) (end 60.96 95.25) (width 0.4) (layer F.Cu) (net 82))
-  (segment (start 59.69 93.98) (end 59.69 92.075) (width 0.4) (layer F.Cu) (net 82))
-  (segment (start 60.96 95.25) (end 59.69 93.98) (width 0.4) (layer F.Cu) (net 82))
-  (segment (start 64.77 166.37) (end 46.355 166.37) (width 0.4) (layer F.Cu) (net 82))
-  (segment (start 52.07 92.075) (end 52.07 90.17) (width 0.4) (layer F.Cu) (net 82))
-  (segment (start 52.07 90.17) (end 52.705 89.535) (width 0.4) (layer F.Cu) (net 82))
-  (segment (start 52.705 89.535) (end 59.055 89.535) (width 0.4) (layer F.Cu) (net 82))
-  (segment (start 59.69 90.17) (end 59.69 92.075) (width 0.4) (layer F.Cu) (net 82))
-  (segment (start 59.055 89.535) (end 59.69 90.17) (width 0.4) (layer F.Cu) (net 82))
   (segment (start 110.49 131.445) (end 110.49 134.62) (width 1) (layer F.Cu) (net 54))
   (segment (start 105.41 134.62) (end 105.41 131.445) (width 1) (layer F.Cu) (net 55))
@@
   (segment (start 69.215 127) (end 72.39 123.825) (width 0.4) (layer F.Cu) (net 81))
   (segment (start 64.77 60.325) (end 55.245 60.325) (width 0.4) (layer F.Cu) (net 81))
+  (segment (start 65.405 165.735) (end 65.405 131.445) (width 0.4) (layer F.Cu) (net 82))
+  (segment (start 64.77 166.37) (end 65.405 165.735) (width 0.4) (layer F.Cu) (net 82))
+  (segment (start 65.405 127.635) (end 65.405 125.095) (width 0.4) (layer F.Cu) (net 82))
+  (segment (start 65.405 131.445) (end 65.405 127.635) (width 0.4) (layer F.Cu) (net 82))
+  (segment (start 65.405 127.635) (end 65.405 127) (width 0.4) (layer F.Cu) (net 82))
+  (segment (start 65.405 125.095) (end 68.58 121.92) (width 0.4) (layer F.Cu) (net 82))
+  (segment (start 68.58 121.92) (end 68.58 109.22) (width 0.4) (layer F.Cu) (net 82))
+  (segment (start 68.58 109.22) (end 60.96 101.6) (width 0.4) (layer F.Cu) (net 82))
+  (segment (start 60.96 101.6) (end 60.96 95.25) (width 0.4) (layer F.Cu) (net 82))
+  (segment (start 59.69 93.98) (end 59.69 92.075) (width 0.4) (layer F.Cu) (net 82))
+  (segment (start 60.96 95.25) (end 59.69 93.98) (width 0.4) (layer F.Cu) (net 82))
+  (segment (start 64.77 166.37) (end 46.355 166.37) (width 0.4) (layer F.Cu) (net 82))
+  (segment (start 52.07 92.075) (end 52.07 90.17) (width 0.4) (layer F.Cu) (net 82))
+  (segment (start 52.07 90.17) (end 52.705 89.535) (width 0.4) (layer F.Cu) (net 82))
+  (segment (start 52.705 89.535) (end 59.055 89.535) (width 0.4) (layer F.Cu) (net 82))
+  (segment (start 59.69 90.17) (end 59.69 92.075) (width 0.4) (layer F.Cu) (net 82))
+  (segment (start 59.055 89.535) (end 59.69 90.17) (width 0.4) (layer F.Cu) (net 82))
 )
