File: speichermodul.sch (KiCad schematic (older format))
At the start: 67 parts, among them IC1 6116, J1 2PinTerminalBlocktg, J2 2PinTerminalBlocktg, J3 2PinTerminalBlocktg, P1 CONN_3X2, P8 CONN_02X10, P9 CONN_02X10, SW1 SW_PUSH-tg, SW2 SW_PUSH-tg, U1 7400, U2 74LS08, U3 74LS08, U4 74LS14, U5 74LS540, U6 74LS540

Commit message: LEDs richtig rum gedreht
Connections:
- wire segments 318 -> 250
Changed lines of the file:
@@
 EESchema Schematic File Version 4
-EELAYER 29 0
+EELAYER 30 0
 EELAYER END
 $Descr A4 11693 8268
@@
 F 3 "~" H 7950 5550 60  0000 C CNN
 	1    7950 5550
-	0    1    1    0
+	0    -1   -1   0
 $EndComp
 $Comp
@@
 F 3 "~" H 8450 5550 60  0000 C CNN
 	1    8450 5550
-	0    1    1    0
+	0    -1   -1   0
 $EndComp
 $Comp
@@
 	5700 1650 5700 1850
 Wire Wire Line
-	37600 -12100 37600 -21800
-Wire Wire Line
-	37600 -21800 42950 -21800
-Wire Wire Line
-	42950 -21800 42950 -11850
-Wire Wire Line
-	42950 -11850 54850 -11850
-Wire Wire Line
-	54850 -11850 54850 -1350
-Wire Wire Line
-	54850 -1350 47700 -1350
-Wire Wire Line
-	47700 -1350 47700 20550
-Wire Wire Line
-	47700 20550 41950 20550
-Wire Wire Line
-	41950 20550 41950 12350
-Wire Wire Line
-	41950 12350 38500 12350
-Wire Wire Line
-	38500 12350 38500 20300
-Wire Wire Line
-	38500 20300 32700 20300
-Wire Wire Line
-	32700 20300 32700 -3000
-Wire Wire Line
-	32700 -3000 22850 -3000
-Wire Wire Line
-	22850 -3000 22850 -6100
-Wire Wire Line
-	22850 -6100 18500 -6100
-Wire Wire Line
-	18500 -6100 18500 -8000
-Wire Wire Line
-	18500 -8000 22500 -8000
-Wire Wire Line
-	18500 -8000 18500 -9000
-Wire Wire Line
-	18500 -9000 22500 -9000
-Connection ~ 18500 -8000
-Wire Wire Line
-	14550 -12100 37600 -12100
-Wire Wire Line
-	14550 -12100 14550 -9800
-Wire Wire Line
-	18500 -9000 18500 -9800
-Connection ~ 18500 -9000
-Wire Wire Line
-	18500 -9800 14550 -9800
-Wire Wire Line
-	38600 -18050 39500 -18050
-Wire Wire Line
-	39500 -18050 39500 -17550
-Wire Wire Line
-	39500 -17550 38600 -17550
-Wire Wire Line
-	38600 -17550 38600 -18050
-Wire Wire Line
-	41150 -17500 42450 -17500
-Wire Wire Line
-	42450 -17500 42450 -18050
-Wire Wire Line
-	42450 -18050 41150 -18050
-Wire Wire Line
-	41150 -18050 41150 -17500
-Wire Wire Line
-	39950 -15200 40600 -15200
-Wire Wire Line
-	40600 -15200 40600 -16450
-Wire Wire Line
-	40600 -16450 39950 -16450
-Wire Wire Line
-	39950 -16450 39950 -15200
-Wire Wire Line
-	38400 -13700 38800 -13700
-Wire Wire Line
-	38800 -13700 38800 -13200
-Wire Wire Line
-	38800 -13200 39350 -13200
-Wire Wire Line
-	39350 -13200 39350 -12650
-Wire Wire Line
-	39350 -12650 41600 -12650
-Wire Wire Line
-	41600 -12650 41600 -13100
-Wire Wire Line
-	41600 -13100 42150 -13100
-Wire Wire Line
-	42150 -13100 42150 -13700
-Wire Wire Line
-	42150 -13700 42600 -13700
-Wire Wire Line
-	42600 -13700 42600 -14300
-Wire Wire Line
-	42600 -14300 41850 -14300
-Wire Wire Line
-	41850 -14300 41850 -13600
-Wire Wire Line
-	41850 -13600 41500 -13600
-Wire Wire Line
-	41500 -13600 41500 -13150
-Wire Wire Line
-	41500 -13150 39650 -13150
-Wire Wire Line
-	39650 -13150 39650 -13650
-Wire Wire Line
-	39650 -13650 39200 -13650
-Wire Wire Line
-	39200 -13650 39200 -14050
-Wire Wire Line
-	39200 -14050 38400 -14050
-Wire Wire Line
-	38400 -14050 38400 -13700
-Wire Wire Line
-	55750 -26500 55750 -14450
-Wire Wire Line
-	55750 -14450 66900 -14450
-Wire Wire Line
-	71650 -25450 71650 -18950
-Wire Wire Line
-	71650 -18950 58050 -18950
-Wire Wire Line
-	66750 -25350 57150 -25350
-Wire Wire Line
-	57150 -25350 57150 -15850
-Wire Wire Line
-	57150 -15850 72550 -15850
-Wire Wire Line
-	60750 -21750 69950 -21750
-Wire Wire Line
-	69950 -21750 69950 -27500
-Wire Wire Line
-	69950 -27500 75100 -27500
-Wire Wire Line
-	75100 -27500 75100 -15100
-Wire Wire Line
-	75100 -15100 57050 -15100
-Wire Wire Line
 	10100 5800 10100 5700

Commit message: Speichermodul weitergebaut
Parts:
- added unit 7 of U4
Connections:
- wire segments 250 -> 301

Commit message: Speicher weitergebaut
Parts:
- removed J1, J2, J3: 2PinTerminalBlocktg, 2PinTerminalBlocktg, symbol allBonsaiSymbolLibs:2PinTerminalBlocktg-2PinTerminalBlocktg
- removed RP2: R_PACK8BUSSED, Housings_SIP:SIP9_Housing_BigPads, symbol allBonsaiSymbolLibs:R_PACK8BUSSED
- removed SW1, SW2: SW_PUSH-tg, tg_foodprint:SW_PUSH_LCD_E3_SAxxxx_tg_V2, symbol allBonsaiSymbolLibs:SW_PUSH-tg-switchlibtg
- removed U1: 7400, Housings_DIP:DIP-14_W7.62mm_LongPads, symbol allBonsaiSymbolLibs:7400
- removed U2, U3: 74LS08, Housings_DIP:DIP-14_W7.62mm_LongPads, symbol allBonsaiSymbolLibs:74LS08
- removed U4: 74LS14, Housings_DIP:DIP-14_W7.62mm_LongPads, symbol allBonsaiSymbolLibs:74LS14
- added C8: CP, Capacitor_THT:CP_Radial_D8.0mm_P2.50mm, symbol Device:CP
- added J1, J2, J3: Conn_01x02, Connector_Molex:Molex_KK-254_AE-6410-02A_1x02_P2.54mm_Vertical, symbol Connector_Generic:Conn_01x02
- added RN1: R_Network08, Resistor_THT:R_Array_SIP9, symbol Device:R_Network08
- added SW1, SW2: Digitast, bonsai:Switch_Digitast, symbol Bonsai:Digitast
- added U1: 74HC00, Package_DIP:DIP-14_W7.62mm_Socket_LongPads, symbol Bonsai:7400
- added U2, U3: 74HC08, Package_DIP:DIP-14_W7.62mm_Socket_LongPads, symbol Bonsai:7408
- added U4: 74HC14, Package_DIP:DIP-14_W7.62mm_Socket_LongPads, symbol Bonsai:7414
- C1, C6, C7: footprint Capacitors_ThroughHole:C_Disc_D10.0mm_W2.5mm_P5.00mm -> Capacitor_THT:C_Disc_D10.0mm_W2.5mm_P5.00mm
- C2, C3, C4, C5: footprint tg_foodprint:yyDisc_D10.0mm_W2.5mm_P.00mm -> Capacitor_THT:C_Disc_D10.0mm_W2.5mm_P5.00mm
- D1, D2: footprint LEDs:LED_D3.0mm -> LED_THT:LED_D3.0mm
- D10, D11, D12, D13, D14, D15, D16, D17, D18, D3, D4, D5, D6, D7, D8, D9: footprint LEDs:LED_D1.8mm_W1.8mm_H2.4mm_Horizontal_O3.81mm_Z8.2mm -> LED_THT:LED_D3.0mm
- IC1: footprint Housings_DIP:DIP-24_W15.24mm_Socket_LongPads -> Package_DIP:DIP-24_W15.24mm_Socket_LongPads
- P1: footprint Connectors_Samtec:SDL-106-X-XX_2x03 -> Connector_PinHeader_2.54mm:PinHeader_2x03_P2.54mm_Vertical
- P8: footprint Connectors_Samtec:SDL-120-X-XX_2x10 -> Connector_PinHeader_2.54mm:PinHeader_2x10_P2.54mm_Vertical
- P9: footprint Connect:IDC_Header_Straight_20pins -> Connector_PinHeader_2.54mm:PinHeader_2x10_P2.54mm_Vertical
- R1: value 1,7k -> 4k7; footprint Discret:R3 -> Resistor_THT:R_Axial_DIN0207_L6.3mm_D2.5mm_P10.16mm_Horizontal
- R10, R11, R12, R13, R14, R15, R16, R17, R18, R19, R20, R21, R22, R23, R4, R7, R8, R9: footprint Resistors_ThroughHole:R_Axial_DIN0207_L6.3mm_D2.5mm_P10.16mm_Horizontal -> Resistor_THT:R_Axial_DIN0207_L6.3mm_D2.5mm_P10.16mm_Horizontal
- R2: value 4,7k -> 4k7; footprint allBonsaiFootprintsLibs:R_Axial_DIN0207_L6.3mm_D2.5mm_P10.16mm_Horizontal -> Resistor_THT:R_Axial_DIN0207_L6.3mm_D2.5mm_P10.16mm_Horizontal
- R24, R25, R3: footprint Resistors_ThroughHole:R_Axial_DIN0309_L9.0mm_D3.2mm_P15.24mm_Horizontal -> Resistor_THT:R_Axial_DIN0207_L6.3mm_D2.5mm_P10.16mm_Horizontal
- R5: footprint allBonsaiFootprintsLibs:R_Axial_DIN0207_L6.3mm_D2.5mm_P10.16mm_Horizontal -> Resistor_THT:R_Axial_DIN0207_L6.3mm_D2.5mm_P10.16mm_Horizontal
- RP1: footprint Resistors_ThroughHole:R_Array_SIP5 -> Resistor_THT:R_Array_SIP5
- U5: footprint Housings_DIP:DIP-20_W7.62mm_Socket_LongPads -> Package_DIP:DIP-20_W7.62mm_Socket_LongPads; symbol allBonsaiSymbolLibs:74LS540 -> allBonsaiSymbolLibs:74LS540-74xx
- U6: footprint Housings_DIP:DIP-20_W7.62mm_LongPads -> Package_DIP:DIP-20_W7.62mm_Socket_LongPads; symbol allBonsaiSymbolLibs:74LS540 -> allBonsaiSymbolLibs:74LS540-74xx
Connections:
- wire segments 301 -> 311

Commit message: Speicher Layout EinTaktReset VCO
Parts:
- D36: footprint Diodes_ThroughHole:D_DO-41_SOD81_P10.16mm_Horizontal -> Diode_THT:D_A-405_P10.16mm_Horizontal
- SW1: value Digitast -> Digitast rot
- SW2: value Digitast -> Digitast grün
Connections:
- net labels added: readMem, writeMem
- net labels removed: RD, WR
- no-connect marks 1 -> 3
Changed lines of the file:
@@
 Text Label 12400 3550 0    60   Italic 0
 A7
-Connection ~ 2150 6750
-Wire Wire Line
-	2150 6000 2150 6750
+Connection ~ 2150 6800
+Wire Wire Line
+	2150 6000 2150 6800
 Wire Wire Line
 	3600 6000 2150 6000
@@
 	3750 5550 3250 5550
 Wire Wire Line
-	3750 6750 3250 6750
-Wire Wire Line
-	2250 6650 2250 6750
-Connection ~ 2250 6750
-Wire Wire Line
-	3750 6550 3600 6550
-Wire Wire Line
-	3600 6550 3600 6350
+	3750 6800 3250 6800
+Wire Wire Line
+	2250 6700 2250 6800
+Connection ~ 2250 6800
+Wire Wire Line
+	3750 6600 3600 6600
+Wire Wire Line
+	3600 6600 3600 6350
 Wire Wire Line
 	2050 4200 2050 4500
@@
 	3600 6350 2050 6350
 Wire Wire Line
-	2150 7250 2150 6750
+	2150 7250 2150 6800
 Wire Wire Line
 	1100 5700 1100 5750
 Wire Wire Line
-	5000 6650 4850 6650
+	5000 6700 4850 6700
 Wire Wire Line
 	5000 5650 4850 5650
@@
 	7500 6150 6350 6150
 Wire Wire Line
-	6350 6600 6100 6550
+	6350 6600 6100 6600
 Connection ~ 7500 6450
 Wire Wire Line
@@
 	14850 2450 14800 2450
 Wire Wire Line
-	2150 6750 2250 6750
-Wire Wire Line
-	5000 6150 5000 6450
+	2150 6800 2250 6800
+Wire Wire Line
+	5000 6150 5000 6500
 Wire Wire Line
 	7500 6450 7500 6500
@@
 	2050 4800 2050 5050
 Wire Wire Line
-	2250 6750 2250 6850
+	2250 6800 2250 6900
 Wire Wire Line
 	1800 7250 1800 7150
@@
 F 0 "D36" V 2001 3228 50  0000 L CNN
 F 1 "D" V 2092 3228 50  0000 L CNN
-F 2 "Diodes_ThroughHole:D_DO-41_SOD81_P10.16mm_Horizontal" V 2191 3228 60  0001 L CNN
+F 2 "Diode_THT:D_A-405_P10.16mm_Horizontal" V 2191 3228 60  0001 L CNN
 F 3 "" H 2100 3150 60  0000 C CNN
 	1    2100 3150
@@
 EN
 Text GLabel 7500 5350 0    50   Output ~ 0
-RD
+writeMem
 Text GLabel 1100 6200 3    50   Output ~ 0
 AUTO
-Text GLabel 7850 7100 0    50   Output ~ 0
-WR
+Text GLabel 7950 7100 0    50   Output ~ 0
+readMem
 Wire Wire Line
 	2250 5450 2250 5550
@@
 	2050 5050 1900 5050
 Connection ~ 2050 5550
-Text GLabel 1300 2000 2    50   Input ~ 0
+Text GLabel 1800 2150 2    50   Input ~ 0
 EN
 Wire Wire Line
-	1300 2000 1150 2000
-Wire Wire Line
-	1300 1900 1150 1900
-Text GLabel 1350 2200 2    50   Input ~ 0
-RD
-Text GLabel 1300 2300 2    50   Input ~ 0
+	1800 2150 1650 2150
+Wire Wire Line
+	1850 1850 1650 1850
+Text GLabel 1850 1950 2    50   Input ~ 0
+writeMem
+Text GLabel 1800 2250 2    50   Input ~ 0
 AUTO
-Text GLabel 1300 1900 2    50   Input ~ 0
-WR
-Wire Wire Line
-	1350 2200 1150 2200
-Wire Wire Line
-	1300 2300 1150 2300
+Text GLabel 1850 1850 2    50   Input ~ 0
+readMem
+Wire Wire Line
+	1850 1950 1650 1950
+Wire Wire Line
+	1800 2250 1650 2250
 $Comp
 L Connector_Generic:Conn_01x02 J2
 U 1 1 6007B890
-P 950 2200
-F 0 "J2" H 1030 2192 50  0000 L CNN
-F 1 "Conn_01x02" H 1030 2101 50  0000 L CNN
-F 2 "Connector_Molex:Molex_KK-254_AE-6410-02A_1x02_P2.54mm_Vertical" H 950 2200 50  0001 C CNN
-F 3 "~" H 950 2200 50  0001 C CNN
-	1    950  2200
+P 1450 2150
+F 0 "J2" H 1530 2142 50  0000 L CNN
+F 1 "Conn_01x02" H 1530 2051 50  0000 L CNN
+F 2 "Connector_Molex:Molex_KK-254_AE-6410-02A_1x02_P2.54mm_Vertical" H 1450 2150 50  0001 C CNN
+F 3 "~" H 1450 2150 50  0001 C CNN
+	1    1450 2150
 	-1   0    0    -1
 $EndComp
@@
 L Connector_Generic:Conn_01x02 J1
 U 1 1 6007BB67
-P 950 1900
-F 0 "J1" H 1030 1892 50  0000 L CNN
-F 1 "Conn_01x02" H 1030 1801 50  0000 L CNN
-F 2 "Connector_Molex:Molex_KK-254_AE-6410-02A_1x02_P2.54mm_Vertical" H 950 1900 50  0001 C CNN
-F 3 "~" H 950 1900 50  0001 C CNN
-	1    950  1900
+P 1450 1850
+F 0 "J1" H 1530 1842 50  0000 L CNN
+F 1 "Conn_01x02" H 1530 1751 50  0000 L CNN
+F 2 "Connector_Molex:Molex_KK-254_AE-6410-02A_1x02_P2.54mm_Vertical" H 1450 1850 50  0001 C CNN
+F 3 "~" H 1450 1850 50  0001 C CNN
+	1    1450 1850
 	-1   0    0    -1
 $EndComp
@@
 P 1400 4950
 F 0 "SW1" H 1400 5286 50  0000 C CNN
-F 1 "Digitast" H 1400 5195 50  0000 C CNN
+F 1 "Digitast rot" H 1400 5195 50  0000 C CNN
 F 2 "bonsai:Switch_Digitast" H 1400 5202 60  0001 C CNN
 F 3 "" H 1400 4950 60  0000 C CNN
@@
 P 1100 7150
 F 0 "SW2" H 1100 7486 50  0000 C CNN
-F 1 "Digitast" H 1100 7395 50  0000 C CNN
+F 1 "Digitast grün" H 1100 7395 50  0000 C CNN
 F 2 "bonsai:Switch_Digitast" H 1100 6919 60  0001 C CNN
 F 3 "" H 1100 7150 60  0000 C CNN
@@
 L Bonsai:7400 U1
 U 4 1 60A695B7
-P 2750 6750
-F 0 "U1" H 2750 6900 50  0000 C CNN
-F 1 "74HC00" H 2750 6600 50  0000 C CNN
-F 2 "Package_DIP:DIP-14_W7.62mm_Socket_LongPads" H 2750 6750 50  0001 C CNN
-F 3 "" H 2750 6750 50  0001 C CNN
-	4    2750 6750
+P 2750 6800
+F 0 "U1" H 2750 6950 50  0000 C CNN
+F 1 "74HC00" H 2750 6650 50  0000 C CNN
+F 2 "Package_DIP:DIP-14_W7.62mm_Socket_LongPads" H 2750 6800 50  0001 C CNN
+F 3 "" H 2750 6800 50  0001 C CNN
+	4    2750 6800
 	1    0    0    -1
 $EndComp
@@
 L Bonsai:7408 U2
 U 2 1 60BC8E49
-P 4300 6650
-F 0 "U2" H 4300 6500 50  0000 C CNN
-F 1 "74HC08" H 4300 6800 50  0000 C CNN
-F 2 "Package_DIP:DIP-14_W7.62mm_Socket_LongPads" H 4300 6650 50  0001 C CNN
-F 3 "" H 4300 6650 50  0001 C CNN
-	2    4300 6650
+P 4300 6700
+F 0 "U2" H 4300 6550 50  0000 C CNN
+F 1 "74HC08" H 4300 6850 50  0000 C CNN
+F 2 "Package_DIP:DIP-14_W7.62mm_Socket_LongPads" H 4300 6700 50  0001 C CNN
+F 3 "" H 4300 6700 50  0001 C CNN
+	2    4300 6700
 	1    0    0    1
 $EndComp
@@
 L Bonsai:7408 U2
 U 3 1 60BE6C52
-P 5550 6550
-F 0 "U2" H 5550 6400 50  0000 C CNN
-F 1 "74HC08" H 5550 6700 50  0000 C CNN
-F 2 "Package_DIP:DIP-14_W7.62mm_Socket_LongPads" H 5550 6550 50  0001 C CNN
-F 3 "" H 5550 6550 50  0001 C CNN
-	3    5550 6550
+P 5550 6600
+F 0 "U2" H 5550 6450 50  0000 C CNN
+F 1 "74HC08" H 5550 6750 50  0000 C CNN
+F 2 "Package_DIP:DIP-14_W7.62mm_Socket_LongPads" H 5550 6600 50  0001 C CNN
+F 3 "" H 5550 6600 50  0001 C CNN
+	3    5550 6600
 	1    0    0    1
 $EndComp
@@
 Wire Wire Line
 	1800 3300 1800 3350
+Connection ~ 1800 3350
+Wire Wire Line
+	1800 3350 2100 3350
+$Comp
+L Bonsai:7414 U4
+U 6 1 6114C53D
+P 7500 8900
+F 0 "U4" V 7454 9078 50  0000 L CNN
+F 1 "74HC14" V 7545 9078 50  0000 L CNN
+F 2 "Package_DIP:DIP-14_W7.62mm_Socket_LongPads" H 7550 8900 50  0001 C CNN
+F 3 "" H 7550 8900 50  0001 C CNN
+	6    7500 8900
+	0    1    1    0
+$EndComp
+NoConn ~ 1900 4850
+NoConn ~ 1600 7050
 Wire Bus Line
 	10500 3900 10500 6150
@@
 Wire Bus Line
 	12450 5350 12450 9100
-Connection ~ 1800 3350
-Wire Wire Line
-	1800 3350 2100 3350
-$Comp
-L Bonsai:7414 U4
-U 6 1 6114C53D
-P 7500 8900
-F 0 "U4" V 7454 9078 50  0000 L CNN
-F 1 "74HC14" V 7545 9078 50  0000 L CNN
-F 2 "Package_DIP:DIP-14_W7.62mm_Socket_LongPads" H 7550 8900 50  0001 C CNN
-F 3 "" H 7550 8900 50  0001 C CNN
-	6    7500 8900
-	0    1    1    0
-$EndComp
 $EndSCHEMATC

Commit message: Speicher vor Tausch der Taster
Parts:
- added unit 3 of U3
- added unit 5 of U4
- added unit 4 of U4
- U3: value 74HC08 -> 74HC14
Connections:
- wire segments 311 -> 317
- no-connect marks 3 -> 6
Changed lines of the file:
@@
 P 8150 5750
 F 0 "U3" H 8150 5850 50  0000 C CNN
-F 1 "74HC08" H 8150 5600 50  0000 C CNN
+F 1 "74HC14" H 8150 5600 50  0000 C CNN
 F 2 "Package_DIP:DIP-14_W7.62mm_Socket_LongPads" H 8150 5750 50  0001 C CNN
 F 3 "" H 8150 5750 50  0001 C CNN
@@
 P 9550 5850
 F 0 "U3" H 9550 5950 50  0000 C CNN
-F 1 "74HC08" H 9550 5700 50  0000 C CNN
+F 1 "74HC14" H 9550 5700 50  0000 C CNN
 F 2 "Package_DIP:DIP-14_W7.62mm_Socket_LongPads" H 9550 5850 50  0001 C CNN
 F 3 "" H 9550 5850 50  0001 C CNN
@@
 P 8150 6550
 F 0 "U3" H 8150 6650 50  0000 C CNN
-F 1 "74HC08" H 8150 6400 50  0000 C CNN
+F 1 "74HC14" H 8150 6400 50  0000 C CNN
 F 2 "Package_DIP:DIP-14_W7.62mm_Socket_LongPads" H 8150 6550 50  0001 C CNN
 F 3 "" H 8150 6550 50  0001 C CNN
@@
 P 7700 3250
 F 0 "U3" H 7700 3350 50  0000 C CNN
-F 1 "74HC08" H 7700 3100 50  0000 C CNN
+F 1 "74HC14" H 7700 3100 50  0000 C CNN
 F 2 "Package_DIP:DIP-14_W7.62mm_Socket_LongPads" H 7700 3250 50  0001 C CNN
 F 3 "" H 7700 3250 50  0001 C CNN
@@
 NoConn ~ 1900 4850
 NoConn ~ 1600 7050
+$Comp
+L Bonsai:7408 U3
+U 3 1 5FE0EEBD
+P 7250 1750
+F 0 "U3" H 7250 1850 50  0000 C CNN
+F 1 "74HC14" H 7250 1600 50  0000 C CNN
+F 2 "Package_DIP:DIP-14_W7.62mm_Socket_LongPads" H 7250 1750 50  0001 C CNN
+F 3 "" H 7250 1750 50  0001 C CNN
+	3    7250 1750
+	1    0    0    -1
+$EndComp
+$Comp
+L power:VCC #PWR0110
+U 1 1 5FE0F3DA
+P 6650 1550
+F 0 "#PWR0110" H 6650 1400 50  0001 C CNN
+F 1 "VCC" H 6667 1723 50  0000 C CNN
+F 2 "" H 6650 1550 50  0000 C CNN
+F 3 "" H 6650 1550 50  0000 C CNN
+	1    6650 1550
+	1    0    0    -1
+$EndComp
+Wire Wire Line
+	6650 1550 6650 1650
+Wire Wire Line
+	6650 1850 6700 1850
+Wire Wire Line
+	6700 1650 6650 1650
+Connection ~ 6650 1650
+Wire Wire Line
+	6650 1650 6650 1850
+$Comp
+L Bonsai:7414 U4
+U 5 1 5FE4C703
+P 10300 1750
+F 0 "U4" V 10254 1928 50  0000 L CNN
+F 1 "74HC14" V 10345 1928 50  0000 L CNN
+F 2 "Package_DIP:DIP-14_W7.62mm_Socket_LongPads" H 10350 1750 50  0001 C CNN
+F 3 "" H 10350 1750 50  0001 C CNN
+	5    10300 1750
+	1    0    0    -1
+$EndComp
+$Comp
+L power:VCC #PWR0112
+U 1 1 5FFAD0F7
+P 9750 1750
+F 0 "#PWR0112" H 9750 1600 50  0001 C CNN
+F 1 "VCC" H 9767 1923 50  0000 C CNN
+F 2 "" H 9750 1750 50  0000 C CNN
+F 3 "" H 9750 1750 50  0000 C CNN
+	1    9750 1750
+	1    0    0    -1
+$EndComp
+Wire Wire Line
+	9750 1750 9850 1750
+$Comp
+L Bonsai:7414 U4
+U 4 1 60044C43
+P 9100 1750
+F 0 "U4" V 9054 1928 50  0000 L CNN
+F 1 "74HC14" V 9145 1928 50  0000 L CNN
+F 2 "Package_DIP:DIP-14_W7.62mm_Socket_LongPads" H 9150 1750 50  0001 C CNN
+F 3 "" H 9150 1750 50  0001 C CNN
+	4    9100 1750
+	1    0    0    -1
+$EndComp
+$Comp
+L power:VCC #PWR027
+U 1 1 600464A4
+P 8550 1750
+F 0 "#PWR027" H 8550 1600 50  0001 C CNN
+F 1 "VCC" H 8567 1923 50  0000 C CNN
+F 2 "" H 8550 1750 50  0000 C CNN
+F 3 "" H 8550 1750 50  0000 C CNN
+	1    8550 1750
+	1    0    0    -1
+$EndComp
+Wire Wire Line
+	8650 1750 8550 1750
+NoConn ~ 7800 1750
+NoConn ~ 9550 1750
+NoConn ~ 10750 1750
 Wire Bus Line
 	10500 3900 10500 6150

Commit message: viele kleine Änderungen
Parts:
- added C9: 100n, Capacitor_THT:C_Disc_D10.0mm_W2.5mm_P5.00mm, symbol allBonsaiSymbolLibs:C
Connections:
- net labels added: ~AUTO, ~readMem, ~writeEin, ~writeMem
- net labels removed: AUTO, EN, readMem, writeMem
- wire segments 317 -> 328
Other:
- note added: "read"
- note added: "write"

Commit message: viel Kleinkram
Parts:
- R7, R8: value R -> 150
Changed lines of the file:
@@
 P 9050 8000
 F 0 "R7" V 9130 8000 40  0000 C CNN
-F 1 "R" V 9057 8001 40  0000 C CNN
+F 1 "150" V 9057 8001 40  0000 C CNN
 F 2 "Resistor_THT:R_Axial_DIN0207_L6.3mm_D2.5mm_P10.16mm_Horizontal" V 8980 8000 30  0001 C CNN
 F 3 "~" H 9050 8000 30  0000 C CNN
@@
 P 9550 8000
 F 0 "R8" V 9630 8000 40  0000 C CNN
-F 1 "R" V 9557 8001 40  0000 C CNN
+F 1 "150" V 9557 8001 40  0000 C CNN
 F 2 "Resistor_THT:R_Axial_DIN0207_L6.3mm_D2.5mm_P10.16mm_Horizontal" V 9480 8000 30  0001 C CNN
 F 3 "~" H 9550 8000 30  0000 C CNN
