File: power/power.kicad_pcb (KiCad board)
At the start: 2 copper layers, 70 x 65 mm, 27 parts, among them J1 CLIFF_FCR681465P, J10 Conn_01x02, J11 Conn_01x02, J12 Conn_01x02, J2 Screw_Terminal_01x02, J3 Conn_01x02, J4 Conn_01x02, J5 Conn_01x02, J7 Conn_01x02, J8 Conn_01x02, J9 Conn_01x02, Q1 IRF9530, U1 L7805

Commit message: - alles auf KiCad 7 umgestellt - EinTaktReset neu (mit Mikrocontroller)
Other:
- net class Default removed
