File: Akku-PC/Akku.kicad_pcb (KiCad board)
At the start: 2 copper layers, 100 x 160 mm, 60 parts, among them J1 Conn_02x10_Odd_Even, J2 Conn_01x02, J3 Conn_01x04, J4 Conn_01x02, J5 Conn_02x10_Odd_Even, J6 Conn_02x10_Odd_Even, J7 Conn_01x02, J8 Conn_01x02, SW1 Digitast, SW2 Digitast, SW3 Digitast, U1 74HC14, U2 74HC00, U4 74HC08, U5 74LS193, U6 74LS541, U7 74LS193, U8 74LS540

Commit message: Alle Vorwiderstände vor LEDs in 680 Ohm geändert (Issue 5)
Parts:
- R10, R11, R14, R9: value 150 -> 680
- R13, R15, R16, R17, R18, R19, R20, R21: value 330 -> 680
- RPA1: value R_PACK4BUSSED -> R_PACK4BUSSED 4k7
- U5, U7: value 74LS193 -> 74HCT193
- U6: value 74LS541 -> 74HC541
- U8: value 74LS540 -> 74HC540
Connections:
- U4 pad 6: Net-(U4-Pad6) -> unconnected-(U4-Pad6)
- U4 pad 8: Net-(U4-Pad8) -> unconnected-(U4-Pad8)
- U5 pad 12: Net-(U5-Pad12) -> unconnected-(U5-TcUp-Pad12)
- U5 pad 13: Net-(U5-Pad13) -> unconnected-(U5-TcDw-Pad13)
