File: Befehle/Befehle.kicad_pcb (KiCad board)
At the start: 2 copper layers, 100 x 160 mm, 78 parts, among them J1 Conn_02x10_Odd_Even, J2 Conn_01x02, J3 Conn_01x04, J4 Conn_02x10_Odd_Even, J5 Conn_01x02, J6 Conn_01x04, U1 74LS14, U2 74LS541, U3 74LS540, U4 74HC139, U5 74HCT373, U6 74HC540, U7 74HCT02, U8 7408, U9 7400

Commit message: Alle Vorwiderstände vor LEDs in 680 Ohm geändert (Issue 5)
Parts:
- R1, R10, R12, R13, R14, R15, R16, R17, R2, R3, R4, R5, R6, R7, R8: value 330 -> 680
- RP1: value R_PACK4BUSSED -> R_PACK4BUSSED 10k
- U1: value 74LS14 -> 74HC14
- U2: value 74LS541 -> 74HC541
- U3: value 74LS540 -> 74HC540
- U8: value 7408 -> 74HC08
- U9: value 7400 -> 74HC00
Connections:
- J2 pad 2: Net-(J2-Pad2) -> unconnected-(J2-Pin_2-Pad2)
- U1 pad 8: Net-(U1-Pad8) -> unconnected-(U1-Pad8)
- U4 pad 10: Net-(U4-Pad10) -> unconnected-(U4B-O2-Pad10)
- U4 pad 11: Net-(U4-Pad11) -> unconnected-(U4B-O1-Pad11)
- U4 pad 12: Net-(U4-Pad12) -> unconnected-(U4B-O0-Pad12)
- U4 pad 9: Net-(U4-Pad9) -> unconnected-(U4B-O3-Pad9)
- U6 pad 13: Net-(U6-Pad13) -> unconnected-(U6-Pad13)
- U6 pad 14: Net-(U6-Pad14) -> unconnected-(U6-Pad14)
- U9 pad 11: Net-(U9-Pad11) -> unconnected-(U9-Pad11)
- U9 pad 8: Net-(U9-Pad8) -> unconnected-(U9-Pad8)
