File: EinTaktReset/EinTaktReset.kicad_pcb (KiCad board)
At the start: 2 copper layers, 100 x 160 mm, 45 parts, among them J1 Conn_01x02, J2 Conn_01x03, J3 Conn_01x03, J4 Conn_01x03, J5 Conn_01x02, J6 Conn_01x02, J7 Conn_02x03_Odd_Even, P1 CONN_02X10, P4 CONN_02X10, SW1 Digitast, SW10 SPST, SW11 SPST, SW12 SPST, SW13 SPST, SW2 Digitast, SW3 SW_SPDT, SW4 SW_SPDT, SW5 SPST, SW6 SW_SPDT, SW7 SPST, SW8 SPST, SW9 SPST, U2 ATmega48-20P, U3 74HC541, U5 7400, Y1 Crystal

Commit message: Alle Vorwiderstände vor LEDs in 680 Ohm geändert (Issue 5)
Parts:
- R4, R7: value 330 -> 680
- RP1: value R_PACK8BUSSED -> R_PACK8BUSSED 10k
- U5: value 7400 -> 74HC00
- Y1: value Crystal -> Crystal 10 MHz
Changed lines of the file:
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@@
         (effects (font (size 1 1) (thickness 0.15)))
     )
-    (fp_text value "R_PACK8BUSSED" (at 11.43 2.4) (layer "Eco2.User")
+    (fp_text value "R_PACK8BUSSED 10k" (at 11.43 2.4) (layer "Eco2.User")
         (effects (font (size 1 1) (thickness 0.15)))
     )
@@
         (effects (font (size 1 1) (thickness 0.15)))
     )
-    (fp_text value "330" (at 5.08 2.37 90) (layer "Eco2.User")
+    (fp_text value "680" (at 5.08 2.37 90) (layer "Eco2.User")
         (effects (font (size 1 1) (thickness 0.15)))
     )
@@
         (effects (font (size 1 1) (thickness 0.15)))
     )
-    (fp_text value "330" (at 5.08 2.37 90) (layer "Eco2.User")
+    (fp_text value "680" (at 5.08 2.37 90) (layer "Eco2.User")
         (effects (font (size 1 1) (thickness 0.15)))
     )
@@
         (effects (font (size 1 1) (thickness 0.15)))
     )
-    (fp_text value "7400" (at 3.81 17.57 90) (layer "Eco2.User")
+    (fp_text value "74HC00" (at 3.81 17.57 90) (layer "Eco2.User")
         (effects (font (size 1 1) (thickness 0.15)))
     )
@@
         (effects (font (size 1 1) (thickness 0.15)))
     )
-    (fp_text value "Crystal" (at 2.44 3.525) (layer "F.Fab")
+    (fp_text value "Crystal 10 MHz" (at 2.44 3.525) (layer "F.Fab")
         (effects (font (size 1 1) (thickness 0.15)))
     )
