File: Speicher/speichermodul.kicad_pcb (KiCad board)
At the start: 2 copper layers, 100 x 160 mm, 70 parts, among them IC1 6116, J1 Conn_01x02, J2 Conn_01x02, J3 Conn_01x02, P1 CONN_3X2, P8 CONN_02X10, P9 CONN_02X10, SW1 Digitast rot, SW2 Digitast grün, U1 74HC00, U2 74HC08, U3 74HC14, U4 74HC14, U5 74LS540, U6 74LS540

Commit message: Alle Vorwiderstände vor LEDs in 680 Ohm geändert (Issue 5)
Parts:
- IC1: value 6116 -> M48Z02
- R10, R11, R12, R13, R14, R15, R16, R17, R18, R19, R20, R21, R22, R23, R4, R9: value 330 -> 680
- R7, R8: value 150 -> 680
- RN1: value R_Network08 -> R_Network08 10k
- U5, U6: value 74LS540 -> 74HCT540
Connections:
- RP1 pad 5: Net-(RP1-Pad5) -> unconnected-(RP1-P5-Pad5)
- SW1 pad 2: Net-(SW1-Pad2) -> unconnected-(SW1-Pad2)
- SW2 pad 2: Net-(SW2-Pad2) -> unconnected-(SW2-Pad2)
- U3 pad 8: Net-(U3-Pad8) -> unconnected-(U3-Pad8)
- U4 pad 10: Net-(U4-Pad10) -> unconnected-(U4-Pad10)
- U4 pad 8: Net-(U4-Pad8) -> unconnected-(U4-Pad8)
