File: Steuerwerk/Steuerwerk.kicad_pcb (KiCad board)
At the start: 2 copper layers, 100 x 160 mm, 332 parts, among them J1 Conn_01x04, J2 Conn_01x02, J3 Conn_01x03, J4 Conn_01x03, J5 Conn_01x02, J6 Conn_01x04, J7 Conn_01x02, J8 Conn_01x04, J9 Conn_01x02, Q1 Q_PNP_BCE, U1 74LS161, U2 74LS138, U3 74LS138, U4 74240, U5 74LS374, U6 74LS374, U7 74541, U8 74541

Commit message: Alle Vorwiderstände vor LEDs in 680 Ohm geändert (Issue 5)
Parts:
- R1, R10, R11, R12, R13, R14, R15, R16, R17, R18, R19, R20, R21, R22, R23, R3, R4, R5, R6, R7, R8, R9: value 330 -> 680
- RP1: value R_PACK8BUSSED -> R_PACK8BUSSED 10K
- RP2: value R_PACK8BUSSED -> R_PACK8BUSSED 10k
- U1: value 74LS161 -> 74LHC161
- U2, U3: value 74LS138 -> 74HC138
- U4: value 74240 -> 74HC240
- U5, U6: value 74LS374 -> 74HC374
- U7, U8: value 74541 -> 74HC541
Connections:
- U1 pad 15: Net-(U1-Pad15) -> unconnected-(U1-Tc-Pad15)
- U4 pad 12: Net-(U4-Pad12) -> unconnected-(U4-Pad12)
- U4 pad 14: Net-(U4-Pad14) -> unconnected-(U4-Pad14)
- U4 pad 16: Net-(U4-Pad16) -> unconnected-(U4-Pad16)
